File: ESP/Energy Monitor - ESP32 Integrated/Comm Interfaces.sch (KiCad schematic (older format))
At the start: 18 parts, among them J10 Conn_02x08_Odd_Even, J11 Conn_02x08_Odd_Even, J12 Conn_02x08_Odd_Even, J7 Conn_02x08_Odd_Even, J8 Conn_02x08_Odd_Even, J9 Conn_02x08_Odd_Even, U3 TCA9548APWR, U4 MCP23017_SO, U5 

Commit message: Layout and assembly.
Parts:
- added D10, D11, D7, D8, D9: LED_Small, custom:CHIPLED_0603, symbol Device:LED_Small
- added R37, R38: 499K, Resistor_SMD:R_0603_1608Metric_Pad1.05x0.95mm_HandSolder, symbol Device:R_Small
- added R39, R40, R41, R42, R43: 1K, Resistor_SMD:R_0603_1608Metric_Pad1.05x0.95mm_HandSolder, symbol Device:R_Small
- added U10, U11, U12, U13, U14, U15, U16, U17, U18, U19, U20, U21, U22, U23, U24, U9: QUAD-ESD-DIODE, Package_TO_SOT_SMD:SOT-23-6_Handsoldering, symbol custom:QUAD-ESD-DIODE
Connections:
- net labels added: SCL7, SCL8, SDA7, SDA8
- wire segments 297 -> 439
Other:
- note added: "Plugin-Boards \nhave pull ups. This allows \nboard detection by \nchecking SCL/SDA \nstate after switching \nmultiplexer"
- moved on the sheet: C16, R4, U5
