File: ESP/Energy Monitor - ESP32 Integrated/Energy Monitor - ESP32 Integrated.kicad_pcb (KiCad board)
At the start: 4 copper layers, 92 parts, among them J13 RJ45_Amphenol_RJMG1BD3B8K1ANR, J2 Conn_01x04, J3 Conn_01x04, J4 Conn_01x04, J5 Conn_01x05, J6 Conn_01x05, Q2 BC817-40(SOT23), Q3 BC817-40(SOT23), U1 TPS62082, U2 XL2001, U3 TCA9548APWR, U4 MCP23017_SO, U5 , U6 CH340C, U7 LAN8710A-EZC(QFN32), U8 ESP32-PICO-D4

Commit message: Layout and assembly.
Parts:
- removed D2, D3, D4, D5: BAT54S, Package_TO_SOT_SMD:SOT-23
- added C17: 1nF/2000V/10%/X7R/C1206, Capacitor_SMD:C_1206_3216Metric_Pad1.42x1.75mm_HandSolder, F.Cu at (23.0, -5.99)
- added D10: LED_Small, custom:CHIPLED_0603, F.Cu at (42.4, -36.5)
- added D11: LED_Small, custom:CHIPLED_0603, F.Cu at (44.8, -36.5)
- added D7: LED_Small, custom:CHIPLED_0603, F.Cu at (42.4, -40.1)
- added D8: LED_Small, custom:CHIPLED_0603, F.Cu at (38.0, -35.1)
- added D9: LED_Small, custom:CHIPLED_0603, F.Cu at (44.8, -40.1)
- added J10: Conn_02x08_Odd_Even, Connector_IDC:IDC-Header_2x08_P2.54mm_Vertical, F.Cu at (35.0, -76.0)
- added R37: 499K, Resistor_SMD:R_0603_1608Metric_Pad1.05x0.95mm_HandSolder, F.Cu at (56.1, -57.8)
- added R38: 499K, Resistor_SMD:R_0603_1608Metric_Pad1.05x0.95mm_HandSolder, F.Cu at (56.2, -56.2)
- added R39: 1K, Resistor_SMD:R_0603_1608Metric_Pad1.05x0.95mm_HandSolder, F.Cu at (34.7, -40.9)
- added R40: 1K, Resistor_SMD:R_0603_1608Metric_Pad1.05x0.95mm_HandSolder, F.Cu at (34.7, -38.4)
- added R41: 1K, Resistor_SMD:R_0603_1608Metric_Pad1.05x0.95mm_HandSolder, F.Cu at (39.0, -40.9)
- added R42: 1K, Resistor_SMD:R_0603_1608Metric_Pad1.05x0.95mm_HandSolder, F.Cu at (34.7, -35.8)
- added R43: 1K, Resistor_SMD:R_0603_1608Metric_Pad1.05x0.95mm_HandSolder, F.Cu at (39.0, -38.4)
- added U10: QUAD-ESD-DIODE, Package_TO_SOT_SMD:SOT-23-6_Handsoldering, F.Cu at (35.0, -64.8)
- added U11: QUAD-ESD-DIODE, Package_TO_SOT_SMD:SOT-23-6_Handsoldering, F.Cu at (29.2, -64.8)
- added U12: QUAD-ESD-DIODE, Package_TO_SOT_SMD:SOT-23-6_Handsoldering, B.Cu at (58.8, -79.8)
- added U13: QUAD-ESD-DIODE, Package_TO_SOT_SMD:SOT-23-6_Handsoldering, B.Cu at (38.8, -79.8)
- added U14: QUAD-ESD-DIODE, Package_TO_SOT_SMD:SOT-23-6_Handsoldering, B.Cu at (18.8, -79.8)
- added U15: QUAD-ESD-DIODE, Package_TO_SOT_SMD:SOT-23-6_Handsoldering, F.Cu at (52.5, -45.8)
- added U16: QUAD-ESD-DIODE, Package_TO_SOT_SMD:SOT-23-6_Handsoldering, F.Cu at (5.00, -64.8)
- added U17: QUAD-ESD-DIODE, Package_TO_SOT_SMD:SOT-23-6_Handsoldering, F.Cu at (5.00, -59.2)
- added U18: QUAD-ESD-DIODE, Package_TO_SOT_SMD:SOT-23-6_Handsoldering, F.Cu at (23.6, -64.0)
- added U19: QUAD-ESD-DIODE, Package_TO_SOT_SMD:SOT-23-6_Handsoldering, B.Cu at (68.2, -91.5)
- added U20: QUAD-ESD-DIODE, Package_TO_SOT_SMD:SOT-23-6_Handsoldering, B.Cu at (58.4, -91.5)
- added U21: QUAD-ESD-DIODE, Package_TO_SOT_SMD:SOT-23-6_Handsoldering, B.Cu at (48.2, -91.5)
- added U22: QUAD-ESD-DIODE, Package_TO_SOT_SMD:SOT-23-6_Handsoldering, B.Cu at (38.2, -91.5)
- added U23: QUAD-ESD-DIODE, Package_TO_SOT_SMD:SOT-23-6_Handsoldering, B.Cu at (28.2, -91.5)
- added U24: QUAD-ESD-DIODE, Package_TO_SOT_SMD:SOT-23-6_Handsoldering, B.Cu at (18.2, -91.5)
- added U9: QUAD-ESD-DIODE, Package_TO_SOT_SMD:SOT-23-6_Handsoldering, F.Cu at (40.8, -64.8)
- moved R22 154.6 mm to (96.2, -17.0), turned to 270 degrees
- moved Q3 152.9 mm to (90.0, -14.2)
- moved C21 151.1 mm to (92.8, -19.4), turned to 270 degrees
- moved C20 148.5 mm to (85.8, -22.0), turned to 90 degrees
- moved Q2 148.1 mm to (90.0, -18.0)
- moved R21 144.2 mm to (94.5, -19.4), turned to 90 degrees
- moved R18 142.4 mm to (92.8, -14.0), turned to 90 degrees
- moved C18 142.2 mm to (84.0, -22.0), turned to 90 degrees
- moved R17 141.5 mm to (87.5, -16.0), turned to 270 degrees
- moved C31 139.7 mm to (94.5, -15.8), turned to 90 degrees
- moved C19 131.8 mm to (77.8, -14.5), turned to 270 degrees
- moved R14 130.5 mm to (76.5, -19.8), turned to 180 degrees
- moved R16 130.0 mm to (89.5, -20.8), turned to 180 degrees
- moved R15 121.7 mm to (76.5, -17.8), turned to 180 degrees
- moved R2 114.0 mm to (90.2, -38.8), turned to 180 degrees
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Connections:
- net Net-(J13-PadR2) renamed /ESP32/TXN
- net Net-(J13-PadR3) renamed /ESP32/RXP
- net Net-(J13-PadR6) renamed /ESP32/RXN
- A1 pad 3: (no net) -> Net-(A1-Pad3)
- A1 pad 4: (no net) -> Net-(A1-Pad4)
- J13 pad R1: /ESP32/PHY_CT -> /ESP32/TXP
- J13 pad R7: (no net) -> Net-(J13-PadR7)
- R11 pad 2: /ESP32/PHY_CT -> /ESP32/TXP
- U1 pad 4: (no net) -> Net-(U1-Pad4)
- U1 pad 6: (no net) -> Net-(U1-Pad6)
- U2 pad 2: (no net) -> Net-(U2-Pad2)
- U3 pad 1: Net-(U3-Pad1) -> Net-(R41-Pad1)
- U3 pad 2: Net-(U3-Pad2) -> Net-(R40-Pad1)
- U3 pad 21: Net-(U3-Pad21) -> Net-(R39-Pad1)
- U4 pad 11: (no net) -> Net-(U4-Pad11)
- U4 pad 14: (no net) -> Net-(U4-Pad14)
- U4 pad 19: (no net) -> Net-(U4-Pad19)
- U4 pad 21: /COM/IRQ_9 -> Net-(R42-Pad1)
- U4 pad 22: /COM/IRQ_10 -> Net-(R41-Pad1)
- U4 pad 23: /COM/IRQ_11 -> Net-(R40-Pad1)
- U4 pad 24: /COM/IRQ_12 -> Net-(R39-Pad1)
- U4 pad 25: Net-(U4-Pad25) -> /COM/IRQ_9
- U4 pad 26: Net-(U3-Pad1) -> /COM/IRQ_10
- U4 pad 27: Net-(U3-Pad2) -> /COM/IRQ_11
- U4 pad 28: Net-(U3-Pad21) -> /COM/IRQ_12
- U5 pad 14: (no net) -> Net-(U5-Pad14)
- U5 pad 15: (no net) -> Net-(U5-Pad15)
- U5 pad 16: (no net) -> Net-(U5-Pad16)
- U5 pad 17: (no net) -> Net-(U5-Pad17)
- U5 pad 20: Net-(U3-Pad21) -> Net-(R39-Pad1)
- U5 pad 21: Net-(U3-Pad2) -> Net-(R40-Pad1)
- U5 pad 22: Net-(U3-Pad1) -> Net-(R41-Pad1)
- U5 pad 23: Net-(U4-Pad25) -> Net-(R42-Pad1)
- U6 pad 10: (no net) -> Net-(U6-Pad10)
- U6 pad 11: (no net) -> Net-(U6-Pad11)
- U6 pad 12: (no net) -> Net-(U6-Pad12)
- U6 pad 15: (no net) -> Net-(U6-Pad15)
- U6 pad 7: (no net) -> Net-(U6-Pad7)
- U6 pad 8: (no net) -> Net-(U6-Pad8)
- U6 pad 9: (no net) -> Net-(U6-Pad9)
- U7 pad 14: (no net) -> Net-(U7-Pad14)
- U7 pad 18: (no net) -> Net-(U7-Pad18)
- U7 pad 20: (no net) -> Net-(U7-Pad20)
- U7 pad 26: (no net) -> Net-(U7-Pad26)
- U7 pad 29: /ESP32/PHY_CT -> /ESP32/TXP
- U7 pad 4: (no net) -> Net-(U7-Pad4)
- U8 pad 20: (no net) -> Net-(U8-Pad20)
- U8 pad 28: (no net) -> Net-(U8-Pad28)
- U8 pad 29: (no net) -> Net-(U8-Pad29)
- U8 pad 30: (no net) -> Net-(U8-Pad30)
- U8 pad 31: (no net) -> Net-(U8-Pad31)
- U8 pad 32: (no net) -> Net-(U8-Pad32)
- U8 pad 33: (no net) -> Net-(U8-Pad33)
- U8 pad 34: (no net) -> Net-(U8-Pad34)
- U8 pad 44: (no net) -> Net-(U8-Pad44)
- U8 pad 45: (no net) -> Net-(U8-Pad45)
- U8 pad 47: (no net) -> Net-(U8-Pad47)
- U8 pad 48: (no net) -> Net-(U8-Pad48)
- U8 pad 5: (no net) -> Net-(U8-Pad5)
- U8 pad 6: (no net) -> Net-(U8-Pad6)
- U8 pad 7: (no net) -> Net-(U8-Pad7)
- U8 pad 8: (no net) -> Net-(U8-Pad8)
- UJ1 pad 1: (no net) -> Net-(UJ1-Pad1)
- UJ1 pad 4: (no net) -> Net-(UJ1-Pad4)
