File: ESP/Energy Monitor - ESP32 Integrated/External I2C 1-Wire.sch (KiCad schematic (older format))
At the start: 15 parts, among them J2 Conn_01x04, J3 Conn_01x04, J4 Conn_01x04, J5 Conn_01x05, J6 Conn_01x05

Commit message: Layout and assembly.
Parts:
- removed D2, D3, D4, D5: BAT54S, Package_TO_SOT_SMD:SOT-23, symbol Device:D_Schottky_x2_Serial_AKC
Changed lines of the file:
@@
 Wire Wire Line
 	4850 3700 4000 3700
-Wire Wire Line
-	3000 3800 4100 3800
 Text HLabel 3000 3700 0    50   Output ~ 0
 EXT_SDA_PT_2
@@
 Connection ~ 4000 3700
 Wire Wire Line
-	4000 3700 3550 3700
-Wire Wire Line
 	4300 3300 4300 3350
 Wire Wire Line
@@
 	4000 1450 4000 1650
 Connection ~ 4000 1650
-Wire Wire Line
-	4000 1650 3250 1650
 Wire Wire Line
 	4300 1200 4300 1250
@@
 Wire Wire Line
 	2350 6600 2350 5950
-$Comp
-L Device:D_Schottky_x2_Serial_AKC D5
-U 1 1 642D7D0B
-P 4300 4650
-F 0 "D5" V 4346 4730 50  0000 L CNN
-F 1 "BAT54S" V 4255 4730 50  0000 L CNN
-F 2 "Package_TO_SOT_SMD:SOT-23" H 4300 4650 50  0001 C CNN
-F 3 "~" H 4300 4650 50  0001 C CNN
-	1    4300 4650
-	0    1    -1   0
-$EndComp
-$Comp
-L power:+3.3V #PWR?
-U 1 1 642D7D11
-P 4300 4300
-AR Path="/5F5150CA/642D7D11" Ref="#PWR?"  Part="1"
-AR Path="/6379919C/642D7D11" Ref="#PWR0144"  Part="1"
-F 0 "#PWR0144" H 4300 4150 50  0001 C CNN
-F 1 "+3.3V" H 4315 4473 50  0000 C CNN
-F 2 "" H 4300 4300 50  0001 C CNN
-F 3 "" H 4300 4300 50  0001 C CNN
-	1    4300 4300
-	1    0    0    -1
-$EndComp
-$Comp
-L power:GND #PWR?
-U 1 1 642D7D17
-P 4300 5000
-AR Path="/5F5150CA/642D7D17" Ref="#PWR?"  Part="1"
-AR Path="/6379919C/642D7D17" Ref="#PWR0145"  Part="1"
-F 0 "#PWR0145" H 4300 4750 50  0001 C CNN
-F 1 "GND" H 4305 4827 50  0000 C CNN
-F 2 "" H 4300 5000 50  0001 C CNN
-F 3 "" H 4300 5000 50  0001 C CNN
-	1    4300 5000
-	1    0    0    -1
-$EndComp
-$Comp
-L Device:D_Schottky_x2_Serial_AKC D3
-U 1 1 642D91C1
-P 3750 4650
-F 0 "D3" V 3796 4730 50  0000 L CNN
-F 1 "BAT54S" V 3705 4730 50  0000 L CNN
-F 2 "Package_TO_SOT_SMD:SOT-23" H 3750 4650 50  0001 C CNN
-F 3 "~" H 3750 4650 50  0001 C CNN
-	1    3750 4650
-	0    1    -1   0
-$EndComp
-$Comp
-L power:+3.3V #PWR?
-U 1 1 642D91C7
-P 3750 4300
-AR Path="/5F5150CA/642D91C7" Ref="#PWR?"  Part="1"
-AR Path="/6379919C/642D91C7" Ref="#PWR0146"  Part="1"
-F 0 "#PWR0146" H 3750 4150 50  0001 C CNN
-F 1 "+3.3V" H 3765 4473 50  0000 C CNN
-F 2 "" H 3750 4300 50  0001 C CNN
-F 3 "" H 3750 4300 50  0001 C CNN
-	1    3750 4300
-	1    0    0    -1
-$EndComp
-$Comp
-L power:GND #PWR?
-U 1 1 642D91CD
-P 3750 5000
-AR Path="/5F5150CA/642D91CD" Ref="#PWR?"  Part="1"
-AR Path="/6379919C/642D91CD" Ref="#PWR0147"  Part="1"
-F 0 "#PWR0147" H 3750 4750 50  0001 C CNN
-F 1 "GND" H 3755 4827 50  0000 C CNN
-F 2 "" H 3750 5000 50  0001 C CNN
-F 3 "" H 3750 5000 50  0001 C CNN
-	1    3750 5000
-	1    0    0    -1
-$EndComp
-$Comp
-L Device:D_Schottky_x2_Serial_AKC D4
-U 1 1 642DEF8D
-P 4250 2450
-F 0 "D4" V 4296 2530 50  0000 L CNN
-F 1 "BAT54S" V 4205 2530 50  0000 L CNN
-F 2 "Package_TO_SOT_SMD:SOT-23" H 4250 2450 50  0001 C CNN
-F 3 "~" H 4250 2450 50  0001 C CNN
-	1    4250 2450
-	0    1    -1   0
-$EndComp
-$Comp
-L power:+3.3V #PWR?
-U 1 1 642DEF93
-P 4250 2100
-AR Path="/5F5150CA/642DEF93" Ref="#PWR?"  Part="1"
-AR Path="/6379919C/642DEF93" Ref="#PWR0148"  Part="1"
-F 0 "#PWR0148" H 4250 1950 50  0001 C CNN
-F 1 "+3.3V" H 4265 2273 50  0000 C CNN
-F 2 "" H 4250 2100 50  0001 C CNN
-F 3 "" H 4250 2100 50  0001 C CNN
-	1    4250 2100
-	1    0    0    -1
-$EndComp
-$Comp
-L power:GND #PWR?
-U 1 1 642DEF99
-P 4250 2800
-AR Path="/5F5150CA/642DEF99" Ref="#PWR?"  Part="1"
-AR Path="/6379919C/642DEF99" Ref="#PWR0149"  Part="1"
-F 0 "#PWR0149" H 4250 2550 50  0001 C CNN
-F 1 "GND" H 4255 2627 50  0000 C CNN
-F 2 "" H 4250 2800 50  0001 C CNN
-F 3 "" H 4250 2800 50  0001 C CNN
-	1    4250 2800
-	1    0    0    -1
-$EndComp
-$Comp
-L Device:D_Schottky_x2_Serial_AKC D2
-U 1 1 642E0B9E
-P 3450 2400
-F 0 "D2" V 3496 2480 50  0000 L CNN
-F 1 "BAT54S" V 3405 2480 50  0000 L CNN
-F 2 "Package_TO_SOT_SMD:SOT-23" H 3450 2400 50  0001 C CNN
-F 3 "~" H 3450 2400 50  0001 C CNN
-	1    3450 2400
-	0    1    -1   0
-$EndComp
-$Comp
-L power:+3.3V #PWR?
-U 1 1 642E0BA4
-P 3450 2050
-AR Path="/5F5150CA/642E0BA4" Ref="#PWR?"  Part="1"
-AR Path="/6379919C/642E0BA4" Ref="#PWR0150"  Part="1"
-F 0 "#PWR0150" H 3450 1900 50  0001 C CNN
-F 1 "+3.3V" H 3465 2223 50  0000 C CNN
-F 2 "" H 3450 2050 50  0001 C CNN
-F 3 "" H 3450 2050 50  0001 C CNN
-	1    3450 2050
-	1    0    0    -1
-$EndComp
-$Comp
-L power:GND #PWR?
-U 1 1 642E0BAA
-P 3450 2750
-AR Path="/5F5150CA/642E0BAA" Ref="#PWR?"  Part="1"
-AR Path="/6379919C/642E0BAA" Ref="#PWR0151"  Part="1"
-F 0 "#PWR0151" H 3450 2500 50  0001 C CNN
-F 1 "GND" H 3455 2577 50  0000 C CNN
-F 2 "" H 3450 2750 50  0001 C CNN
-F 3 "" H 3450 2750 50  0001 C CNN
-	1    3450 2750
-	1    0    0    -1
-$EndComp
-Wire Wire Line
-	4050 2450 4050 1750
-Connection ~ 4050 1750
-Wire Wire Line
-	4050 1750 4300 1750
-Wire Wire Line
-	3000 1750 4050 1750
-Wire Wire Line
-	3250 2400 3250 1650
-Connection ~ 3250 1650
-Wire Wire Line
-	3250 1650 3000 1650
-Wire Wire Line
-	4100 4650 4100 3800
-Connection ~ 4100 3800
-Wire Wire Line
-	4100 3800 4300 3800
-Wire Wire Line
-	3550 4650 3550 3700
-Connection ~ 3550 3700
-Wire Wire Line
-	3550 3700 3000 3700
-Wire Wire Line
-	3450 2050 3450 2100
-Wire Wire Line
-	3450 2700 3450 2750
-Wire Wire Line
-	4250 2100 4250 2150
-Wire Wire Line
-	4250 2750 4250 2800
-Wire Wire Line
-	3750 4300 3750 4350
-Wire Wire Line
-	3750 4950 3750 5000
-Wire Wire Line
-	4300 4950 4300 5000
 Wire Wire Line
 	2750 6250 2750 6300
@@
 Wire Wire Line
 	2350 6600 2550 6600
-Wire Wire Line
-	4300 4300 4300 4350
 Wire Wire Line
 	2350 5950 3450 5950
@@
 Wire Wire Line
 	4150 6150 4500 6150
+Wire Wire Line
+	3000 3800 4300 3800
+Wire Wire Line
+	3000 3700 4000 3700
+Wire Wire Line
+	3000 1750 4300 1750
+Wire Wire Line
+	3000 1650 4000 1650
 $EndSCHEMATC
