File: ESP/ESP32 Water Meter Monitor/ESP32 Water Meter Monitor.sch (KiCad schematic (older format))
At the start: 60 parts, among them J1 Conn_01x02, J11 Conn_01x05, J2 Conn_01x05, J3 Conn_01x01, J4 Conn_01x01, J5 Conn_01x05, J6 Conn_01x05, J7 Conn_01x05, SW1 SW_Push, SW2 SW_Push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

Commit message: Now with USB interface.
Parts:
- removed J2: Conn_01x05, Connector_PinHeader_2.54mm:PinHeader_1x05_P2.54mm_Vertical, symbol Connector_Generic:Conn_01x05
- removed J7: Conn_01x05, Connector_JST:JST_XH_B8B-XH-AM_1x08_P2.50mm_Vertical, symbol Connector_Generic:Conn_01x08
- added D14, D15: BAT54S, Package_TO_SOT_SMD:SOT-23, symbol Device:D_Schottky_x2_Serial_AKC
- added J7: Conn_01x09, Connector_JST:JST_XH_B9B-XH-AM_1x09_P2.50mm_Vertical, symbol Connector_Generic:Conn_01x09
- J6: value Conn_01x05 -> Conn_01x09; footprint Connector_JST:JST_XH_B8B-XH-AM_1x08_P2.50mm_Vertical -> Connector_JST:JST_XH_B9B-XH-AM_1x09_P2.50mm_Vertical; symbol Connector_Generic:Conn_01x08 -> Connector_Generic:Conn_01x09
- LCD1: symbol custom:0.96"-SSD1306-DISP-I2C -> ESP32-Water-Meter-Monitor-rescue:0.96"-SSD1306-DISP-I2C-custom
- U2: symbol custom:XL2001 -> ESP32-Water-Meter-Monitor-rescue:XL2001-custom
Connections:
- net +3V3: now also D14.2 (K), D15.2 (K), J7.2 (Pin_2)
- net +5V: now also J7.1 (Pin_1)
- net GND: now also J6.9 (Pin_9), D14.1 (A), D15.1 (A), J7.9 (Pin_9); no longer J6.8 (Pin_8)
- net at U1.12 (IO27): now also D11.3 (common), J7.3 (Pin_3)
- net at U1.23 (IO15): now also D15.3 (common), J7.4 (Pin_4)
- net at U1.26 (IO4): now also J6.3 (Pin_3), D14.3 (common); no longer D11.3 (common)
- net at D4.3 (common), U1.27 (IO16): now also J6.4 (Pin_4); no longer J6.3 (Pin_3)
- net at D10.3 (common), U1.28 (IO17): now also J6.5 (Pin_5), J7.5 (Pin_5); no longer J6.4 (Pin_4)
- net at D9.3 (common), U1.29 (IO5): now also J6.6 (Pin_6), J7.6 (Pin_6); no longer J6.5 (Pin_5)
- net at D6.3 (common), U1.30 (IO18): now also J6.7 (Pin_7), J7.7 (Pin_7); no longer J6.6 (Pin_6)
- net at D5.3 (common), U1.31 (IO19): now also J6.8 (Pin_8), J7.8 (Pin_8); no longer J6.7 (Pin_7)
- no-connect marks 17 -> 13
Other:
- moved on the sheet: D10, D11, D4, D5, D6, D9

Commit message: And ordered.
Parts:
- added R17, R18, R19, R20: 4.7K, Resistor_SMD:R_0603_1608Metric_Pad1.05x0.95mm_HandSolder, symbol Device:R_Small
Connections:
- net +3V3: now also R17.2, R18.2, R19.2, R20.2
- net at D11.3 (common), J7.3 (Pin_3), U1.12 (IO27): now also R19.1
- net at D15.3 (common), J7.4 (Pin_4), U1.23 (IO15): now also R20.1
- net at D14.3 (common), J6.3 (Pin_3), U1.26 (IO4): now also R17.1
- net at D4.3 (common), J6.4 (Pin_4), U1.27 (IO16): now also R18.1
Other:
- moved on the sheet: R6
Changed lines of the file:
@@
 Text Label 3950 2600 0    50   ~ 0
 RXD
-Text Label 2850 2950 0    50   ~ 0
+Text Label 2950 2950 0    50   ~ 0
 PROG
 $Comp
@@
 L Device:R_Small R6
 U 1 1 5F562790
-P 3150 2750
-F 0 "R6" V 2954 2750 50  0000 C CNN
-F 1 "4.7K" V 3045 2750 50  0000 C CNN
-F 2 "Resistor_SMD:R_0603_1608Metric_Pad1.05x0.95mm_HandSolder" H 3150 2750 50  0001 C CNN
-F 3 "~" H 3150 2750 50  0001 C CNN
-	1    3150 2750
+P 3250 2750
+F 0 "R6" V 3054 2750 50  0000 C CNN
+F 1 "4.7K" V 3145 2750 50  0000 C CNN
+F 2 "Resistor_SMD:R_0603_1608Metric_Pad1.05x0.95mm_HandSolder" H 3250 2750 50  0001 C CNN
+F 3 "~" H 3250 2750 50  0001 C CNN
+	1    3250 2750
 	-1   0    0    1
 $EndComp
@@
 L power:+3V3 #PWR022
 U 1 1 5F56334E
-P 3150 2500
-F 0 "#PWR022" H 3150 2350 50  0001 C CNN
-F 1 "+3V3" H 3165 2673 50  0000 C CNN
-F 2 "" H 3150 2500 50  0001 C CNN
-F 3 "" H 3150 2500 50  0001 C CNN
-	1    3150 2500
+P 3250 2500
+F 0 "#PWR022" H 3250 2350 50  0001 C CNN
+F 1 "+3V3" H 3265 2673 50  0000 C CNN
+F 2 "" H 3250 2500 50  0001 C CNN
+F 3 "" H 3250 2500 50  0001 C CNN
+	1    3250 2500
 	1    0    0    -1
 $EndComp
@@
 	2750 2950 3150 2950
 Wire Wire Line
-	3150 2950 3150 2850
-Wire Wire Line
-	3150 2650 3150 2500
+	3250 2950 3250 2850
+Wire Wire Line
+	3250 2650 3250 2500
 $Comp
 L Device:R_Small R4
@@
 Connection ~ 6250 5400
 Wire Wire Line
-	4700 7150 4900 7150
+	4700 7150 4800 7150
 Wire Wire Line
 	4700 5300 4700 7150
@@
 	3900 2600 4250 2600
 Wire Wire Line
-	3150 2950 4100 2950
+	3150 2950 3250 2950
 Wire Wire Line
 	4100 2950 4100 2800
@@
 	1000 2050 1000 2950
 Connection ~ 1000 2950
+Connection ~ 3250 2950
+Wire Wire Line
+	3250 2950 4100 2950
+$Comp
+L Device:R_Small R19
+U 1 1 5F57C9F7
+P 8550 5150
+F 0 "R19" V 8354 5150 50  0000 C CNN
+F 1 "4.7K" V 8445 5150 50  0000 C CNN
+F 2 "Resistor_SMD:R_0603_1608Metric_Pad1.05x0.95mm_HandSolder" H 8550 5150 50  0001 C CNN
+F 3 "~" H 8550 5150 50  0001 C CNN
+	1    8550 5150
+	-1   0    0    1
+$EndComp
+$Comp
+L Device:R_Small R20
+U 1 1 5F57E1AD
+P 9000 5150
+F 0 "R20" V 8804 5150 50  0000 C CNN
+F 1 "4.7K" V 8895 5150 50  0000 C CNN
+F 2 "Resistor_SMD:R_0603_1608Metric_Pad1.05x0.95mm_HandSolder" H 9000 5150 50  0001 C CNN
+F 3 "~" H 9000 5150 50  0001 C CNN
+	1    9000 5150
+	-1   0    0    1
+$EndComp
+$Comp
+L Device:R_Small R18
+U 1 1 5F57F0D1
+P 5250 6200
+F 0 "R18" V 5054 6200 50  0000 C CNN
+F 1 "4.7K" V 5145 6200 50  0000 C CNN
+F 2 "Resistor_SMD:R_0603_1608Metric_Pad1.05x0.95mm_HandSolder" H 5250 6200 50  0001 C CNN
+F 3 "~" H 5250 6200 50  0001 C CNN
+	1    5250 6200
+	-1   0    0    1
+$EndComp
+$Comp
+L Device:R_Small R17
+U 1 1 5F580116
+P 4800 6950
+F 0 "R17" V 4604 6950 50  0000 C CNN
+F 1 "4.7K" V 4695 6950 50  0000 C CNN
+F 2 "Resistor_SMD:R_0603_1608Metric_Pad1.05x0.95mm_HandSolder" H 4800 6950 50  0001 C CNN
+F 3 "~" H 4800 6950 50  0001 C CNN
+	1    4800 6950
+	-1   0    0    1
+$EndComp
+$Comp
+L power:+3V3 #PWR055
+U 1 1 5F5805C4
+P 4800 6800
+F 0 "#PWR055" H 4800 6650 50  0001 C CNN
+F 1 "+3V3" H 4815 6973 50  0000 C CNN
+F 2 "" H 4800 6800 50  0001 C CNN
+F 3 "" H 4800 6800 50  0001 C CNN
+	1    4800 6800
+	1    0    0    -1
+$EndComp
+Wire Wire Line
+	4800 6800 4800 6850
+Wire Wire Line
+	4800 7050 4800 7150
+Connection ~ 4800 7150
+Wire Wire Line
+	4800 7150 4900 7150
+$Comp
+L power:+3V3 #PWR056
+U 1 1 5F591BC9
+P 5250 6050
+F 0 "#PWR056" H 5250 5900 50  0001 C CNN
+F 1 "+3V3" H 5265 6223 50  0000 C CNN
+F 2 "" H 5250 6050 50  0001 C CNN
+F 3 "" H 5250 6050 50  0001 C CNN
+	1    5250 6050
+	1    0    0    -1
+$EndComp
+Wire Wire Line
+	5250 6050 5250 6100
+Wire Wire Line
+	5250 6300 5250 6350
+Connection ~ 5250 6350
+$Comp
+L power:+3V3 #PWR057
+U 1 1 5F5A36BF
+P 8550 5000
+F 0 "#PWR057" H 8550 4850 50  0001 C CNN
+F 1 "+3V3" H 8565 5173 50  0000 C CNN
+F 2 "" H 8550 5000 50  0001 C CNN
+F 3 "" H 8550 5000 50  0001 C CNN
+	1    8550 5000
+	1    0    0    -1
+$EndComp
+$Comp
+L power:+3V3 #PWR058
+U 1 1 5F5A3CA1
+P 9000 5000
+F 0 "#PWR058" H 9000 4850 50  0001 C CNN
+F 1 "+3V3" H 9015 5173 50  0000 C CNN
+F 2 "" H 9000 5000 50  0001 C CNN
+F 3 "" H 9000 5000 50  0001 C CNN
+	1    9000 5000
+	1    0    0    -1
+$EndComp
+Wire Wire Line
+	9000 5000 9000 5050
+Wire Wire Line
+	9000 5250 9000 5400
+Connection ~ 9000 5400
+Wire Wire Line
+	8550 5000 8550 5050
+Wire Wire Line
+	8550 5250 8550 5300
+Connection ~ 8550 5300
 $EndSCHEMATC

Commit message: Misc Bits.
Parts:
- C1, C10, C4, C7: symbol Device:CP1 -> ESP32-Water-Meter-Monitor-rescue:CP1-Device
- D10, D11, D14, D15, D2, D3, D4, D5, D6, D9: symbol Device:D_Schottky_x2_Serial_AKC -> ESP32-Water-Meter-Monitor-rescue:D_Schottky_x2_Serial_AKC-Device
- J1: footprint Connector_PinHeader_2.54mm:PinHeader_1x02_P2.54mm_Vertical -> Connector_JST:JST_XH_B2B-XH-AM_1x02_P2.50mm_Vertical
- LCD1: symbol ESP32-Water-Meter-Monitor-rescue:0.96"-SSD1306-DISP-I2C-custom -> ESP32-Water-Meter-Monitor-rescue:0.96"-SSD1306-DISP-I2C-custom-ESP32-Water-Meter-Monitor-rescue
- U2: symbol ESP32-Water-Meter-Monitor-rescue:XL2001-custom -> ESP32-Water-Meter-Monitor-rescue:XL2001-custom-ESP32-Water-Meter-Monitor-rescue
Changed lines of the file:
@@
 	1650 950  1850 950
 $Comp
-L Device:CP1 C7
+L ESP32-Water-Meter-Monitor-rescue:CP1-Device C7
 U 1 1 5F5C3C2C
 P 1850 1150
@@
 $EndComp
 $Comp
-L ESP32-Water-Meter-Monitor-rescue:XL2001-custom U2
+L ESP32-Water-Meter-Monitor-rescue:XL2001-custom-ESP32-Water-Meter-Monitor-rescue U2
 U 1 1 5F554CA0
 P 3750 950
@@
 	2300 1000 2300 950
 $Comp
-L Device:CP1 C4
+L ESP32-Water-Meter-Monitor-rescue:CP1-Device C4
 U 1 1 5F541A1E
 P 5900 1150
@@
 $EndComp
 $Comp
-L Device:CP1 C1
+L ESP32-Water-Meter-Monitor-rescue:CP1-Device C1
 U 1 1 5F5409F2
 P 2300 1150
@@
 F 0 "J1" H 618 1025 50  0000 C CNN
 F 1 "Conn_01x02" H 618 1116 50  0001 C CNN
-F 2 "Connector_PinHeader_2.54mm:PinHeader_1x02_P2.54mm_Vertical" H 700 1350 50  0001 C CNN
+F 2 "Connector_JST:JST_XH_B2B-XH-AM_1x02_P2.50mm_Vertical" H 700 1350 50  0001 C CNN
 F 3 "~" H 700 1350 50  0001 C CNN
 	1    700  1350
@@
 $EndComp
 $Comp
-L Device:CP1 C10
+L ESP32-Water-Meter-Monitor-rescue:CP1-Device C10
 U 1 1 5F5AA457
 P 2450 2450
@@
 	8550 4050 8950 4050
 $Comp
-L ESP32-Water-Meter-Monitor-rescue:0.96"-SSD1306-DISP-I2C-custom LCD1
+L ESP32-Water-Meter-Monitor-rescue:0.96"-SSD1306-DISP-I2C-custom-ESP32-Water-Meter-Monitor-rescue LCD1
 U 1 1 5F67CC7A
 P 7650 2550
@@
 Connection ~ 8550 4150
 $Comp
-L Device:D_Schottky_x2_Serial_AKC D3
+L ESP32-Water-Meter-Monitor-rescue:D_Schottky_x2_Serial_AKC-Device D3
 U 1 1 5F7001C7
 P 10350 4050
@@
 $EndComp
 $Comp
-L Device:D_Schottky_x2_Serial_AKC D2
+L ESP32-Water-Meter-Monitor-rescue:D_Schottky_x2_Serial_AKC-Device D2
 U 1 1 5F7083BC
 P 10050 4500
@@
 	5200 4250 6650 4250
 $Comp
-L Device:D_Schottky_x2_Serial_AKC D4
+L ESP32-Water-Meter-Monitor-rescue:D_Schottky_x2_Serial_AKC-Device D4
 U 1 1 5FB0D1DF
 P 5500 6850
@@
 $EndComp
 $Comp
-L Device:D_Schottky_x2_Serial_AKC D11
+L ESP32-Water-Meter-Monitor-rescue:D_Schottky_x2_Serial_AKC-Device D11
 U 1 1 5FAF3874
 P 8750 6150
@@
 $EndComp
 $Comp
-L Device:D_Schottky_x2_Serial_AKC D10
+L ESP32-Water-Meter-Monitor-rescue:D_Schottky_x2_Serial_AKC-Device D10
 U 1 1 5FA97C30
 P 8350 6150
@@
 $EndComp
 $Comp
-L Device:D_Schottky_x2_Serial_AKC D9
+L ESP32-Water-Meter-Monitor-rescue:D_Schottky_x2_Serial_AKC-Device D9
 U 1 1 5FA97743
 P 7950 6150
@@
 $EndComp
 $Comp
-L Device:D_Schottky_x2_Serial_AKC D6
+L ESP32-Water-Meter-Monitor-rescue:D_Schottky_x2_Serial_AKC-Device D6
 U 1 1 5FA96DAB
 P 7550 6150
@@
 $EndComp
 $Comp
-L Device:D_Schottky_x2_Serial_AKC D5
+L ESP32-Water-Meter-Monitor-rescue:D_Schottky_x2_Serial_AKC-Device D5
 U 1 1 5FA95DD8
 P 7150 6150
@@
 Connection ~ 4900 3950
 $Comp
-L Device:D_Schottky_x2_Serial_AKC D15
+L ESP32-Water-Meter-Monitor-rescue:D_Schottky_x2_Serial_AKC-Device D15
 U 1 1 5F6D6FF1
 P 9200 6150
@@
 $EndComp
 $Comp
-L Device:D_Schottky_x2_Serial_AKC D14
+L ESP32-Water-Meter-Monitor-rescue:D_Schottky_x2_Serial_AKC-Device D14
 U 1 1 5F6E7F2B
 P 5100 7150
