File: ESP/ESP32 Water Meter Monitor/USB Interface.sch (KiCad schematic (older format))
At the start: 12 parts, among them J2 USB_B_Micro, Q1 BC817, Q2 BC817, U4 CH340C

Commit message: Misc Bits.
Parts:
- J2: symbol Connector:USB_B_Micro -> ESP32-Water-Meter-Monitor-rescue:USB_B_Micro-Connector
Changed lines of the file:
@@
 	6550 5750 7100 5750
 $Comp
-L Connector:USB_B_Micro J2
+L ESP32-Water-Meter-Monitor-rescue:USB_B_Micro-Connector J2
 U 1 1 5F844DA0
 P 1750 4450
+AR Path="/5F844DA0" Ref="J2"  Part="1"
+AR Path="/5F7DDE6B/5F844DA0" Ref="J2"  Part="1"
 F 0 "J2" H 1807 4917 50  0000 C CNN
 F 1 "USB_B_Micro" H 1807 4826 50  0000 C CNN
