File: ESP/ESP32 Water Meter Monitor R2/ESP32 Water Meter Monitor R2.sch (KiCad schematic (older format))
At the start: 63 parts, among them J1 Conn_01x02, J11 Conn_01x05, J3 Conn_01x01, J4 Conn_01x01, J5 Conn_01x05, J6 Conn_01x09, J7 Conn_01x09, SW1 SW_Push, SW2 SW_Push, U1 ESP32-WROOM-32D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

Commit message: Misc Bits.
Parts:
- removed D13: LED, custom:CHIPLED_0603, symbol Device:LED
- removed J3, J4: Conn_01x01, Connector_Pin:Pin_D1.3mm_L11.0mm, symbol Connector_Generic:Conn_01x01
- removed R11: 470R, Resistor_SMD:R_0603_1608Metric, symbol Device:R_Small
- added D18: BAT54S, Package_TO_SOT_SMD:SOT-23, symbol Device:D_Schottky_x2_Serial_AKC
- added J10, J9: Conn_01x05, Connector_JST:JST_XH_B3B-XH-AM_1x03_P2.50mm_Vertical, symbol Connector_Generic:Conn_01x03
- added J8: Conn_01x05, Connector_JST:JST_XH_B4B-XH-AM_1x04_P2.50mm_Vertical, symbol Connector_Generic:Conn_01x04
- J1: footprint Connector_PinHeader_2.54mm:PinHeader_1x02_P2.54mm_Vertical -> Connector_JST:JST_XH_B2B-XH-AM_1x02_P2.50mm_Vertical
Connections:
- net +3V3: now also D18.2 (K), J10.1 (Pin_1), J8.1 (Pin_1), J9.1 (Pin_1)
- net GND: now also D18.1 (A), J10.3 (Pin_3), J8.4 (Pin_4), J9.3 (Pin_3)
- net SCL_LOC: now also J8.2 (Pin_2)
- net SDA_LOC: now also J8.3 (Pin_3)
- net at U1.16 (IO13): now also D18.3 (common), J10.2 (Pin_2), J9.2 (Pin_2)
Other:
- moved on the sheet: H1, H2, H3, H4
