File: ESP/ESP32 Weather Particulate Counter/ESP32 Weather Particulate Counter.kicad_pcb (KiCad board)
At the start: 4 copper layers, 50 x 60 mm, 75 parts, among them J1 Conn_01x02, J10 WIND, J11 Conn_01x05, J2 Conn_01x05, J3 Conn_01x01, J4 Conn_01x01, J5 Conn_01x08, J6 Conn_01x08, J7 Conn_01x04, J8 Conn_01x04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

Commit message: Blerp.
Other:
- net class Default removed
