File: ESP/ESP32 Weather Particulate Counter - R2/ESP32 Weather Particulate Counter-r2.sch (KiCad schematic (older format))
At the start: 75 parts, among them J1 Conn_01x02, J10 WIND, J11 Conn_01x05, J2 Conn_01x05, J3 Conn_01x01, J4 Conn_01x01, J5 Conn_01x08, J6 Conn_01x08, J7 Conn_01x04, J8 Conn_01x04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

Commit message: Blerp.
Connections:
- net +5V: now also J5.8 (Pin_8), J6.8 (Pin_8); no longer J5.1 (Pin_1), J6.1 (Pin_1)
- net GND: now also J5.7 (Pin_7), J6.7 (Pin_7); no longer J5.2 (Pin_2), J6.2 (Pin_2)
- net PT_RESET: now also J5.3 (Pin_3), J6.3 (Pin_3); no longer J5.6 (Pin_6), J6.6 (Pin_6)
- net PT_SET: now also J5.6 (Pin_6), J6.6 (Pin_6); no longer J5.3 (Pin_3), J6.3 (Pin_3)
- net at D6.3 (common), J8.3 (Pin_3), R19.1: now also U1.11 (IO26); no longer U1.14 (IO12)
- net at D5.3 (common), J7.3 (Pin_3), R18.1: now also U1.12 (IO27); no longer U1.16 (IO13)
- net at U1.6 (IO34): now also D3.3 (common), R23.1
- net at U1.7 (IO35): now also D4.3 (common), R24.1
- net at J5.4 (Pin_4): now also R11.1; no longer R9.1
- net at J5.5 (Pin_5): now also R9.1; no longer R11.1
- net at J6.4 (Pin_4): now also R10.1; no longer R8.1
- net at J6.5 (Pin_5): now also R8.1; no longer R10.1
- net RAIN_GAUGE: no longer names the net of D2.3 (common), R20.1, U1.10 (IO25)
- removed net WIND_DIR: D3.3 (common), R23.1, U1.11 (IO26), U1.8 (IO32)
- removed net WIND_PULSE: D4.3 (common), R24.1, U1.12 (IO27)
- no-connect marks 27 -> 25
Other:
- note removed: "J5, J6 are backwards!\nPlantower numbers the connecor \nin their modules in reverse from the \nconnector manufacturer!\nEither place connectors backwards, or \nrewire cable to be crossover."
- note removed: "R19 breaks boot (it switches the \nflash to 1.8V mode by pulling GPIO12 \nhigh at boot).\nRemove R19 and do not use J8"
Changed lines of the file:
@@
 Text Label 3000 5550 0    50   ~ 0
 PROG
-$Comp
-L RF_Module:ESP32-WROOM-32D U1
-U 1 1 5F547F90
-P 2150 4150
-F 0 "U1" H 2350 5550 50  0000 C CNN
-F 1 "ESP32-WROOM-32D" H 1600 2750 50  0000 C CNN
-F 2 "RF_Module:ESP32-WROOM-32" H 2150 2650 50  0001 C CNN
-F 3 "https://www.espressif.com/sites/default/files/documentation/esp32-wroom-32d_esp32-wroom-32u_datasheet_en.pdf" H 1850 4200 50  0001 C CNN
-	1    2150 4150
-	1    0    0    -1
-$EndComp
 Wire Wire Line
 	2150 5800 2150 5550
@@
 NoConn ~ 4900 2700
 $Comp
-L Connector_Generic:Conn_01x08 J5
-U 1 1 5F66642C
-P 6400 3850
-F 0 "J5" H 6480 3796 50  0000 L CNN
-F 1 "Conn_01x08" H 6480 3751 50  0001 L CNN
-F 2 "Connector_Molex:Molex_PicoBlade_53047-0810_1x08_P1.25mm_Vertical" H 6480 3705 50  0001 L CNN
-F 3 "~" H 6400 3850 50  0001 C CNN
-	1    6400 3850
-	1    0    0    -1
-$EndComp
-$Comp
 L power:+5V #PWR06
 U 1 1 5F6683F6
@@
 L Connector_Generic:Conn_01x08 J6
 U 1 1 5F67C133
-P 7250 3850
-F 0 "J6" H 7330 3796 50  0000 L CNN
-F 1 "Conn_01x08" H 7330 3751 50  0001 L CNN
-F 2 "Connector_Molex:Molex_PicoBlade_53047-0810_1x08_P1.25mm_Vertical" H 7330 3705 50  0001 L CNN
-F 3 "~" H 7250 3850 50  0001 C CNN
-	1    7250 3850
-	1    0    0    -1
+P 7250 3950
+F 0 "J6" H 7330 3896 50  0000 L CNN
+F 1 "Conn_01x08" H 7330 3851 50  0001 L CNN
+F 2 "Connector_Molex:Molex_PicoBlade_53047-0810_1x08_P1.25mm_Vertical" H 7330 3805 50  0001 L CNN
+F 3 "~" H 7250 3950 50  0001 C CNN
+	1    7250 3950
+	1    0    0    1
 $EndComp
 Wire Wire Line
@@
 NoConn ~ 7050 4150
 Wire Wire Line
-	7050 4050 6200 4050
+	7050 4050 6600 4050
 Connection ~ 6200 4050
 Wire Wire Line
 	6200 4050 6050 4050
 Wire Wire Line
-	7050 3750 6200 3750
+	7050 3750 6600 3750
 Connection ~ 6200 3750
 Wire Wire Line
@@
 Connection ~ 8400 5500
 Wire Wire Line
-	2750 3550 3450 3550
-Wire Wire Line
 	9500 5650 9600 5650
 Connection ~ 9600 5650
@@
 Wire Wire Line
 	2750 4350 3650 4350
-Wire Wire Line
-	2750 3650 3350 3650
-Wire Wire Line
-	3350 3650 3350 5050
 Wire Wire Line
 	9600 5400 9850 5400
@@
 	5700 5950 5700 6400
 Wire Wire Line
-	3250 5150 5800 5150
-Wire Wire Line
 	5800 5150 5800 5850
 Connection ~ 5800 5850
@@
 Wire Wire Line
 	5700 5950 5700 5250
-Wire Wire Line
-	5700 5250 3150 5250
 Connection ~ 5700 5950
 Wire Wire Line
@@
 	3900 6700 3950 6700
 Wire Wire Line
-	3450 3550 3450 4950
-Wire Wire Line
 	3950 3900 3950 4450
 Connection ~ 3950 4450
@@
 	2750 4450 3950 4450
 Wire Wire Line
-	2750 4850 3150 4850
-Wire Wire Line
-	3150 4850 3150 5250
-Wire Wire Line
 	3050 4650 2750 4650
 Wire Wire Line
 	3050 4650 3050 5350
-Wire Wire Line
-	2750 4750 3250 4750
-Wire Wire Line
-	3250 4750 3250 4950
 $Comp
 L Device:D_Schottky_x2_Serial_AKC D5
@@
 NoConn ~ 4250 6900
 NoConn ~ 4250 7000
-NoConn ~ 2750 5250
-NoConn ~ 2750 5150
 NoConn ~ 2750 5050
 NoConn ~ 2750 4950
@@
 NoConn ~ 1550 3250
 NoConn ~ 8300 3050
-Text Notes 5650 3150 0    50   ~ 0
-J5, J6 are backwards!\nPlantower numbers the connecor \nin their modules in reverse from the \nconnector manufacturer!\nEither place connectors backwards, or \nrewire cable to be crossover.
-Text Notes 7800 4800 0    50   ~ 0
-R19 breaks boot (it switches the \nflash to 1.8V mode by pulling GPIO12 \nhigh at boot).\nRemove R19 and do not use J8
-Text Label 3500 5350 0    50   ~ 0
-RAIN_GAUGE
-Text Label 3500 5150 0    50   ~ 0
-WIND_DIR
-Text Label 3500 5250 0    50   ~ 0
-WIND_PULSE
-Wire Wire Line
-	2750 4950 3250 4950
-Connection ~ 3250 4950
-Wire Wire Line
-	3250 4950 3250 5150
+$Comp
+L RF_Module:ESP32-WROOM-32D U1
+U 1 1 5F547F90
+P 2150 4150
+F 0 "U1" H 2350 5550 50  0000 C CNN
+F 1 "ESP32-WROOM-32D" H 1600 2750 50  0000 C CNN
+F 2 "RF_Module:ESP32-WROOM-32" H 2150 2650 50  0001 C CNN
+F 3 "https://www.espressif.com/sites/default/files/documentation/esp32-wroom-32d_esp32-wroom-32u_datasheet_en.pdf" H 1850 4200 50  0001 C CNN
+	1    2150 4150
+	1    0    0    -1
+$EndComp
+Wire Wire Line
+	2750 5250 5700 5250
+Wire Wire Line
+	2750 5150 5800 5150
+Wire Wire Line
+	2750 4750 3450 4750
+Wire Wire Line
+	3450 4750 3450 4950
+Wire Wire Line
+	2750 4850 3350 4850
+Wire Wire Line
+	3350 4850 3350 5050
+Connection ~ 6600 4050
+Wire Wire Line
+	6600 4050 6200 4050
+Connection ~ 6600 3750
+Wire Wire Line
+	6600 3750 6200 3750
+$Comp
+L Connector_Generic:Conn_01x08 J5
+U 1 1 5F66642C
+P 6400 3950
+F 0 "J5" H 6480 3896 50  0000 L CNN
+F 1 "Conn_01x08" H 6480 3851 50  0001 L CNN
+F 2 "Connector_Molex:Molex_PicoBlade_53047-0810_1x08_P1.25mm_Vertical" H 6480 3805 50  0001 L CNN
+F 3 "~" H 6400 3950 50  0001 C CNN
+	1    6400 3950
+	1    0    0    1
+$EndComp
 $EndSCHEMATC
