File: ESP/Air Quality Sensor - R1/Air Quality Sensor - R1/Sensors.kicad_sch (KiCad schematic)
At the start: 27 parts, among them U1 CCS811, U2 SGP40, U3 SCD4X, U4 Sensair_Sunrise_006-0-0007, U5 BME680, U6 MICS-VZ-89TE‎, U7 SCD30

Commit message: Pile of uncommitted boards.
Parts:
- added C11: 0.1u, Capacitor_SMD:C_0603_1608Metric, symbol Device:C_Small
Connections:
- net +3V3: now also C11.1
- net GND: now also C11.2
- net SCL renamed SCL_1
- net SCL_1: no longer U1.10 (SCL), U2.6 (SCL), U6.2 (SCL)
- net SDA renamed SDA_1
- net SDA_1: no longer U1.9 (SDA), U2.3 (SDA), U6.4 (SDA)
- new net SCL_2: U1.10 (SCL), U2.6 (SCL), U6.2 (SCL)
- new net SDA_2: U1.9 (SDA), U2.3 (SDA), U6.4 (SDA)
Other:
- note added: "These devices all have heaters"
- note added: "These devices don't self-heat"
- moved on the sheet: C1, C10, C2, C3, C4, C5, C6, C7, C9, R1, R2, R3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
