File: ESP/Air Quality Sensor - R1/Air Quality Sensor - R1/Air Quality Sensor - R1.kicad_sch (KiCad schematic)
At the start: 0 parts

Commit message: Pile of uncommitted boards.
Parts:
- added D1: LED, custom:CHIPLED_0603, symbol Device:LED
- added H1, H2, H3, H4: MountingHole, MountingHole:MountingHole_3.2mm_M3_Pad_Via, symbol Mechanical:MountingHole
- added J1: Conn_01x05, Connector_JST:JST_XH_B3B-XH-AM_1x03_P2.50mm_Vertical, symbol Connector_Generic:Conn_01x03
- added J2: Conn_01x09, Connector_JST:JST_XH_B9B-XH-AM_1x09_P2.50mm_Vertical, symbol Connector_Generic:Conn_01x09
- added J3: Conn_01x05, Connector_JST:JST_XH_B5B-XH-AM_1x05_P2.50mm_Vertical, symbol Connector_Generic:Conn_01x05
- added J4: Conn_01x04, Connector_JST:JST_XH_B4B-XH-AM_1x04_P2.50mm_Vertical, symbol Connector_Generic:Conn_01x04
- added R10, R11, R13, R6, R7, R8, R9: 4.7K, Resistor_SMD:R_0603_1608Metric, symbol Device:R_Small
- added R12, R14: 470R, Resistor_SMD:R_0603_1608Metric, symbol Device:R_Small
- added TP10, TP6, TP7, TP8, TP9: TestPoint_Small, Connector_Pin:Pin_D1.0mm_L10.0mm, symbol Connector:TestPoint_Small
- added U8: ESP32-POE, custom:ESP32-POE, symbol custom:ESP32-POE
Connections:
- new net: J2.7 (Pin_7), R14.2, U8.18 (GPIO15/HS2_CMD)
- new net: J1.2 (Pin_2), J2.8 (Pin_8), U8.19 (GPIO14/HS2_CLK)
- new net: J4.2 (Pin_2), R13.1, U8.13 (GPIO35)
- new net: D1.2 (A), R12.1
- new net: J3.4 (Pin_4), R11.1, U8.10 (GPIO5/SPI_CS)
- new net: R12.2, U8.7 (GPIO2/HS2_DATA0)
- new net: J3.3 (Pin_3), R10.1, U8.9 (GPIO4/U1TXD)
- new net: J4.3 (Pin_3), R14.1
- new net +3V3: J1.1 (Pin_1), J2.2 (Pin_2), J3.2 (Pin_2), R10.2, R11.2, R13.2, R6.2, R7.2, R8.2, R9.2, U8.2 (3.3V)
- new net +5V: J2.1 (Pin_1), J3.1 (Pin_1), J4.1 (Pin_1), U8.1 (5V)
- new net GND: D1.1 (K), J1.3 (Pin_3), J2.9 (Pin_9), J3.5 (Pin_5), J4.4 (Pin_4), TP10.1, U8.3 (GND)
- new net SENS/SCL_1: J2.6 (Pin_6), R8.1, TP6.1, U8.15 (GPIO33)
- new net SENS/SCL_2: J2.4 (Pin_4), R6.1, TP8.1, U8.17 (GPIO16/I2C-SCL)
- new net SENS/SDA_1: J2.5 (Pin_5), R9.1, TP7.1, U8.16 (GPIO32)
- new net SENS/SDA_2: J2.3 (Pin_3), R7.1, TP9.1, U8.20 (GPIO13/I2C-SDA)
Other:
- sheet SENS ports: added SCL_1, SCL_2, SDA_1, SDA_2; removed SCL, SDA
- note added: "1-Wire Temp Sensors"
- note added: "4-Wire PWM fan"
- note added: "Debug"
- note added: "Ext I2C display (?)"

Commit message: Reworking things to use the new controller PCB.
Parts:
- removed J3: Conn_01x05, Connector_JST:JST_XH_B5B-XH-AM_1x05_P2.50mm_Vertical, symbol Connector_Generic:Conn_01x05
- removed R10, R11: 4.7K, Resistor_SMD:R_0603_1608Metric, symbol Device:R_Small
- removed TP6, TP7, TP8, TP9: TestPoint_Small, Connector_Pin:Pin_D1.0mm_L10.0mm, symbol Connector:TestPoint_Small
- removed U8: ESP32-POE, custom:ESP32-POE, symbol custom:ESP32-POE
- added J3: ESP32-DevBoard-Header, Connector_PinHeader_2.54mm:PinHeader_2x20_P2.54mm_Vertical, symbol connectors:ESP32-DevBoard-Header
Connections:
- net +3V3: now also J3.3 (3V3), J3.33 (3V3), J3.34 (3V3), J3.4 (3V3)
- net +5V: now also J3.35 (5V0), J3.36 (5V0)
- net GND: now also J3.1 (GND), J3.2 (GND), J3.31 (GND), J3.32 (GND), J3.39 (GND), J3.40 (GND), J3.5 (GND), J3.6 (GND)
- net SENS/SCL_1: now also J3.20 (IO22)
- net SENS/SCL_2: now also R7.1, J3.11 (IO32); no longer R6.1
- net SENS/SDA_1: now also J3.23 (IO21)
- net SENS/SDA_2: now also R6.1, J3.12 (IO33); no longer R7.1
- net at J2.7 (Pin_7), R14.2: now also J3.30 (IO15)
- net at J1.2 (Pin_2), J2.8 (Pin_8): now also J3.26 (IO5)
- net at J4.2 (Pin_2), R13.1: now also J3.18 (IO13)
- net at R12.2: now also J3.16 (IO14)
Other:
- moved on the sheet: D1, H1, H2, H3, H4, R12, R14, R6, R7, TP10

Commit message: Projects Projects Projects Projects.
Parts:
- added J5: Conn_01x09, Connector_Molex:Molex_PicoBlade_53047-0710_1x07_P1.25mm_Vertical, symbol Connector_Generic:Conn_01x07
- added R10, R11: 4.7K, Resistor_SMD:R_0603_1608Metric, symbol Device:R_Small
- J1: footprint Connector_JST:JST_XH_B3B-XH-AM_1x03_P2.50mm_Vertical -> Connector_JST:JST_XH_B3B-XH-A_1x03_P2.50mm_Vertical
- J2: footprint Connector_JST:JST_XH_B9B-XH-AM_1x09_P2.50mm_Vertical -> Connector_JST:JST_XH_B9B-XH-A_1x09_P2.50mm_Vertical
- J4: footprint Connector_JST:JST_XH_B4B-XH-AM_1x04_P2.50mm_Vertical -> Connector_JST:JST_XH_B4B-XH-A_1x04_P2.50mm_Vertical
Connections:
- net +5V: now also J5.4 (Pin_4)
- net GND: now also J5.3 (Pin_3)
- net at J1.2 (Pin_2), J2.8 (Pin_8): now also J3.24 (IO19); no longer J3.26 (IO5)
- net at J3.25 (IO18): now also R10.2
- net at J3.27 (IO4): now also R11.2
- new net: J5.5 (Pin_5), R10.1
- new net: J5.6 (Pin_6), R11.1

Commit message: Blerp.
Parts:
- added J6: Conn_01x08, Connector_Molex:Molex_PicoBlade_53047-0910_1x09_P1.25mm_Vertical, symbol Connector_Generic:Conn_01x09
Connections:
- net +3V3: now also J6.2 (Pin_2)
- net +5V: now also J6.1 (Pin_1)
- net GND: now also J6.9 (Pin_9)
- net at J3.13 (IO25): now also J6.7 (Pin_7)
- net at J3.14 (IO26): now also J6.8 (Pin_8)
- net at J3.15 (IO27): now also J6.6 (Pin_6)
- net at J3.17 (IO12): now also J6.5 (Pin_5)
- net at J3.19 (IO23): now also J6.4 (Pin_4)
- net at J3.26 (IO5): now also J6.3 (Pin_3)
Changed lines of the file:
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@@
+    (stroke (width 0) (type default) (color 0 0 0 0))
+  )
+  (wire (pts (xy 60.96 158.75) (xy 73.66 158.75))
     (stroke (width 0) (type default) (color 0 0 0 0))
   )
@@
     (stroke (width 0) (type default) (color 0 0 0 0))
   )
+  (wire (pts (xy 71.12 161.29) (xy 73.66 161.29))
+    (stroke (width 0) (type default) (color 0 0 0 0))
+  )
   (wire (pts (xy 148.59 144.78) (xy 151.13 144.78))
     (stroke (width 0) (type default) (color 0 0 0 0))
@@
     (stroke (width 0) (type default) (color 0 0 0 0))
   )
+  (wire (pts (xy 15.24 151.13) (xy 15.24 69.85))
+    (stroke (width 0) (type default) (color 0 0 0 0))
+  )
   (wire (pts (xy 148.59 142.24) (xy 148.59 144.78))
     (stroke (width 0) (type default) (color 0 0 0 0))
@@
     (stroke (width 0) (type default) (color 0 0 0 0))
   )
+  (wire (pts (xy 25.4 72.39) (xy 13.97 72.39))
+    (stroke (width 0) (type default) (color 0 0 0 0))
+  )
   (wire (pts (xy 148.59 111.76) (xy 127 111.76))
     (stroke (width 0) (type default) (color 0 0 0 0))
@@
     (stroke (width 0) (type default) (color 0 0 0 0))
   )
+  (wire (pts (xy 60.96 64.77) (xy 60.96 158.75))
+    (stroke (width 0) (type default) (color 0 0 0 0))
+  )
   (wire (pts (xy 127 76.2) (xy 127 111.76))
     (stroke (width 0) (type default) (color 0 0 0 0))
@@
     (stroke (width 0) (type default) (color 0 0 0 0))
   )
+  (wire (pts (xy 59.69 80.01) (xy 59.69 146.05))
+    (stroke (width 0) (type default) (color 0 0 0 0))
+  )
+  (wire (pts (xy 25.4 67.31) (xy 17.78 67.31))
+    (stroke (width 0) (type default) (color 0 0 0 0))
+  )
   (wire (pts (xy 146.05 121.92) (xy 146.05 124.46))
     (stroke (width 0) (type default) (color 0 0 0 0))
@@
     (stroke (width 0) (type default) (color 0 0 0 0))
   )
+  (wire (pts (xy 15.24 69.85) (xy 25.4 69.85))
+    (stroke (width 0) (type default) (color 0 0 0 0))
+  )
+  (wire (pts (xy 17.78 153.67) (xy 73.66 153.67))
+    (stroke (width 0) (type default) (color 0 0 0 0))
+  )
   (wire (pts (xy 166.37 45.72) (xy 166.37 46.99))
     (stroke (width 0) (type default) (color 0 0 0 0))
@@
     (stroke (width 0) (type default) (color 0 0 0 0))
   )
+  (wire (pts (xy 71.12 140.97) (xy 73.66 140.97))
+    (stroke (width 0) (type default) (color 0 0 0 0))
+  )
   (wire (pts (xy 137.16 104.14) (xy 137.16 99.06))
     (stroke (width 0) (type default) (color 0 0 0 0))
@@
     (stroke (width 0) (type default) (color 0 0 0 0))
   )
+  (wire (pts (xy 25.4 64.77) (xy 19.05 64.77))
+    (stroke (width 0) (type default) (color 0 0 0 0))
+  )
+  (wire (pts (xy 19.05 156.21) (xy 73.66 156.21))
+    (stroke (width 0) (type default) (color 0 0 0 0))
+  )
   (wire (pts (xy 132.08 85.09) (xy 132.08 106.68))
     (stroke (width 0) (type default) (color 0 0 0 0))
@@
     (stroke (width 0) (type default) (color 0 0 0 0))
   )
+  (wire (pts (xy 13.97 72.39) (xy 13.97 148.59))
+    (stroke (width 0) (type default) (color 0 0 0 0))
+  )
   (wire (pts (xy 22.86 54.61) (xy 25.4 54.61))
     (stroke (width 0) (type default) (color 0 0 0 0))
   )
+  (wire (pts (xy 53.34 64.77) (xy 60.96 64.77))
+    (stroke (width 0) (type default) (color 0 0 0 0))
+  )
   (wire (pts (xy 53.34 49.53) (xy 55.88 49.53))
     (stroke (width 0) (type default) (color 0 0 0 0))
@@
     (stroke (width 0) (type default) (color 0 0 0 0))
   )
+  (wire (pts (xy 19.05 64.77) (xy 19.05 156.21))
+    (stroke (width 0) (type default) (color 0 0 0 0))
+  )
+  (wire (pts (xy 73.66 146.05) (xy 59.69 146.05))
+    (stroke (width 0) (type default) (color 0 0 0 0))
+  )
   (wire (pts (xy 166.37 52.07) (xy 166.37 69.85))
     (stroke (width 0) (type default) (color 0 0 0 0))
@@
     (stroke (width 0) (type default) (color 0 0 0 0))
   )
+  (wire (pts (xy 17.78 67.31) (xy 17.78 153.67))
+    (stroke (width 0) (type default) (color 0 0 0 0))
+  )
   (wire (pts (xy 77.47 107.95) (xy 87.63 107.95))
     (stroke (width 0) (type default) (color 0 0 0 0))
@@
     (stroke (width 0) (type default) (color 0 0 0 0))
   )
+  (wire (pts (xy 71.12 163.83) (xy 71.12 161.29))
+    (stroke (width 0) (type default) (color 0 0 0 0))
+  )
+  (wire (pts (xy 71.12 138.43) (xy 71.12 140.97))
+    (stroke (width 0) (type default) (color 0 0 0 0))
+  )
   (wire (pts (xy 139.7 58.42) (xy 180.34 58.42))
     (stroke (width 0) (type default) (color 0 0 0 0))
@@
     (stroke (width 0) (type default) (color 0 0 0 0))
   )
+  (wire (pts (xy 15.24 151.13) (xy 73.66 151.13))
+    (stroke (width 0) (type default) (color 0 0 0 0))
+  )
   (wire (pts (xy 53.34 97.79) (xy 55.88 97.79))
     (stroke (width 0) (type default) (color 0 0 0 0))
@@
     (stroke (width 0) (type default) (color 0 0 0 0))
   )
+  (wire (pts (xy 53.34 80.01) (xy 59.69 80.01))
+    (stroke (width 0) (type default) (color 0 0 0 0))
+  )
   (wire (pts (xy 148.59 114.3) (xy 124.46 114.3))
     (stroke (width 0) (type default) (color 0 0 0 0))
@@
     (stroke (width 0) (type default) (color 0 0 0 0))
   )
+  (wire (pts (xy 64.77 143.51) (xy 73.66 143.51))
+    (stroke (width 0) (type default) (color 0 0 0 0))
+  )
   (wire (pts (xy 53.34 85.09) (xy 67.31 85.09))
     (stroke (width 0) (type default) (color 0 0 0 0))
@@
     (stroke (width 0) (type default) (color 0 0 0 0))
   )
+  (wire (pts (xy 13.97 148.59) (xy 73.66 148.59))
+    (stroke (width 0) (type default) (color 0 0 0 0))
+  )
   (wire (pts (xy 109.22 135.89) (xy 109.22 137.16))
     (stroke (width 0) (type default) (color 0 0 0 0))
@@
     (stroke (width 0) (type default) (color 0 0 0 0))
   )
+  (wire (pts (xy 64.77 138.43) (xy 64.77 143.51))
+    (stroke (width 0) (type default) (color 0 0 0 0))
+  )
   (wire (pts (xy 148.59 121.92) (xy 146.05 121.92))
     (stroke (width 0) (type default) (color 0 0 0 0))
@@
     (stroke (width 0) (type default) (color 0 0 0 0))
   )
-  (text "Ext I2C display (?)" (at 58.42 143.51 0)
+  (text "Ext I2C display (?)" (at 120.65 134.62 0)
     (effects (font (size 1.27 1.27)) (justify left bottom))
   )
@@
     )
     (property "Datasheet" "" (id 3) (at 166.37 45.72 0)
+      (effects (font (size 1.27 1.27)) hide)
+    )
+    (pin "1")
+  )
+  (symbol (lib_id "power:+5V") (at 71.12 138.43 0) (unit 1)
+    (in_bom yes) (on_board yes)
+    (property "Reference" "#PWR043" (id 0) (at 71.12 142.24 0)
+      (effects (font (size 1.27 1.27)) hide)
+    )
+    (property "Value" "+5V" (id 1) (at 69.85 134.62 0))
+    (property "Footprint" "" (id 2) (at 71.12 138.43 0)
+      (effects (font (size 1.27 1.27)) hide)
+    )
+    (property "Datasheet" "" (id 3) (at 71.12 138.43 0)
       (effects (font (size 1.27 1.27)) hide)
     )
@@
     (pin "2")
   )
+  (symbol (lib_id "power:GND") (at 71.12 163.83 0) (unit 1)
+    (in_bom yes) (on_board yes)
+    (property "Reference" "#PWR045" (id 0) (at 71.12 170.18 0)
+      (effects (font (size 1.27 1.27)) hide)
+    )
+    (property "Value" "GND" (id 1) (at 71.247 168.2242 0))
+    (property "Footprint" "" (id 2) (at 71.12 163.83 0)
+      (effects (font (size 1.27 1.27)) hide)
+    )
+    (property "Datasheet" "" (id 3) (at 71.12 163.83 0)
+      (effects (font (size 1.27 1.27)) hide)
+    )
+    (pin "1")
+  )
   (symbol (lib_id "power:GND") (at 96.52 170.18 0) (unit 1)
     (in_bom yes) (on_board yes)
@@
     (pin "1")
     (pin "2")
+  )
+  (symbol (lib_id "power:+3V3") (at 64.77 138.43 0) (unit 1)
+    (in_bom yes) (on_board yes)
+    (property "Reference" "#PWR042" (id 0) (at 64.77 142.24 0)
+      (effects (font (size 1.27 1.27)) hide)
+    )
+    (property "Value" "+3V3" (id 1) (at 65.151 134.0358 0))
+    (property "Footprint" "" (id 2) (at 64.77 138.43 0)
+      (effects (font (size 1.27 1.27)) hide)
+    )
+    (property "Datasheet" "" (id 3) (at 64.77 138.43 0)
+      (effects (font (size 1.27 1.27)) hide)
+    )
+    (pin "1")
   )
   (symbol (lib_id "connectors:ESP32-DevBoard-Header") (at 38.1 72.39 0) (unit 1)
@@
     (pin "1")
   )
+  (symbol (lib_id "Connector_Generic:Conn_01x09") (at 78.74 151.13 0) (unit 1)
+    (in_bom yes) (on_board yes)
+    (property "Reference" "J6" (id 0) (at 76.6572 137.795 0))
+    (property "Value" "Conn_01x08" (id 1) (at 76.6572 159.6136 0)
+      (effects (font (size 1.27 1.27)) hide)
+    )
+    (property "Footprint" "Connector_Molex:Molex_PicoBlade_53047-0910_1x09_P1.25mm_Vertical" (id 2) (at 78.74 151.13 0)
+      (effects (font (size 1.27 1.27)) hide)
+    )
+    (property "Datasheet" "~" (id 3) (at 78.74 151.13 0)
+      (effects (font (size 1.27 1.27)) hide)
+    )
+    (pin "1")
+    (pin "2")
+    (pin "3")
+    (pin "4")
+    (pin "5")
+    (pin "6")
+    (pin "7")
+    (pin "8")
+    (pin "9")
+  )
   (symbol (lib_id "power:+3V3") (at 58.42 40.64 0) (unit 1)
     (in_bom yes) (on_board yes)
@@
       (reference "#PWR041") (unit 1) (value "GND") (footprint "")
     )
+    (path "/67443fbf-7fe2-4837-993c-0dba01d657e0"
+      (reference "#PWR042") (unit 1) (value "+3V3") (footprint "")
+    )
+    (path "/06ec3b09-2788-4deb-aa36-cfdacf9c2adf"
+      (reference "#PWR043") (unit 1) (value "+5V") (footprint "")
+    )
     (path "/a0d8e861-09bb-4835-9b2d-a093ba396bf8"
       (reference "#PWR044") (unit 1) (value "GND") (footprint "")
     )
+    (path "/33cbf7a5-344d-4e8f-ab59-268d8dbcd631"
+      (reference "#PWR045") (unit 1) (value "GND") (footprint "")
+    )
     (path "/3d2c1950-f6aa-4497-b2c6-a5d784533a6f"
       (reference "#PWR046") (unit 1) (value "GND") (footprint "")
@@
       (reference "J5") (unit 1) (value "Conn_01x09") (footprint "Connector_Molex:Molex_PicoBlade_53047-0710_1x07_P1.25mm_Vertical")
     )
+    (path "/e7814b55-e347-4b63-bcae-8b52aaf0f828"
+      (reference "J6") (unit 1) (value "Conn_01x08") (footprint "Connector_Molex:Molex_PicoBlade_53047-0910_1x09_P1.25mm_Vertical")
+    )
     (path "/e79152bf-ef81-4636-92c2-c03a1cbac590/8d264cc2-a1ff-4462-9ab6-9d50323b6105"
