File: ESP/DC Current Monitor/R1/PV Panel Monitor/PV Panel Monitor.kicad_pcb (KiCad board)
At the start: 4 copper layers, 50 x 50 mm, 66 parts, among them J1 Conn_01x04, U1 INA1228, U2 INA1228, U3 INA1228, U4 INA228, U5 ADS122C04, U6 ADM3260ARSZ

Commit message: Pile of uncommitted boards.
Parts:
- added C23: 0.1u, Capacitor_SMD:C_0603_1608Metric, F.Cu at (114.3, 78.1)
- added C24: 0.1u, Capacitor_SMD:C_0603_1608Metric, F.Cu at (106.3, 78.1)
- added C25: 0.1u, Capacitor_SMD:C_0603_1608Metric, F.Cu at (106.3, 75.6)
- added C26: 0.1u, Capacitor_SMD:C_0603_1608Metric, F.Cu at (106.3, 80.6)
- added R21: TBD, Resistor_SMD:R_0603_1608Metric, F.Cu at (118.3, 80.6)
- added R22: TBD, Resistor_SMD:R_0603_1608Metric, F.Cu at (110.3, 80.6)
- added R23: TBD, Resistor_SMD:R_0603_1608Metric, F.Cu at (110.3, 78.1)
- added R24: TBD, Resistor_SMD:R_0603_1608Metric, F.Cu at (110.3, 75.6)
- added R25: TBD, Resistor_SMD:R_0603_1608Metric, F.Cu at (118.3, 75.6)
- added R26: TBD, Resistor_SMD:R_0603_1608Metric, F.Cu at (114.3, 75.6)
- added R27: TBD, Resistor_SMD:R_0603_1608Metric, F.Cu at (114.3, 80.6)
- added R28: TBD, Resistor_SMD:R_0603_1608Metric, F.Cu at (118.3, 78.1)
Connections:
- U1 pad 10: Net-(R1-Pad3) -> Net-(U1-Pad10)
- U1 pad 3: Net-(U1-Pad3) -> unconnected-(U1-Pad3)
- U1 pad 9: Net-(R1-Pad2) -> Net-(U1-Pad9)
- U2 pad 10: Net-(R2-Pad3) -> Net-(U2-Pad10)
- U2 pad 3: Net-(U2-Pad3) -> unconnected-(U2-Pad3)
- U2 pad 9: Net-(R2-Pad2) -> Net-(U2-Pad9)
- U3 pad 10: Net-(R3-Pad3) -> Net-(U3-Pad10)
- U3 pad 3: Net-(U3-Pad3) -> unconnected-(U3-Pad3)
- U3 pad 9: Net-(R3-Pad2) -> Net-(U3-Pad9)
- U4 pad 10: Net-(R4-Pad3) -> Net-(U4-Pad10)
- U4 pad 3: Net-(U4-Pad3) -> unconnected-(U4-Pad3)
- U4 pad 9: Net-(R4-Pad2) -> Net-(U4-Pad9)
- U5 pad 14: Net-(U5-Pad14) -> unconnected-(U5-Pad14)
- U6 pad 15: Net-(U6-Pad15) -> unconnected-(U6-Pad15)
- U6 pad 6: Net-(U6-Pad6) -> unconnected-(U6-Pad6)
Routing:
- net Net-(R1-Pad3): track 17.9 -> 11.9 mm
- net Net-(R1-Pad2): track 17.0 -> 11.1 mm
- net Net-(R4-Pad3): track 16.7 -> 12.3 mm
- net Net-(R4-Pad2): track 15.9 -> 11.7 mm
- net Net-(R3-Pad2): track 16.0 -> 12.6 mm
- net Net-(U4-Pad10): track 0.00 -> 3.35 mm
- net Net-(R3-Pad3): track 16.8 -> 13.7 mm
- net Net-(R2-Pad2): track 16.1 -> 13.0 mm
- net Net-(U4-Pad9): track 0.00 -> 3.10 mm
- net Net-(R2-Pad3): track 16.9 -> 14.1 mm
- net Net-(R2-Pad4): track 28.6 -> 30.5 mm
- net Net-(U3-Pad9): track 0.00 -> 1.60 mm
- net Net-(U1-Pad10): track 0.00 -> 1.36 mm
- net Net-(U3-Pad10): track 0.00 -> 1.35 mm
- net Net-(U2-Pad9): track 0.00 -> 1.35 mm
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Other:
- net class Default removed
