File: ESP/RPi-Power R1/RPi-Power R1.kicad_pcb (KiCad board)
At the start: 2 copper layers, 53.3 x 25.4 mm, 22 parts, among them J1 Conn_01x02, J2 Raspberry_Pi_2_3, J3 Conn_01x01, J4 Conn_01x01, J5 Conn_01x03, J6 Conn_01x06, J7 Conn_01x03, U2 XL2012

Commit message: Pile of uncommitted boards.
Parts:
- added D4: LED, custom:CHIPLED_0603, F.Cu at (45.1, -5.71)
- added D5: LED, custom:CHIPLED_0603, F.Cu at (45.1, -8.89)
- added R3: R_Small, Resistor_SMD:R_0603_1608Metric, F.Cu at (42.5, -9.27)
- added R4: R_Small, Resistor_SMD:R_0603_1608Metric, F.Cu at (43.2, -12.1)
- J5: value Conn_01x03 -> Conn_01x05; footprint Connector_JST:JST_SH_BM04B-SRSS-TB_1x04-1MP_P1.00mm_Vertical -> Connector_JST:JST_SH_BM05B-SRSS-TB_1x05-1MP_P1.00mm_Vertical
- moved C8 1.02 mm to (38.7, -5.08)
- moved J4 0.81 mm to (8.76, -15.5)
- moved J3 0.72 mm to (8.76, -11.8)
- moved C3 0.51 mm to (34.3, -3.68)
- moved J5 0.38 mm to (39.6, -13.7)
Connections:
- J2 pad 1: Net-(J2-Pad1) -> +3V3
- J2 pad 10: Net-(J2-Pad10) -> unconnected-(J2-Pad10)
- J2 pad 11: Net-(J2-Pad11) -> unconnected-(J2-Pad11)
- J2 pad 12: Net-(J2-Pad12) -> unconnected-(J2-Pad12)
- J2 pad 13: Net-(J2-Pad13) -> unconnected-(J2-Pad13)
- J2 pad 15: Net-(J2-Pad15) -> unconnected-(J2-Pad15)
- J2 pad 16: Net-(J2-Pad16) -> unconnected-(J2-Pad16)
- J2 pad 17: Net-(J2-Pad17) -> +3V3
- J2 pad 18: Net-(J2-Pad18) -> unconnected-(J2-Pad18)
- J2 pad 19: Net-(J2-Pad19) -> unconnected-(J2-Pad19)
- J2 pad 22: Net-(J2-Pad22) -> unconnected-(J2-Pad22)
- J2 pad 24: Net-(J2-Pad24) -> unconnected-(J2-Pad24)
- J2 pad 26: Net-(J2-Pad26) -> unconnected-(J2-Pad26)
- J2 pad 29: Net-(J2-Pad29) -> unconnected-(J2-Pad29)
- J2 pad 3: Net-(J2-Pad3) -> unconnected-(J2-Pad3)
- J2 pad 31: Net-(J2-Pad31) -> unconnected-(J2-Pad31)
- J2 pad 32: Net-(J2-Pad32) -> unconnected-(J2-Pad32)
- J2 pad 33: Net-(J2-Pad33) -> unconnected-(J2-Pad33)
- J2 pad 5: Net-(J2-Pad5) -> unconnected-(J2-Pad5)
- J2 pad 7: Net-(J2-Pad7) -> unconnected-(J2-Pad7)
- J2 pad 8: Net-(J2-Pad8) -> unconnected-(J2-Pad8)
- J5 pad 2: Net-(J2-Pad27) -> +3V3
- J5 pad 3: Net-(J2-Pad28) -> Net-(J2-Pad27)
- J5 pad 4: GND -> Net-(J2-Pad28)
- U2 pad 2: Net-(U2-Pad2) -> unconnected-(U2-Pad2)
Routing:
- net +3V3: track 0.00 -> 50.4 mm
- net +5V: track 155.5 -> 141.9 mm
- net GND: track 54.6 -> 63.6 mm
- net Net-(D4-Pad2): track 0.00 -> 3.52 mm
- net Net-(D5-Pad2): track 0.00 -> 2.44 mm
- net Net-(J2-Pad37): track 18.1 -> 17.0 mm
Other:
- net class Default removed
- board text added: "PiPower C.Wolf 2023-01"
