File: ESP/ESP32 Dev Carrier - R1/power_supply.kicad_sch (KiCad schematic)
At the start: 15 parts, among them J1 Conn_01x02, U2 XL2001, U3 AMS1117-3.3

Commit message: Reworking things to use the new controller PCB.
Parts:
- D1: footprint Diode_SMD:D_SMA -> Diode_SMD:D_SMC
Changed lines of the file:
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@@
       (effects (font (size 1.27 1.27)) (justify left))
     )
-    (property "Footprint" "Diode_SMD:D_SMA" (id 2) (at 146.05 96.52 0)
+    (property "Footprint" "Diode_SMD:D_SMC" (id 2) (at 146.05 96.52 0)
       (effects (font (size 1.27 1.27)) hide)
     )
