File: ESP/ESP32 Ethernet Dev Carrier - R1/ESP32 Ethernet Dev Carrier - R1.kicad_pcb (KiCad board)
At the start: 4 copper layers, 75 x 75 mm, 84 parts, among them J1 Conn_01x02, J10 Conn_01x09, J11 Conn_01x04, J12 Conn_01x04, J13 Conn_01x04, J14 Conn_01x04, J2 USB_C_Receptacle_USB2.0, J3 Conn_02x20_Top_Bottom, J4 Conn_01x05, J5 Conn_01x05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

Commit message: More work.
Parts:
- removed D14, D15, D17: BAT54S, Package_TO_SOT_SMD:SOT-23
- removed D8: LED, custom:CHIPLED_0603
- removed J13, J14: Conn_01x04, Connector_JST:JST_XH_B4B-XH-A_1x04_P2.50mm_Vertical
- removed J7, J8: Conn_01x09, Connector_JST:JST_XH_B9B-XH-A_1x09_P2.50mm_Vertical
- removed R23: 4.7K, Resistor_SMD:R_0603_1608Metric
- removed R27: 470R, Resistor_SMD:R_0603_1608Metric
- added C14: 0.1 uF, Capacitor_SMD:C_0603_1608Metric, F.Cu at (48.0, 41.7)
- added C15: 22 uF, Capacitor_SMD:C_0603_1608Metric, F.Cu at (48.0, 43.2)
- added C16: 0.1 uF, Capacitor_SMD:C_0603_1608Metric, F.Cu at (42.9, 52.8)
- added C17: 22 uF, Capacitor_SMD:C_0603_1608Metric, F.Cu at (41.4, 52.8)
- added C18: 2.2 uF, Capacitor_SMD:C_0603_1608Metric, F.Cu at (40.1, 49.8)
- added C19: 0.1 uF, Capacitor_SMD:C_0603_1608Metric, F.Cu at (41.9, 49.8)
- added C20: 100nF/50V/20%/Y5V/C0603, Capacitor_SMD:C_0603_1608Metric, F.Cu at (60.7, 49.8)
- added C21: 1nF/2000V/10%/X7R/C1206, Capacitor_SMD:C_1206_3216Metric, F.Cu at (48.8, 64.5)
- added C22: NA(1nF/2000V/10%/X7R/C1206), Capacitor_SMD:C_1206_3216Metric, F.Cu at (70.6, 64.0)
- added C23: 0.1 uF, Capacitor_SMD:C_0603_1608Metric, F.Cu at (40.4, 46.0)
- added C24: 12 pF, Capacitor_SMD:C_0603_1608Metric, F.Cu at (53.3, 45.7)
- added C25: 12 pF, Capacitor_SMD:C_0603_1608Metric, F.Cu at (56.6, 49.8)
- added FB1: FerriteBead, Capacitor_SMD:C_0603_1608Metric, F.Cu at (38.9, 52.3)
- added LAN1: RJLD-060TC1(LPJ4013EDNL), custom:RJLBC-060TC1, F.Cu at (59.2, 63.5)
- added R28: 0R/R0603, Resistor_SMD:R_0603_1608Metric, F.Cu at (49.5, 53.8)
- added R29: 10R, Resistor_SMD:R_0603_1608Metric, F.Cu at (63.2, 24.4)
- added R30: 10R, Resistor_SMD:R_0603_1608Metric, F.Cu at (55.2, 23.9)
- added R31: 0R/R0603, Resistor_SMD:R_0603_1608Metric, F.Cu at (48.0, 53.8)
- added R32: 10R, Resistor_SMD:R_0603_1608Metric, F.Cu at (59.4, 24.4)
- added R33: 10R, Resistor_SMD:R_0603_1608Metric, F.Cu at (52.9, 22.1)
- added R34: 10R, Resistor_SMD:R_0603_1608Metric, F.Cu at (50.8, 25.7)
- added R35: 0R/R0603, Resistor_SMD:R_0603_1608Metric, F.Cu at (46.5, 53.8)
- added R36: 0R/R0603, Resistor_SMD:R_0603_1608Metric, F.Cu at (45.2, 53.8)
- added R37: 470R/R0603, Resistor_SMD:R_0603_1608Metric, F.Cu at (45.0, 35.1)
- added R38: 470R/R0603, Resistor_SMD:R_0603_1608Metric, F.Cu at (70.6, 67.6)
- added R39: 10K, Resistor_SMD:R_0603_1608Metric, F.Cu at (40.4, 47.5)
- added R40: 6.49K, Resistor_SMD:R_0603_1608Metric, F.Cu at (59.2, 34.3)
- added U5: KSZ8081RNA, Package_DFN_QFN:QFN-24-1EP_4x4mm_P0.5mm_EP2.6x2.6mm, F.Cu at (46.5, 47.5)
- added Y1: Crystal, Crystal:Crystal_SMD_3225-4Pin_3.2x2.5mm, F.Cu at (53.3, 48.8)
- J3: value Conn_02x20_Top_Bottom -> ESP32-DevBoard-Header
- R20: value 4.7K -> 470R
- R21: value 4.7K -> 10R
- moved R19 130.1 mm to (68.1, -70.1), turned to 0 degrees
- moved D6 126.1 mm to (68.5, -73.5)
- moved J9 115.1 mm to (20.7, -72.4), turned to 0 degrees
- moved R18 112.9 mm to (48.4, -51.1), turned to 0 degrees
- moved J10 111.0 mm to (20.7, -64.6), turned to 0 degrees
- moved R20 108.0 mm to (43.5, -46.7), turned to 0 degrees
- moved D11 105.8 mm to (63.6, -69.1)
- moved D5 102.3 mm to (34.2, -50.1)
- moved D10 94.4 mm to (43.9, -50.1)
- moved D9 92.9 mm to (34.2, -45.7)
- moved D13 86.8 mm to (39.0, -50.1)
- moved D2 83.9 mm to (63.6, -73.5)
- moved J12 78.0 mm to (20.7, -49.0), turned to 0 degrees
- moved J11 77.8 mm to (37.7, -56.8), turned to 0 degrees
- moved J6 76.1 mm to (47.7, -72.4), turned to 0 degrees
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Connections:
- C8 pad 1: /RESET -> /USB Interface/RESET
- D16 pad 3: /IO19 -> Net-(D16-Pad3)
- D18 pad 3: /IO22 -> /IO35
- D2 pad 3: /IO21 -> /IO34
- D5 pad 3: /IO26 -> Net-(D5-Pad3)
- D6 pad 3: /IO25 -> Net-(D6-Pad3)
- J10 pad 7: /IO25 -> Net-(D6-Pad3)
- J10 pad 8: /IO26 -> Net-(D5-Pad3)
- J11 pad 3: /IO19 -> Net-(D16-Pad3)
- J12 pad 3: /IO19 -> Net-(D16-Pad3)
- J4 pad 3: /IO22 -> /IO35
- J4 pad 4: /IO21 -> /IO34
- J5 pad 3: /IO22 -> /IO35
- J5 pad 4: /IO21 -> /IO34
- J6 pad 3: /IO22 -> /IO35
- J6 pad 4: /IO21 -> /IO34
- J9 pad 7: /IO25 -> Net-(D6-Pad3)
- J9 pad 8: /IO26 -> Net-(D5-Pad3)
- Q1 pad 3: /RESET -> /USB Interface/RESET
- R14 pad 1: /IO22 -> /IO35
- R15 pad 1: /IO21 -> /IO34
- R20 pad 1: /IO35 -> /IO36
- R20 pad 2: +3V3 -> /Ethernet PHY/RMII_REF_CLK_50M
- R21 pad 1: /IO34 -> Net-(R21-Pad1)
- R21 pad 2: +3V3 -> /IO21
- R22 pad 1: /IO19 -> Net-(D16-Pad3)
- R3 pad 1: Net-(R3-Pad1) -> /USB Interface/RESET
- SW1 pad 1: Net-(R3-Pad1) -> /USB Interface/RESET
Routing:
- net +5V: track 225.5 -> 66.2 mm, vias 4 -> 5
- net /IO5: track 140.5 -> 58.9 mm, vias 2 -> 1
- net /IO27: track 101.9 -> 27.6 mm
- net /IO15: track 128.5 -> 58.6 mm, vias 2 -> 1
- net /IO19: track 98.1 -> 51.4 mm
- net /IO18: track 105.4 -> 59.7 mm
- net /IO34: track 107.8 -> 64.7 mm, vias 2 -> 1
- net /IO26: track 100.5 -> 59.4 mm
- net /IO25: track 103.2 -> 63.7 mm
- net /IO35: track 101.7 -> 63.0 mm, vias 2 -> 1
- net /IO32: track 100.6 -> 66.3 mm
- net /IO33: track 98.4 -> 64.6 mm
- net +3V3: track 82.4 -> 48.8 mm, vias 22 -> 6
- net /IO22: track 83.8 -> 52.0 mm
- net /IO21: track 84.8 -> 53.5 mm
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Other:
- board text added: "TX RX D13 3V3"
- board text removed: "TX RX 3V3 P13 P27"

Commit message: Blerp.
Parts:
- added D14: BAT54S, Package_TO_SOT_SMD:SOT-23, F.Cu at (88.2, -47.4)
- added D8: BAT54S, Package_TO_SOT_SMD:SOT-23, F.Cu at (88.2, -42.9)
- added J7: Conn_01x04, Connector_JST:JST_XH_B4B-XH-A_1x04_P2.50mm_Vertical, F.Cu at (74.7, -38.4)
- added J8: Conn_01x04, Connector_JST:JST_XH_B4B-XH-A_1x04_P2.50mm_Vertical, F.Cu at (74.7, -46.2)
- added R23: 0R/R0603, Resistor_SMD:R_0603_1608Metric, F.Cu at (68.3, 42.2)
- added R27: 10R, Resistor_SMD:R_0603_1608Metric, F.Cu at (72.3, 42.2)
- R28, R31: value 0R/R0603 -> 10R
- R29, R33, R34: value 10R -> 0R/R0603
- R35, R36: value 0R/R0603 -> 470R/R0603
- R37: value 470R/R0603 -> 10K
- R38: value 470R/R0603 -> 6.49K
- moved C6 42.9 mm to (28.7, 50.4), turned to 90 degrees
- moved C11 37.4 mm to (28.7, 44.8), turned to -90 degrees
- moved U3 36.0 mm to (24.3, 47.7), turned to 90 degrees
- moved C10 30.3 mm to (17.4, 47.3), turned to -90 degrees
Connections:
- net /Ethernet PHY/RMII_REF_CLK_50M renamed Net-(R20-Pad2)
- net /Ethernet PHY/VDD1.2 renamed /VDD1.2
- net /Ethernet PHY/VDDA3.3 renamed /VDDA3.3
- C8 pad 1: /USB Interface/RESET -> /RESET
- D10 pad 3: /IO32 -> /IO33
- D11 pad 3: /IO5 -> Net-(D11-Pad3)
- D13 pad 3: /IO15 -> /IO5
- D5 pad 3: Net-(D5-Pad3) -> /IO35
- D9 pad 3: /IO33 -> Net-(D9-Pad3)
- J10 pad 5: /IO32 -> Net-(D11-Pad3)
- J10 pad 7: Net-(D6-Pad3) -> Net-(D9-Pad3)
- J10 pad 8: Net-(D5-Pad3) -> Net-(D8-Pad3)
- J3 pad 11: /IO32 -> unconnected-(J3-Pad11)
- J9 pad 5: /IO32 -> Net-(D11-Pad3)
- J9 pad 7: Net-(D6-Pad3) -> Net-(D9-Pad3)
- J9 pad 8: Net-(D5-Pad3) -> Net-(D8-Pad3)
- Q1 pad 3: /USB Interface/RESET -> /RESET
- R1 pad 2: /MOSI -> /IO2
- R18 pad 1: /IO5 -> Net-(D6-Pad3)
- R19 pad 1: /IO15 -> /IO5
- R22 pad 1: Net-(D16-Pad3) -> /IO15
- R28 pad 1: Net-(LAN1-Pad1) -> Net-(R28-Pad1)
- R28 pad 2: /Ethernet PHY/TXP+ -> /IO22
- R29 pad 1: Net-(R29-Pad1) -> Net-(LAN1-Pad2)
- R29 pad 2: /IO19 -> /TXN-
- R3 pad 1: /USB Interface/RESET -> Net-(R3-Pad1)
- R30 pad 2: /IO22 -> /IO25
- R31 pad 1: Net-(LAN1-Pad2) -> Net-(R31-Pad1)
- R31 pad 2: /Ethernet PHY/TXN- -> /IO26
- R32 pad 2: /IO25 -> /IO27
- R33 pad 1: Net-(R33-Pad1) -> Net-(LAN1-Pad7)
- R33 pad 2: /IO26 -> /RXP+
- R34 pad 1: Net-(R34-Pad1) -> Net-(LAN1-Pad8)
- R34 pad 2: /IO27 -> /RXN-
- R35 pad 1: Net-(LAN1-Pad7) -> Net-(LAN1-PadKY1)
- R35 pad 2: /Ethernet PHY/RXP+ -> Net-(R35-Pad2)
- R36 pad 1: Net-(LAN1-Pad8) -> Net-(LAN1-PadKG1)
- R36 pad 2: /Ethernet PHY/RXN- -> GND
- R37 pad 1: Net-(LAN1-PadKY1) -> /IO5
- R37 pad 2: Net-(R37-Pad2) -> GND
- R38 pad 1: Net-(LAN1-PadKG1) -> Net-(R38-Pad1)
- SW1 pad 1: /USB Interface/RESET -> GND
- SW1 pad 2: GND -> Net-(R3-Pad1)
- U5 pad 12: Net-(R33-Pad1) -> Net-(R31-Pad1)
- U5 pad 13: Net-(R32-Pad1) -> Net-(R30-Pad1)
- U5 pad 15: Net-(R34-Pad1) -> Net-(R32-Pad1)
- U5 pad 20: Net-(R29-Pad1) -> Net-(R27-Pad1)
- U5 pad 21: Net-(R30-Pad1) -> Net-(R28-Pad1)
- U5 pad 23: Net-(R37-Pad2) -> Net-(R35-Pad2)
- U5 pad 3: /Ethernet PHY/RXN- -> /RXN-
- U5 pad 4: /Ethernet PHY/RXP+ -> /RXP+
- U5 pad 5: /Ethernet PHY/TXN- -> /TXN-
- U5 pad 6: /Ethernet PHY/TXP+ -> /TXP+
- U5 pad 9: Net-(R40-Pad1) -> Net-(R38-Pad1)
Routing:
- net Net-(R40-Pad1): track 8.06 -> 0.00 mm
- net Net-(R38-Pad1): track 0.00 -> 8.06 mm
- net Net-(R3-Pad1): track 0.00 -> 5.34 mm, vias 0 -> 1
- net Net-(R37-Pad2): track 4.53 -> 0.00 mm
- net Net-(R35-Pad2): track 0.00 -> 4.53 mm
- net Net-(R33-Pad1): track 4.33 -> 0.00 mm
- net Net-(R31-Pad1): track 0.00 -> 4.33 mm
- net Net-(R30-Pad1): track 3.58 -> 0.00 mm
- net Net-(R28-Pad1): track 0.00 -> 3.58 mm
- net /USB Interface/RESET: track 3.46 -> 0.00 mm
- net Net-(R29-Pad1): track 2.60 -> 0.00 mm
- net Net-(R27-Pad1): track 0.00 -> 2.60 mm
- net GND: track 78.4 -> 76.5 mm, vias 34 -> 33
- net +5V: track 66.2 -> 66.7 mm
