File: ESP/ESP32 Ethernet Dev Carrier - R1/ESP32 Ethernet Dev Carrier - R1.kicad_sch (KiCad schematic)
At the start: 49 parts, among them J10 Conn_01x09, J11 Conn_01x04, J12 Conn_01x04, J13 Conn_01x04, J14 Conn_01x04, J3 ESP32-DevBoard-Header, J4 Conn_01x05, J5 Conn_01x05, J6 Conn_01x05, J7 Conn_01x09, J8 Conn_01x09, J9 Conn_01x09, SW1 SW_Push, U1 ESP32-WROVER-B_(16MB)

Commit message: More work.
Parts:
- removed D14, D15: BAT54S, Package_TO_SOT_SMD:SOT-23, symbol ESP32-Water-Meter-Monitor-rescue:D_Schottky_x2_Serial_AKC-Device
- removed D17: BAT54S, Package_TO_SOT_SMD:SOT-23, symbol Device:D_Schottky_x2_Serial_AKC
- removed D8: LED, custom:CHIPLED_0603, symbol Device:LED
- removed J13, J14: Conn_01x04, Connector_JST:JST_XH_B4B-XH-A_1x04_P2.50mm_Vertical, symbol Connector_Generic:Conn_01x04
- removed J7, J8: Conn_01x09, Connector_JST:JST_XH_B9B-XH-A_1x09_P2.50mm_Vertical, symbol Connector_Generic:Conn_01x09
- removed R21, R23: 4.7K, Resistor_SMD:R_0603_1608Metric, symbol Device:R_Small
- removed R27: 470R, Resistor_SMD:R_0603_1608Metric, symbol Device:R_Small
- R20: value 4.7K -> 470R
Connections:
- net +3V3: no longer R20.2
- net Ethernet PHY/RMII_REF_CLK_50M: now also R20.2
- net IO19: no longer D16.3 (common), J11.3 (Pin_3), J12.3 (Pin_3), R22.1
- net IO21: no longer D2.3 (common), J4.4 (Pin_4), J5.4 (Pin_4), J6.4 (Pin_4), R15.1
- net IO22: no longer D18.3 (common), J4.3 (Pin_3), J5.3 (Pin_3), J6.3 (Pin_3), R14.1
- net IO25: no longer D6.3 (common), J10.7 (Pin_7), J9.7 (Pin_7)
- net IO26: no longer D5.3 (common), J10.8 (Pin_8), J9.8 (Pin_8)
- net IO34: now also D2.3 (common), J4.4 (Pin_4), J5.4 (Pin_4), J6.4 (Pin_4), R15.1
- net IO35: now also D18.3 (common), J4.3 (Pin_3), J5.3 (Pin_3), J6.3 (Pin_3), R14.1; no longer R20.1
- net IO36: now also R20.1
- net RESET: no longer C8.1
- net USB Interface/RESET: now reaches R3.1, SW1.1
- net USB Interface/RESET: now also C8.1
- new net: D16.3 (common), J11.3 (Pin_3), J12.3 (Pin_3), R22.1
- new net: D6.3 (common), J10.7 (Pin_7), J9.7 (Pin_7)
- new net: D5.3 (common), J10.8 (Pin_8), J9.8 (Pin_8)
Other:
- moved on the sheet: C10, C8, C9, H1, H2, H3, H4, R3, R4, R5, SW1, U1

Commit message: Blerp.
Parts:
- removed D10, D11, D13, D5, D6, D9: BAT54S, Package_TO_SOT_SMD:SOT-23, symbol ESP32-Water-Meter-Monitor-rescue:D_Schottky_x2_Serial_AKC-Device
- removed D16, D18, D2: BAT54S, Package_TO_SOT_SMD:SOT-23, symbol Device:D_Schottky_x2_Serial_AKC
- removed J10, J9: Conn_01x09, Connector_JST:JST_XH_B9B-XH-A_1x09_P2.50mm_Vertical, symbol Connector_Generic:Conn_01x09
- removed J11, J12: Conn_01x04, Connector_JST:JST_XH_B4B-XH-A_1x04_P2.50mm_Vertical, symbol Connector_Generic:Conn_01x04
- removed J3: ESP32-DevBoard-Header, Connector_PinHeader_2.54mm:PinHeader_2x20_P2.54mm_Vertical, symbol connectors:ESP32-DevBoard-Header
- removed J4, J5, J6: Conn_01x05, Connector_JST:JST_XH_B5B-XH-A_1x05_P2.50mm_Vertical, symbol Connector_Generic:Conn_01x05
- removed R14, R15, R18, R19, R22: 4.7K, Resistor_SMD:R_0603_1608Metric, symbol Device:R_Small
- added C14, C16, C19, C23: 0.1 uF, Capacitor_SMD:C_0603_1608Metric, symbol Device:C_Small
- added C15, C17: 22 uF, Capacitor_SMD:C_0603_1608Metric, symbol Device:C_Small
- added C18: 2.2 uF, Capacitor_SMD:C_0603_1608Metric, symbol Device:C_Small
- added C20: 100nF/50V/20%/Y5V/C0603, Capacitor_SMD:C_0603_1608Metric, symbol ESP32-EVB_Rev_K:C
- added C21: 1nF/2000V/10%/X7R/C1206, Capacitor_SMD:C_1206_3216Metric, symbol ESP32-EVB_Rev_K:C
- added C22: NA(1nF/2000V/10%/X7R/C1206), Capacitor_SMD:C_1206_3216Metric, symbol ESP32-EVB_Rev_K:C
- added C24, C25: 12 pF, Capacitor_SMD:C_0603_1608Metric, symbol Device:C_Small
- added FB1: FerriteBead, Capacitor_SMD:C_0603_1608Metric, symbol Device:FerriteBead
- added LAN1: RJLD-060TC1(LPJ4013EDNL), custom:RJLBC-060TC1, symbol ESP32-EVB_Rev_K:RJLBC-060TC1_GND
- added R21, R27, R28, R30, R31, R32: 10R, Resistor_SMD:R_0603_1608Metric, symbol ESP32-EVB_Rev_K:R
- added R23, R29, R33, R34: 0R/R0603, Resistor_SMD:R_0603_1608Metric, symbol ESP32-EVB_Rev_K:R
- added R35, R36: 470R/R0603, Resistor_SMD:R_0603_1608Metric, symbol ESP32-EVB_Rev_K:R
- added R37: 10K, Resistor_SMD:R_0603_1608Metric, symbol ESP32-EVB_Rev_K:R
- added R38: 6.49K, Resistor_SMD:R_0603_1608Metric, symbol ESP32-EVB_Rev_K:R
- added U5: KSZ8081RNA, Package_DFN_QFN:QFN-24-1EP_4x4mm_P0.5mm_EP2.6x2.6mm, symbol Interface_Ethernet:KSZ8081RNA
- added Y1: Crystal, Crystal:Crystal_SMD_3225-4Pin_3.2x2.5mm, symbol Device:Crystal_GND24_Small
Connections:
- net +3V3: now also C14.1, C15.1, FB1.1, LAN1.AY1 (AY), U5.14 (VDDIO)
- net GND: now also SW1.1, C14.2, C15.2, C16.2, C17.2, C18.2, C19.2, C20.2, C21.2, C22.2, C23.2, C24.2, C25.2, R36.2, R37.2, R38.2, U5.22 (GND), U5.25 (GND), Y1.2, Y1.4; no longer SW1.2
- net IO18: now also U5.10 (MDIO)
- net IO19: now also R27.2
- net IO21: now also R21.2
- net IO22: now also R28.2
- net IO23: now also U5.11 (MDC)
- net IO25: now also R30.2
- net IO26: now also R31.2
- net IO27: now also R32.2
- net IO5: now also C23.1, R37.1, U5.24 (~{RST})
- net RESET: now also C8.1
- net Ethernet PHY/RMII_REF_CLK_50M: no longer names the net of R20.2
- net Ethernet PHY/RMII_REF_CLK_50M: now also U5.16 (REF_CLK)
- net IO2 renamed LED_GREEN
- net LED_GREEN: now also LAN1.AG1 (AG)
- removed net USB Interface/RESET: C8.1, R3.1, SW1.1
- new net: R3.1, SW1.2
- new net: LAN1.1 (TD+), R23.1
- new net: R30.1, U5.13 (RXD0)
- new net: LAN1.KG1 (KG), R36.1
- new net: C21.1, C22.1, LAN1.GND1, LAN1.GND2
- new net: C20.1, LAN1.3 (COM), LAN1.6 (NC)
- new net: R28.1, U5.21 (TXD1)
- new net: R31.1, U5.12 (RXD1)
- new net: LAN1.2 (TD-), R29.1
- new net: LAN1.7 (RD+), R33.1
- new net: LAN1.8 (RD-), R34.1
- new net: LAN1.KY1 (KY), R35.1
- new net: C24.1, U5.8 (XI), Y1.1
- new net: R21.1, U5.19 (TXEN)
- new net: R38.1, U5.9 (REXT)
- new net: C25.1, U5.7 (XO), Y1.3
- new net: R32.1, U5.15 (CRS_DV/PHYAD[1:0])
- new net: R27.1, U5.20 (TXD0)
- new net: R35.2, U5.23 (LED0/ANEN_SPEED)
- new net RXN-: R34.2, U5.3 (RXM)
- new net RXP+: R33.2, U5.4 (RXP)
- new net TXN-: R29.2, U5.5 (TXM)
- new net TXP+: R23.2, U5.6 (TXP)
- new net VDD1.2: C18.1, C19.1, U5.1 (VDD_1.2)
- new net VDDA3.3: C16.1, C17.1, FB1.2, U5.2 (VDDA_3.3)
- no-connect marks 6 -> 8
Other:
- removed sheet Ethernet PHY
- added sheet Connectors (connectors.kicad_sch)
- moved on the sheet: C10, C8, C9, D12, H1, H2, H3, H4, R10, R20, R3, R4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
