File: ESP/ESP32 Ethernet Dev Carrier - R1/ethernet.kicad_sch (KiCad schematic)
At the start: 30 parts

Commit message: More work.
Parts:
- C20: renamed from C?; footprint OLIMEX_RLC-FP:C_0603_5MIL_DWS -> Capacitor_SMD:C_0603_1608Metric
- C21, C22: renamed from C?; footprint OLIMEX_RLC-FP:C_1206_5MIL_DWS_ISO -> Capacitor_SMD:C_1206_3216Metric
- C24, C25: renamed from C?; value 22 pF -> 12 pF; LCSC C15849 -> C38523
- LAN1: renamed from LAN?; footprint OLIMEX_Connectors-FP:RJLBC-060TC1 -> custom:RJLBC-060TC1
- R21, R28, R29, R30, R31, R32, R33, R34, R35, R36, R37, R38, R39, R40: renamed from R?; footprint OLIMEX_RLC-FP:R_0603_5MIL_DWS -> Resistor_SMD:R_0603_1608Metric
- Y1: renamed from Y?; footprint (none) -> Crystal:Crystal_SMD_3225-4Pin_3.2x2.5mm; symbol Device:Crystal -> Device:Crystal_GND24_Small; LCSC (none) -> C9006
- gave numbers to parts that had none: 9
Connections:
- net GND: now also Y1.2, Y1.4
- net at C25.1, U5.7 (XO): now also Y1.3; no longer Y1.2
- net VDDA3.3: now reaches C16.1, C17.1, FB1.2, U5.2 (VDDA_3.3)
- net VDD1.2: now reaches C18.1, C19.1, U5.1 (VDD_1.2)

Commit message: Blerp.
Parts:
- removed C14, C16, C19, C23: 0.1 uF, Capacitor_SMD:C_0603_1608Metric, symbol Device:C_Small
- removed C15, C17: 22 uF, Capacitor_SMD:C_0603_1608Metric, symbol Device:C_Small
- removed C18: 2.2 uF, Capacitor_SMD:C_0603_1608Metric, symbol Device:C_Small
- removed C20: 100nF/50V/20%/Y5V/C0603, Capacitor_SMD:C_0603_1608Metric, symbol ESP32-EVB_Rev_K:C
- removed C21: 1nF/2000V/10%/X7R/C1206, Capacitor_SMD:C_1206_3216Metric, symbol ESP32-EVB_Rev_K:C
- removed C22: NA(1nF/2000V/10%/X7R/C1206), Capacitor_SMD:C_1206_3216Metric, symbol ESP32-EVB_Rev_K:C
- removed C24, C25: 12 pF, Capacitor_SMD:C_0603_1608Metric, symbol Device:C_Small
- removed FB1: FerriteBead, Capacitor_SMD:C_0603_1608Metric, symbol Device:FerriteBead
- removed LAN1: RJLD-060TC1(LPJ4013EDNL), custom:RJLBC-060TC1, symbol ESP32-EVB_Rev_K:RJLBC-060TC1_GND
- removed R21, R29, R30, R32, R33, R34: 10R, Resistor_SMD:R_0603_1608Metric, symbol ESP32-EVB_Rev_K:R
- removed R28, R31, R35, R36: 0R/R0603, Resistor_SMD:R_0603_1608Metric, symbol ESP32-EVB_Rev_K:R
- removed R37, R38: 470R/R0603, Resistor_SMD:R_0603_1608Metric, symbol ESP32-EVB_Rev_K:R
- removed R39: 10K, Resistor_SMD:R_0603_1608Metric, symbol ESP32-EVB_Rev_K:R
- removed R40: 6.49K, Resistor_SMD:R_0603_1608Metric, symbol ESP32-EVB_Rev_K:R
- removed U5: KSZ8081RNA, Package_DFN_QFN:QFN-24-1EP_4x4mm_P0.5mm_EP2.6x2.6mm, symbol Interface_Ethernet:KSZ8081RNA
- removed Y1: Crystal, Crystal:Crystal_SMD_3225-4Pin_3.2x2.5mm, symbol Device:Crystal_GND24_Small
Connections:
- no-connect marks 2 -> 0
Other:
- note removed: "=================== Desired Tdelay=500ms =================== 1. 49.9k/1%/R0603; 10uF/6.3V/20%/X5R/C0603; ===> Tdelay=750ms(Measured) 2. 220k/R0603; 1uF/10V/10%/X5R/C0603; =======> Tdelay=500ms(Measured) = OK!!!"
