File: ESP/ESP32 Ethernet Dev Carrier - R1/usb-interface.kicad_sch (KiCad schematic)
At the start: 19 parts, among them J2 USB_C_Receptacle_USB2.0, Q1 MMS9013, Q2 MMS9013, U4 CP2102N-Axx-xQFN28

Commit message: More work.
Parts:
- removed R?: 10k/R0603, OLIMEX_RLC-FP:R_0603_5MIL_DWS, symbol ESP32-EVB_Rev_K:R
- added R7: 49.9K, Resistor_SMD:R_0603_1608Metric, symbol Device:R_Small
- added R8: 22.1K, Resistor_SMD:R_0603_1608Metric, symbol Device:R_Small
Connections:
- net GND: now also R7.1
- net at R12.1: now also U4.9 (~{RST})
- net at U4.8 (VBUS): now also R7.2, R8.1
- net at J2.A4 (VBUS), J2.A9 (VBUS), J2.B4 (VBUS)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: now also R8.2
Changed lines of the file:
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@@
   (junction (at 48.26 73.66) (diameter 0) (color 0 0 0 0)
   )
+  (junction (at 73.66 91.44) (diameter 0) (color 0 0 0 0)
+  )
   (junction (at 101.6 43.18) (diameter 0) (color 0 0 0 0)
+  )
+  (junction (at 101.6 121.92) (diameter 0) (color 0 0 0 0)
   )
   (junction (at 48.26 76.2) (diameter 0) (color 0 0 0 0)
@@
   (no_connect (at 114.3 68.58))
   (no_connect (at 114.3 66.04))
+  (wire (pts (xy 88.9 71.12) (xy 81.28 71.12))
+    (stroke (width 0) (type default) (color 0 0 0 0))
+  )
   (wire (pts (xy 180.34 106.68) (xy 182.88 86.36))
     (stroke (width 0) (type default) (color 0 0 0 0))
@@
     (stroke (width 0) (type default) (color 0 0 0 0))
   )
-  (wire (pts (xy 162.56 82.55) (xy 162.56 93.98))
+  (wire (pts (xy 73.66 121.92) (xy 101.6 121.92))
     (stroke (width 0) (type default) (color 0 0 0 0))
   )
@@
     (stroke (width 0) (type default) (color 0 0 0 0))
   )
+  (wire (pts (xy 88.9 58.42) (xy 86.36 58.42))
+    (stroke (width 0) (type default) (color 0 0 0 0))
+  )
   (wire (pts (xy 114.3 60.96) (xy 193.04 60.96))
     (stroke (width 0) (type default) (color 0 0 0 0))
@@
     (stroke (width 0) (type default) (color 0 0 0 0))
   )
+  (wire (pts (xy 73.66 91.44) (xy 73.66 93.98))
+    (stroke (width 0) (type default) (color 0 0 0 0))
+  )
   (wire (pts (xy 52.07 82.55) (xy 52.07 66.04))
     (stroke (width 0) (type default) (color 0 0 0 0))
@@
     (stroke (width 0) (type default) (color 0 0 0 0))
   )
-  (wire (pts (xy 205.74 82.55) (xy 162.56 82.55))
-    (stroke (width 0) (type default) (color 0 0 0 0))
-  )
   (wire (pts (xy 144.78 91.44) (xy 144.78 88.9))
     (stroke (width 0) (type default) (color 0 0 0 0))
@@
     (stroke (width 0) (type default) (color 0 0 0 0))
   )
+  (wire (pts (xy 101.6 119.38) (xy 101.6 121.92))
+    (stroke (width 0) (type default) (color 0 0 0 0))
+  )
   (wire (pts (xy 114.3 91.44) (xy 144.78 91.44))
     (stroke (width 0) (type default) (color 0 0 0 0))
@@
     (stroke (width 0) (type default) (color 0 0 0 0))
   )
+  (wire (pts (xy 162.56 88.9) (xy 162.56 93.98))
+    (stroke (width 0) (type default) (color 0 0 0 0))
+  )
   (wire (pts (xy 45.72 78.74) (xy 48.26 78.74))
     (stroke (width 0) (type default) (color 0 0 0 0))
   )
+  (wire (pts (xy 81.28 91.44) (xy 73.66 91.44))
+    (stroke (width 0) (type default) (color 0 0 0 0))
+  )
   (wire (pts (xy 30.48 96.52) (xy 30.48 99.06))
     (stroke (width 0) (type default) (color 0 0 0 0))
@@
     (stroke (width 0) (type default) (color 0 0 0 0))
   )
+  (wire (pts (xy 160.02 88.9) (xy 162.56 88.9))
+    (stroke (width 0) (type default) (color 0 0 0 0))
+  )
   (wire (pts (xy 200.66 104.14) (xy 200.66 106.68))
     (stroke (width 0) (type default) (color 0 0 0 0))
@@
     (stroke (width 0) (type default) (color 0 0 0 0))
   )
+  (wire (pts (xy 81.28 71.12) (xy 81.28 91.44))
+    (stroke (width 0) (type default) (color 0 0 0 0))
+  )
   (wire (pts (xy 101.6 40.64) (xy 101.6 43.18))
     (stroke (width 0) (type default) (color 0 0 0 0))
   )
+  (wire (pts (xy 73.66 83.82) (xy 73.66 58.42))
+    (stroke (width 0) (type default) (color 0 0 0 0))
+  )
   (wire (pts (xy 48.26 73.66) (xy 88.9 73.66))
     (stroke (width 0) (type default) (color 0 0 0 0))
@@
     (stroke (width 0) (type default) (color 0 0 0 0))
   )
+  (wire (pts (xy 73.66 99.06) (xy 73.66 121.92))
+    (stroke (width 0) (type default) (color 0 0 0 0))
+  )
   (wire (pts (xy 60.96 45.72) (xy 60.96 43.18))
+    (stroke (width 0) (type default) (color 0 0 0 0))
+  )
+  (wire (pts (xy 73.66 91.44) (xy 73.66 88.9))
     (stroke (width 0) (type default) (color 0 0 0 0))
   )
@@
     (effects (font (size 1.27 1.27)) (justify left))
   )
-  (hierarchical_label "RESET" (shape output) (at 205.74 82.55 0)
-    (effects (font (size 1.27 1.27)) (justify left))
+  (hierarchical_label "RESET" (shape output) (at 160.02 88.9 180)
+    (effects (font (size 1.27 1.27)) (justify right))
   )
   (hierarchical_label "MISO" (shape input) (at 200.66 60.96 0)
@@
     (pin "2")
   )
+  (symbol (lib_id "Device:R_Small") (at 73.66 86.36 180) (unit 1)
+    (in_bom yes) (on_board yes)
+    (property "Reference" "R8" (id 0) (at 78.6384 86.36 90))
+    (property "Value" "22.1K" (id 1) (at 76.327 86.36 90))
+    (property "Footprint" "Resistor_SMD:R_0603_1608Metric" (id 2) (at 73.66 86.36 0)
+      (effects (font (size 1.27 1.27)) hide)
+    )
+    (property "Datasheet" "~" (id 3) (at 73.66 86.36 0)
+      (effects (font (size 1.27 1.27)) hide)
+    )
+    (property "LCSC" "C23184" (id 4) (at 78.6384 86.36 0)
+      (effects (font (size 1.27 1.27)) hide)
+    )
+    (pin "1")
+    (pin "2")
+  )
   (symbol (lib_id "Device:R_Small") (at 187.96 58.42 90) (mirror x) (unit 1)
     (in_bom yes) (on_board yes)
@@
     (pin "1")
     (pin "2")
+  )
+  (symbol (lib_id "power:GND") (at 101.6 121.92 0) (unit 1)
+    (in_bom yes) (on_board yes)
+    (property "Reference" "#PWR032" (id 0) (at 101.6 128.27 0)
+      (effects (font (size 1.27 1.27)) hide)
+    )
+    (property "Value" "GND" (id 1) (at 101.727 126.3142 0))
+    (property "Footprint" "" (id 2) (at 101.6 121.92 0)
+      (effects (font (size 1.27 1.27)) hide)
+    )
+    (property "Datasheet" "" (id 3) (at 101.6 121.92 0)
+      (effects (font (size 1.27 1.27)) hide)
+    )
+    (property "LCSC" "C14663" (id 4) (at 101.6 128.27 0)
+      (effects (font (size 1.27 1.27)) hide)
+    )
+    (pin "1")
   )
   (symbol (lib_id "power:GND") (at 60.96 50.8 0) (unit 1)
@@
     (pin "2")
   )
-  (symbol (lib_id "ESP32-EVB_Rev_K:R") (at 131.445 128.905 0) (unit 1)
-    (in_bom yes) (on_board yes)
-    (property "Reference" "R?" (id 0) (at 125.095 127.635 0))
-    (property "Value" "10k/R0603" (id 1) (at 140.97 127.635 0))
-    (property "Footprint" "OLIMEX_RLC-FP:R_0603_5MIL_DWS" (id 2) (at 131.445 130.683 0)
-      (effects (font (size 0.762 0.762)) hide)
-    )
-    (property "Datasheet" "" (id 3) (at 131.445 128.905 90)
-      (effects (font (size 0.762 0.762)))
-    )
-    (property "Fieldname 1" "Value 1" (id 4) (at 131.445 128.905 0)
-      (effects (font (size 1.524 1.524)) hide)
-    )
-    (property "Fieldname2" "Value2" (id 5) (at 131.445 128.905 0)
-      (effects (font (size 1.524 1.524)) hide)
-    )
-    (property "Fieldname3" "Value3" (id 6) (at 131.445 128.905 0)
-      (effects (font (size 1.524 1.524)) hide)
-    )
-    (pin "1")
-    (pin "2")
-  )
-  (symbol (lib_id "power:GND") (at 101.6 119.38 0) (unit 1)
-    (in_bom yes) (on_board yes)
-    (property "Reference" "#PWR?" (id 0) (at 101.6 125.73 0)
-      (effects (font (size 1.27 1.27)) hide)
-    )
-    (property "Value" "GND" (id 1) (at 101.727 123.7742 0))
-    (property "Footprint" "" (id 2) (at 101.6 119.38 0)
-      (effects (font (size 1.27 1.27)) hide)
-    )
-    (property "Datasheet" "" (id 3) (at 101.6 119.38 0)
-      (effects (font (size 1.27 1.27)) hide)
-    )
-    (property "LCSC" "C14663" (id 4) (at 101.6 125.73 0)
-      (effects (font (size 1.27 1.27)) hide)
-    )
-    (pin "1")
+  (symbol (lib_id "Device:R_Small") (at 73.66 96.52 180) (unit 1)
+    (in_bom yes) (on_board yes)
+    (property "Reference" "R7" (id 0) (at 78.6384 96.52 90))
+    (property "Value" "49.9K" (id 1) (at 76.327 96.52 90))
+    (property "Footprint" "Resistor_SMD:R_0603_1608Metric" (id 2) (at 73.66 96.52 0)
+      (effects (font (size 1.27 1.27)) hide)
+    )
+    (property "Datasheet" "~" (id 3) (at 73.66 96.52 0)
+      (effects (font (size 1.27 1.27)) hide)
+    )
+    (property "LCSC" "C23184" (id 4) (at 78.6384 96.52 0)
+      (effects (font (size 1.27 1.27)) hide)
+    )
+    (pin "1")
+    (pin "2")
   )
   (symbol (lib_id "power:GND") (at 30.48 99.06 0) (unit 1)

Commit message: Blerp.
Changed lines of the file:
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@@
+    (stroke (width 0) (type default) (color 0 0 0 0))
+  )
+  (wire (pts (xy 162.56 83.82) (xy 162.56 93.98))
     (stroke (width 0) (type default) (color 0 0 0 0))
   )
@@
     (stroke (width 0) (type default) (color 0 0 0 0))
   )
+  (wire (pts (xy 205.74 83.82) (xy 162.56 83.82))
+    (stroke (width 0) (type default) (color 0 0 0 0))
+  )
   (wire (pts (xy 172.72 71.12) (xy 172.72 86.36))
     (stroke (width 0) (type default) (color 0 0 0 0))
@@
     (stroke (width 0) (type default) (color 0 0 0 0))
   )
-  (wire (pts (xy 162.56 88.9) (xy 162.56 93.98))
-    (stroke (width 0) (type default) (color 0 0 0 0))
-  )
   (wire (pts (xy 45.72 78.74) (xy 48.26 78.74))
     (stroke (width 0) (type default) (color 0 0 0 0))
@@
   )
   (wire (pts (xy 48.26 71.12) (xy 48.26 73.66))
-    (stroke (width 0) (type default) (color 0 0 0 0))
-  )
-  (wire (pts (xy 160.02 88.9) (xy 162.56 88.9))
     (stroke (width 0) (type default) (color 0 0 0 0))
   )
@@
     (effects (font (size 1.27 1.27)) (justify left))
   )
-  (hierarchical_label "RESET" (shape output) (at 160.02 88.9 180)
-    (effects (font (size 1.27 1.27)) (justify right))
+  (hierarchical_label "RESET" (shape output) (at 205.74 83.82 0)
+    (effects (font (size 1.27 1.27)) (justify left))
   )
   (hierarchical_label "MISO" (shape input) (at 200.66 60.96 0)
     (effects (font (size 1.27 1.27)) (justify left))
   )
-  (symbol (lib_id "Device:R_Small") (at 129.54 99.06 180) (unit 1)
+  (symbol (lib_id "Device:R_Small") (at 129.54 99.06 180)
     (in_bom yes) (on_board yes)
     (property "Reference" "R17" (id 0) (at 134.5184 99.06 90))
@@
     (pin "2")
   )
-  (symbol (lib_id "Device:R_Small") (at 73.66 86.36 180) (unit 1)
+  (symbol (lib_id "Device:R_Small") (at 73.66 86.36 180)
     (in_bom yes) (on_board yes)
     (property "Reference" "R8" (id 0) (at 78.6384 86.36 90))
@@
     (pin "2")
   )
-  (symbol (lib_id "Device:R_Small") (at 187.96 58.42 90) (mirror x) (unit 1)
+  (symbol (lib_id "Device:R_Small") (at 187.96 58.42 90) (mirror x)
     (in_bom yes) (on_board yes)
     (property "Reference" "R1" (id 0) (at 187.96 53.4416 90))
@@
     (pin "2")
   )
-  (symbol (lib_id "power:GND") (at 59.69 99.06 0) (unit 1)
+  (symbol (lib_id "power:GND") (at 59.69 99.06 0)
     (in_bom yes) (on_board yes)
     (property "Reference" "#PWR0101" (id 0) (at 59.69 105.41 0)
@@
     (pin "1")
   )
-  (symbol (lib_id "Device:R_Small") (at 86.36 48.26 180) (unit 1)
+  (symbol (lib_id "Device:R_Small") (at 86.36 48.26 180)
     (in_bom yes) (on_board yes)
     (property "Reference" "R12" (id 0) (at 91.3384 48.26 90))
@@
     (pin "2")
   )
-  (symbol (lib_id "Device:LED") (at 137.16 77.47 90) (unit 1)
+  (symbol (lib_id "Device:LED") (at 137.16 77.47 90)
     (in_bom yes) (on_board yes)
     (property "Reference" "D3" (id 0) (at 140.1572 76.4794 90)
@@
     (pin "2")
   )
-  (symbol (lib_id "power:GND") (at 101.6 121.92 0) (unit 1)
+  (symbol (lib_id "power:GND") (at 101.6 121.92 0)
     (in_bom yes) (on_board yes)
     (property "Reference" "#PWR032" (id 0) (at 101.6 128.27 0)
@@
     (pin "1")
   )
-  (symbol (lib_id "power:GND") (at 60.96 50.8 0) (unit 1)
+  (symbol (lib_id "power:GND") (at 60.96 50.8 0)
     (in_bom yes) (on_board yes)
     (property "Reference" "#PWR016" (id 0) (at 60.96 57.15 0)
@@
     (pin "1")
   )
-  (symbol (lib_id "power:GND") (at 52.07 99.06 0) (unit 1)
+  (symbol (lib_id "power:GND") (at 52.07 99.06 0)
     (in_bom yes) (on_board yes)
     (property "Reference" "#PWR0103" (id 0) (at 52.07 105.41 0)
@@
     (pin "1")
   )
-  (symbol (lib_id "Device:R_Small") (at 190.5 93.98 180) (unit 1)
+  (symbol (lib_id "Device:R_Small") (at 190.5 93.98 180)
     (in_bom yes) (on_board yes)
     (property "Reference" "R11" (id 0) (at 195.4784 93.98 90))
@@
     (pin "2")
   )
-  (symbol (lib_id "Device:C_Small") (at 60.96 48.26 0) (unit 1)
+  (symbol (lib_id "Device:C_Small") (at 60.96 48.26 0)
     (in_bom yes) (on_board yes)
     (property "Reference" "C12" (id 0) (at 63.2968 47.0916 0)
@@
     (pin "2")
   )
-  (symbol (lib_id "Device:R_Small") (at 52.07 85.09 180) (unit 1)
+  (symbol (lib_id "Device:R_Small") (at 52.07 85.09 180)
     (in_bom yes) (on_board yes)
     (property "Reference" "R24" (id 0) (at 57.0484 85.09 90))
@@
     (pin "2")
   )
-  (symbol (lib_id "Transistor_BJT:BC846") (at 198.12 99.06 0) (unit 1)
+  (symbol (lib_id "Transistor_BJT:BC846") (at 198.12 99.06 0)
     (in_bom yes) (on_board yes) (fields_autoplaced)
     (property "Reference" "Q2" (id 0) (at 202.9714 98.1515 0)
@@
     (pin "3")
   )
-  (symbol (lib_id "Device:R_Small") (at 59.69 85.09 180) (unit 1)
+  (symbol (lib_id "Device:R_Small") (at 59.69 85.09 180)
     (in_bom yes) (on_board yes)
     (property "Reference" "R25" (id 0) (at 64.6684 85.09 90))
@@
     (pin "2")
   )
-  (symbol (lib_id "Device:R_Small") (at 144.78 86.36 180) (unit 1)
+  (symbol (lib_id "Device:R_Small") (at 144.78 86.36 180)
     (in_bom yes) (on_board yes)
     (property "Reference" "R16" (id 0) (at 149.86 86.36 90))
@@
     (pin "2")
   )
-  (symbol (lib_id "Transistor_BJT:BC846") (at 165.1 99.06 0) (mirror y) (unit 1)
+  (symbol (lib_id "Transistor_BJT:BC846") (at 165.1 99.06 0) (mirror y)
     (in_bom yes) (on_board yes) (fields_autoplaced)
     (property "Reference" "Q1" (id 0) (at 160.2487 98.1515 0)
@@
     (pin "3")
   )
-  (symbol (lib_id "Device:LED") (at 144.78 77.47 90) (unit 1)
+  (symbol (lib_id "Device:LED") (at 144.78 77.47 90)
     (in_bom yes) (on_board yes)
     (property "Reference" "D4" (id 0) (at 147.7772 76.4794 90)
@@
     (pin "2")
   )
-  (symbol (lib_id "Device:R_Small") (at 195.58 60.96 90) (mirror x) (unit 1)
+  (symbol (lib_id "Device:R_Small") (at 195.58 60.96 90) (mirror x)
     (in_bom yes) (on_board yes)
     (property "Reference" "R2" (id 0) (at 195.58 63.6016 90))
@@
     (pin "2")
   )
-  (symbol (lib_id "Device:R_Small") (at 73.66 96.52 180) (unit 1)
+  (symbol (lib_id "Device:R_Small") (at 73.66 96.52 180)
     (in_bom yes) (on_board yes)
     (property "Reference" "R7" (id 0) (at 78.6384 96.52 90))
@@
     (pin "2")
   )
-  (symbol (lib_id "power:GND") (at 30.48 99.06 0) (unit 1)
+  (symbol (lib_id "power:GND") (at 30.48 99.06 0)
     (in_bom yes) (on_board yes)
     (property "Reference" "#PWR023" (id 0) (at 30.48 105.41 0)
@@
     (pin "1")
   )
-  (symbol (lib_id "power:+3V3") (at 101.6 40.64 0) (unit 1)
+  (symbol (lib_id "power:+3V3") (at 101.6 40.64 0)
     (in_bom yes) (on_board yes)
     (property "Reference" "#PWR07" (id 0) (at 101.6 44.45 0)
@@
     (pin "1")
   )
-  (symbol (lib_id "power:GND") (at 129.54 121.92 0) (unit 1)
+  (symbol (lib_id "power:GND") (at 129.54 121.92 0)
     (in_bom yes) (on_board yes)
     (property "Reference" "#PWR033" (id 0) (at 129.54 128.27 0)
@@
     (pin "1")
   )
-  (symbol (lib_id "Device:R_Small") (at 172.72 93.98 180) (unit 1)
+  (symbol (lib_id "Device:R_Small") (at 172.72 93.98 180)
     (in_bom yes) (on_board yes)
     (property "Reference" "R9" (id 0) (at 177.6984 93.98 90))
@@
     (pin "2")
   )
-  (symbol (lib_id "Interface_USB:CP2102N-Axx-xQFN28") (at 101.6 86.36 0) (unit 1)
+  (symbol (lib_id "Interface_USB:CP2102N-Axx-xQFN28") (at 101.6 86.36 0)
     (in_bom yes) (on_board yes) (fields_autoplaced)
     (property "Reference" "U4" (id 0) (at 103.6194 118.9895 0)
@@
     (pin "9")
   )
-  (symbol (lib_id "Connector:USB_C_Receptacle_USB2.0") (at 30.48 73.66 0) (unit 1)
+  (symbol (lib_id "Connector:USB_C_Receptacle_USB2.0") (at 30.48 73.66 0)
     (in_bom yes) (on_board yes) (fields_autoplaced)
     (property "Reference" "J2" (id 0) (at 30.48 51.9135 0))
@@
     (pin "S1")
   )
-  (symbol (lib_id "power:GND") (at 73.66 50.8 0) (unit 1)
+  (symbol (lib_id "power:GND") (at 73.66 50.8 0)
     (in_bom yes) (on_board yes)
     (property "Reference" "#PWR027" (id 0) (at 73.66 57.15 0)
@@
     (pin "1")
   )
-  (symbol (lib_id "Device:R_Small") (at 137.16 86.36 180) (unit 1)
+  (symbol (lib_id "Device:R_Small") (at 137.16 86.36 180)
     (in_bom yes) (on_board yes)
     (property "Reference" "R13" (id 0) (at 138.6586 85.1916 0)
@@
     (pin "2")
   )
-  (symbol (lib_id "Device:C_Small") (at 73.66 48.26 0) (unit 1)
+  (symbol (lib_id "Device:C_Small") (at 73.66 48.26 0)
     (in_bom yes) (on_board yes)
     (property "Reference" "C13" (id 0) (at 75.9968 47.0916 0)
