File: Laser Cutter/Interface Board/Interface Board.kicad_pcb (KiCad board)
At the start: 2 copper layers, 43 parts, among them J1 Screw_Terminal_01x02, J2 Screw_Terminal_01x02, J3 Flow Sensor, J4 Screw_Terminal_01x02, J5 Limit Switch X, J6 Limit Switches Out, J7 Limit Switch Y, J8 Door Switch, J9 Flow Sensor, K1 SANYOU_SRD_Form_C, K2 SANYOU_SRD_Form_C, U1 ULN2003, U2 74HC14

Commit message: Pile of uncommitted boards.
Parts:
- added C10: 0.1u, Capacitor_THT:C_Disc_D3.8mm_W2.6mm_P2.50mm, F.Cu at (85.5, -15.8)
- added C11: 470u, Capacitor_THT:CP_Radial_D8.0mm_P3.50mm, F.Cu at (114.3, -6.00)
- added C12: 0.1u, Capacitor_THT:C_Disc_D3.8mm_W2.6mm_P2.50mm, F.Cu at (50.0, -46.8)
- added C13: 100u, Capacitor_THT:CP_Radial_D8.0mm_P3.50mm, F.Cu at (87.5, -92.5)
- added C4: 470u, Capacitor_THT:CP_Radial_D8.0mm_P3.50mm, F.Cu at (49.0, -8.15)
- added C5: 0.1u, Capacitor_THT:C_Disc_D3.8mm_W2.6mm_P2.50mm, F.Cu at (54.8, -4.00)
- added C6: 470u, Capacitor_THT:CP_Radial_D8.0mm_P3.50mm, F.Cu at (69.5, -8.15)
- added C7: 0.1u, Capacitor_THT:C_Disc_D3.8mm_W2.6mm_P2.50mm, F.Cu at (62.8, -4.00)
- added C8: 100u, Capacitor_THT:CP_Radial_D8.0mm_P3.50mm, F.Cu at (18.0, -89.3)
- added C9: 100u, Capacitor_THT:CP_Radial_D8.0mm_P3.50mm, F.Cu at (97.5, -92.5)
- added D10: LED, LED_THT:LED_D5.0mm, F.Cu at (125.0, -13.0)
- added D11: D_Schottky, Diode_THT:D_DO-15_P12.70mm_Horizontal, F.Cu at (91.0, -18.4)
- added D9: D_Schottky, Diode_THT:D_DO-15_P12.70mm_Horizontal, F.Cu at (95.7, -3.00)
- added H1: MountingHole, MountingHole:MountingHole_3.2mm_M3_Pad_Via, F.Cu at (145.0, -5.00)
- added H2: MountingHole, MountingHole:MountingHole_3.2mm_M3_Pad_Via, F.Cu at (145.0, -95.0)
- added H5: MountingHole, MountingHole:MountingHole_3.2mm_M3_Pad_Via, F.Cu at (5.00, -95.0)
- added H6: MountingHole, MountingHole:MountingHole_3.2mm_M3_Pad_Via, F.Cu at (5.00, -5.00)
- added J10: Screw_Terminal_01x02, TerminalBlock:TerminalBlock_bornier-2_P5.08mm, F.Cu at (145.0, -66.0)
- added J11: Limit Switches Out, Connector_JST:JST_XA_B07B-XASK-1_1x07_P2.50mm_Vertical, F.Cu at (145.0, -27.5)
- added J12: Limit Switches Out, Connector_JST:JST_XA_B05B-XASK-1_1x05_P2.50mm_Vertical, F.Cu at (145.0, -43.5)
- added JP5: SolderJumper_3_Bridged12, Jumper:SolderJumper-3_P1.3mm_Bridged12_Pad1.0x1.5mm_NumberLabels, B.Cu at (129.0, -44.5)
- added JP6: SolderJumper_3_Bridged12, Jumper:SolderJumper-3_P1.3mm_Bridged12_Pad1.0x1.5mm_NumberLabels, B.Cu at (108.0, -20.0)
- added JP7: SolderJumper_3_Bridged12, Jumper:SolderJumper-3_P1.3mm_Bridged12_Pad1.0x1.5mm_NumberLabels, B.Cu at (93.0, -24.0)
- added JP8: SolderJumper_3_Bridged12, Jumper:SolderJumper-3_P1.3mm_Bridged12_Pad1.0x1.5mm_NumberLabels, B.Cu at (136.5, -44.5)
- added JP9: SolderJumper_3_Bridged12, Jumper:SolderJumper-3_P1.3mm_Bridged12_Pad1.0x1.5mm_NumberLabels, B.Cu at (43.5, -7.00)
- added PS1: DC-DC, Converter_DCDC:Generic_DCDC_Red, F.Cu at (28.8, -93.6)
- added R16: 10K, Resistor_THT:R_Axial_DIN0204_L3.6mm_D1.6mm_P7.62mm_Horizontal, F.Cu at (129.0, -41.0)
- added R17: 10K, Resistor_THT:R_Axial_DIN0204_L3.6mm_D1.6mm_P7.62mm_Horizontal, F.Cu at (131.5, -41.0)
- added R18: 10K, Resistor_THT:R_Axial_DIN0204_L3.6mm_D1.6mm_P10.16mm_Horizontal, F.Cu at (134.0, -41.0)
- added R19: 1K, Resistor_THT:R_Axial_DIN0204_L3.6mm_D1.6mm_P7.62mm_Horizontal, F.Cu at (85.5, -26.3)
- added R20: 1K, Resistor_THT:R_Axial_DIN0204_L3.6mm_D1.6mm_P7.62mm_Horizontal, F.Cu at (95.2, -7.50)
- added R21: 2.2K, Resistor_THT:R_Axial_DIN0204_L3.6mm_D1.6mm_P7.62mm_Horizontal, F.Cu at (125.0, -9.81)
- added R22: 220, Resistor_THT:R_Axial_DIN0204_L3.6mm_D1.6mm_P7.62mm_Horizontal, F.Cu at (131.2, -24.5)
- added R23: 220, Resistor_THT:R_Axial_DIN0204_L3.6mm_D1.6mm_P7.62mm_Horizontal, F.Cu at (131.2, -22.0)
- added R24: 220, Resistor_THT:R_Axial_DIN0204_L3.6mm_D1.6mm_P7.62mm_Horizontal, F.Cu at (131.2, -19.5)
- added R25: 10K, Resistor_THT:R_Axial_DIN0204_L3.6mm_D1.6mm_P12.7mm_Horizontal, F.Cu at (136.5, -41.0)
- added R26: 10K, Resistor_THT:R_Axial_DIN0204_L3.6mm_D1.6mm_P12.7mm_Horizontal, F.Cu at (139.0, -41.0)
- added R27: 2.2K, Resistor_THT:R_Axial_DIN0204_L3.6mm_D1.6mm_P7.62mm_Horizontal, F.Cu at (28.7, -56.0)
- added R28: 2.2K, Resistor_THT:R_Axial_DIN0204_L3.6mm_D1.6mm_P7.62mm_Horizontal, F.Cu at (28.7, -53.5)
- added R29: 2.2K, Resistor_THT:R_Axial_DIN0204_L3.6mm_D1.6mm_P7.62mm_Horizontal, F.Cu at (28.7, -58.5)
- added R30: 2.2K, Resistor_THT:R_Axial_DIN0204_L3.6mm_D1.6mm_P7.62mm_Horizontal, F.Cu at (28.7, -51.0)
- added RV1: 100K, Potentiometer_THT:Potentiometer_Bourns_3299Y_Vertical, F.Cu at (114.5, -15.1)
- added RV2: 100K, Potentiometer_THT:Potentiometer_Bourns_3299Y_Vertical, F.Cu at (83.5, -8.50)
- added TP1: TestPoint, TestPoint:TestPoint_Loop_D1.80mm_Drill1.0mm_Beaded, F.Cu at (120.5, -18.5)
- added TP2: TestPoint, TestPoint:TestPoint_Loop_D1.80mm_Drill1.0mm_Beaded, F.Cu at (89.5, -29.5)
- added TP3: TestPoint, TestPoint:TestPoint_Loop_D1.80mm_Drill1.0mm_Beaded, F.Cu at (80.0, -13.5)
- added TP4: TestPoint, TestPoint:TestPoint_Loop_D1.80mm_Drill1.0mm_Beaded, F.Cu at (109.5, -8.50)
- added TP5: TestPoint, TestPoint:TestPoint_Loop_D1.80mm_Drill1.0mm_Beaded, F.Cu at (75.0, -21.0)
- added U3: L7805, Package_TO_SOT_THT:TO-220-3_Horizontal_TabDown, F.Cu at (57.5, -9.27)
- added U4: 74HC14, Package_DIP:DIP-14_W7.62mm_Socket_LongPads, F.Cu at (96.7, -28.6)
- D2, D4: footprint Diode_THT:D_DO-15_P15.24mm_Horizontal -> Diode_THT:D_DO-15_P12.70mm_Horizontal
- J3: value Flow Sensor -> Relay Signals
- JP1, JP2, JP3, JP4: moved to B.Cu
- moved JP2 228.3 mm to (121.0, -90.0), turned to -90 degrees
- moved K2 227.7 mm to (116.5, -90.0)
- moved J4 223.3 mm to (145.0, -88.0), turned to -90 degrees
- moved D2 217.3 mm to (111.0, -77.7), turned to -90 degrees
- moved D3 216.0 mm to (105.0, -94.0), turned to 90 degrees
- moved R1 215.4 mm to (107.0, -72.6), turned to -90 degrees
- moved JP1 211.8 mm to (121.0, -72.0), turned to -90 degrees
- moved D4 210.4 mm to (111.0, -95.7), turned to -90 degrees
- moved J6 201.2 mm to (145.5, -54.5), turned to -90 degrees
- moved R4 198.9 mm to (107.0, -90.6), turned to -90 degrees
- moved J1 196.8 mm to (5.00, -77.4), turned to 90 degrees
- moved J3 195.7 mm to (5.00, -67.5), turned to -90 degrees
- moved D5 191.0 mm to (114.0, -61.0), turned to -90 degrees
- moved K1 189.2 mm to (116.5, -72.0)
- moved J2 183.3 mm to (145.0, -77.0), turned to -90 degrees
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Connections:
- D5 pad 1: Net-(D5-Pad1) -> GND
- D5 pad 2: Net-(D5-Pad2) -> Net-(R5-Pad2)
- D6 pad 1: Net-(D6-Pad1) -> GND
- D6 pad 2: Net-(D6-Pad2) -> Net-(R8-Pad2)
- J3 pad 1: Net-(J3-Pad1) -> /RELAY_IN_1
- J3 pad 2: Net-(J3-Pad2) -> /RELAY_IN_2
- J5 pad 1: Net-(J5-Pad1) -> /LSW_X
- J6 pad 1: Net-(D5-Pad2) -> Net-(J6-Pad1)
- J6 pad 2: Net-(D6-Pad2) -> Net-(J6-Pad2)
- J7 pad 1: Net-(J7-Pad1) -> /LSW_Y
- J9 pad 1: +5V -> Net-(J9-Pad1)
- R3 pad 2: Net-(J5-Pad1) -> /LSW_X
- R5 pad 1: Net-(D5-Pad1) -> Net-(J6-Pad1)
- R5 pad 2: GND -> Net-(R5-Pad2)
- R7 pad 2: Net-(J7-Pad1) -> /LSW_Y
- R8 pad 1: Net-(D6-Pad1) -> Net-(J6-Pad2)
- R8 pad 2: GND -> Net-(R8-Pad2)
- U1 pad 1: Net-(J3-Pad1) -> Net-(U1-Pad1)
- U1 pad 10: unconnected-(U1-Pad10) -> Net-(R16-Pad2)
- U1 pad 11: unconnected-(U1-Pad11) -> Net-(R17-Pad2)
- U1 pad 12: unconnected-(U1-Pad12) -> Net-(R18-Pad2)
- U1 pad 13: unconnected-(U1-Pad13) -> Net-(R25-Pad2)
- U1 pad 14: unconnected-(U1-Pad14) -> Net-(R26-Pad2)
- U1 pad 15: Net-(D4-Pad2) -> Net-(D2-Pad2)
- U1 pad 16: Net-(D2-Pad2) -> Net-(D4-Pad2)
- U1 pad 2: Net-(J3-Pad2) -> Net-(U1-Pad2)
- U1 pad 3: Net-(D5-Pad2) -> Net-(J6-Pad1)
- U1 pad 4: Net-(D6-Pad2) -> Net-(J6-Pad2)
- U1 pad 7: unconnected-(U1-Pad7) -> Net-(D10-Pad2)
- U2 pad 10: Net-(JP4-Pad3) -> Net-(J6-Pad2)
- U2 pad 11: Net-(JP4-Pad1) -> /LSW_Y
- U2 pad 12: Net-(JP4-Pad1) -> Net-(J6-Pad1)
- U2 pad 13: Net-(R12-Pad1) -> /LSW_X
- U2 pad 3: Net-(JP3-Pad1) -> Net-(R12-Pad1)
- U2 pad 4: Net-(JP3-Pad3) -> Net-(JP4-Pad1)
- U2 pad 5: Net-(J7-Pad1) -> Net-(JP4-Pad1)
- U2 pad 6: Net-(D6-Pad2) -> Net-(JP4-Pad3)
- U2 pad 8: Net-(D5-Pad2) -> Net-(JP3-Pad3)
- U2 pad 9: Net-(J5-Pad1) -> Net-(JP3-Pad1)
Routing:
- net +12V: track 0.00 -> 483.5 mm, vias 0 -> 2
- net +24V: track 0.00 -> 219.4 mm, vias 0 -> 2
- net Net-(U4-Pad1): track 0.00 -> 146.3 mm, vias 0 -> 1
- net Net-(J6-Pad1): track 0.00 -> 129.6 mm
- net Net-(J6-Pad2): track 0.00 -> 123.5 mm
- net Net-(JP3-Pad2): track 0.00 -> 116.3 mm
- net Net-(D10-Pad2): track 0.00 -> 84.3 mm, vias 0 -> 1
- net Net-(R26-Pad2): track 0.00 -> 81.9 mm
- net Net-(R25-Pad2): track 0.00 -> 81.6 mm
- net Net-(R18-Pad2): track 0.00 -> 77.4 mm
- net Net-(R17-Pad2): track 0.00 -> 75.5 mm
- net Net-(R16-Pad2): track 0.00 -> 74.1 mm
- net Net-(U1-Pad1): track 0.00 -> 67.6 mm
- net Net-(U1-Pad2): track 0.00 -> 66.9 mm
- net /LSW_Y: track 0.00 -> 65.1 mm, vias 0 -> 1
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- added copper zone on In2.Cu, net +5V
- added copper zone on In1.Cu, net GND
Other:
- board outline added: 150 x 100 mm
- copper layers 2 -> 4
- board text added: "12V GND"
- board text added: "5V+ FLOW SENS GND"
- board text added: "DOOR"
- board text added: "DOOR INVERT"
- board text added: "DOOR SW GND"
- board text added: "FLOW I"
- board text added: "FLOW O"
- board text added: "FLOW SENSE INVERT"
- board text added: "FLOW SENSE POWER"
- board text added: "GND 24V IN"
- board text added: "LSW X IN GND LSW LED GND"
- board text added: "LSW X LSW Y"
- board text added: "LSW X OUT LSW Y OUT GND"
- board text added: "LSW Y IN GND LSW LED GND"
- board text added: "RELAY IN 1 RELAY IN 2 GND"
- board text added: "SW1 GND"
- board text added: "SW2 GND"
- board text added: "VCC LS-X LS-Y DOOR FLOW-I FLOW-O GND"
- board text added: "VCC OC-DOOR OC-FLOW-I OC-FLOW-O GND"

Commit message: Blerp.
Routing:
- net GND: track 7.92 -> 10.5 mm
- net +5V: track 56.2 -> 58.7 mm
Other:
- outline, holes or cut-outs redrawn
