File: Laser Cutter/Interface Board/Interface Board.kicad_sch (KiCad schematic)
At the start: 51 parts, among them J1 Screw_Terminal_01x02, J2 Screw_Terminal_01x02, J3 Flow Sensor, J4 Screw_Terminal_01x02, J5 Limit Switch X, J6 Limit Switches Out, J7 Limit Switch Y, J8 Door Switch, J9 Flow Sensor, K1 SANYOU_SRD_Form_C, K2 SANYOU_SRD_Form_C, U1 ULN2003, U2 74HC14

Commit message: Pile of uncommitted boards.
Parts:
- added C10, C12: 0.1u, Capacitor_THT:C_Disc_D3.8mm_W2.6mm_P2.50mm, symbol Device:C_Small
- added C11: 470u, Capacitor_THT:CP_Radial_D8.0mm_P3.50mm, symbol Device:C_Polarized_Small
- added C13: 100u, Capacitor_THT:CP_Radial_D8.0mm_P3.50mm, symbol Device:C_Polarized_Small
- added D10: LED, LED_THT:LED_D5.0mm, symbol Device:LED
- added D11, D9: D_Schottky, Diode_THT:D_DO-15_P12.70mm_Horizontal, symbol Device:D_Schottky
- added H1, H2, H5, H6: MountingHole, MountingHole:MountingHole_3.2mm_M3_Pad_Via, symbol Mechanical:MountingHole
- added J11: Limit Switches Out, Connector_JST:JST_XA_B07B-XASK-1_1x07_P2.50mm_Vertical, symbol Connector_Generic:Conn_01x07
- added J12: Limit Switches Out, Connector_JST:JST_XA_B05B-XASK-1_1x05_P2.50mm_Vertical, symbol Connector_Generic:Conn_01x05
- added JP5, JP6, JP7, JP8, JP9: SolderJumper_3_Bridged12, Jumper:SolderJumper-3_P1.3mm_Bridged12_Pad1.0x1.5mm_NumberLabels, symbol Jumper:SolderJumper_3_Bridged12
- added PS1: DC-DC, Converter_DCDC:Generic_DCDC_Red, symbol Converter_DCDC:DC-DC
- added R16, R17: 10K, Resistor_THT:R_Axial_DIN0204_L3.6mm_D1.6mm_P7.62mm_Horizontal, symbol Device:R_Small
- added R18: 10K, Resistor_THT:R_Axial_DIN0204_L3.6mm_D1.6mm_P10.16mm_Horizontal, symbol Device:R_Small
- added R19, R20: 1K, Resistor_THT:R_Axial_DIN0204_L3.6mm_D1.6mm_P7.62mm_Horizontal, symbol Device:R_Small
- added R21, R27, R28, R29, R30: 2.2K, Resistor_THT:R_Axial_DIN0204_L3.6mm_D1.6mm_P7.62mm_Horizontal, symbol Device:R_Small
- added R22, R23, R24: 220, Resistor_THT:R_Axial_DIN0204_L3.6mm_D1.6mm_P7.62mm_Horizontal, symbol Device:R_Small
- added R25, R26: 10K, Resistor_THT:R_Axial_DIN0204_L3.6mm_D1.6mm_P12.7mm_Horizontal, symbol Device:R_Small
- added RV1, RV2: 100K, Potentiometer_THT:Potentiometer_Bourns_3299Y_Vertical, symbol Device:R_Potentiometer
- added TP1, TP2, TP3, TP4, TP5: TestPoint, TestPoint:TestPoint_Loop_D1.80mm_Drill1.0mm_Beaded, symbol Connector:TestPoint
- added U4: 74HC14, Package_DIP:DIP-14_W7.62mm_Socket_LongPads, symbol 74xx:74HC14
- D2, D4: footprint Diode_THT:D_DO-15_P15.24mm_Horizontal -> Diode_THT:D_DO-15_P12.70mm_Horizontal
- J3: value Flow Sensor -> Relay Signals
- U3: renamed from U?; footprint Package_TO_SOT_THT:TO-220-3_Vertical -> Package_TO_SOT_THT:TO-220-3_Horizontal_TabDown
- gave numbers to parts that had none: 7
Connections:
- net +12V: now also C13.1, JP5.1 (A), JP9.3 (B), PS1.4 (+Vout)
- net +24V: now also JP5.3 (B), JP8.3 (B), PS1.1 (+Vin)
- net +5V: now also C12.1, JP8.1 (A), JP9.1 (A), RV1.1, RV1.2, U4.14 (VCC); no longer J9.1 (Pin_1)
- net GND: now also D5.1 (K), D6.1 (K), C11.2, C12.2, C13.2, D11.2 (A), J11.7 (Pin_7), J12.5 (Pin_5), PS1.2 (-Vin), PS1.3 (-Vout), R21.2, R29.2, R30.2, RV2.2, RV2.3, TP5.1, U4.13, U4.7 (GND); no longer R5.2, R8.2
- net at D2.2 (A), K1.2, R1.2: now also U1.15 (O2); no longer U1.16 (O1)
- net at R12.1, R13.2, R14.2: now also U2.3; no longer U2.13
- net at JP3.1 (A), U2.2: now also U2.9; no longer U2.3
- net at U2.4: now also JP4.1 (A), U2.5; no longer JP3.3 (B)
- net LSW_Y: now reaches J7.1 (Pin_1), R7.2
- net LSW_Y: now also U2.11; no longer U2.5
- net at D8.2 (A), JP4.2 (C), U1.6 (I6): now also R23.1, U4.1
- net at U1.1 (I1): now also R27.2; no longer J3.1 (Pin_1)
- net at U1.2 (I2): now also R28.2; no longer J3.2 (Pin_2)
- net at D4.2 (A), K2.2, R4.2: now also U1.16 (O1); no longer U1.15 (O2)
- net at R8.1: now also J6.2 (Pin_2), U1.4 (I4), U2.10; no longer D6.1 (K)
- net at JP4.3 (B): now also U2.6; no longer U2.10
- net at J6.1 (Pin_1), U1.3 (I3): now also R5.1, U2.12; no longer D5.2 (A), U2.8
- net LSW_X: now reaches J5.1 (Pin_1), R3.2
- net LSW_X: now also U2.13; no longer U2.9
- net at D7.2 (A), JP3.2 (C), U1.5 (I5): now also R22.1
- net at U1.10 (O7): now also J12.4 (Pin_4), R16.2
- net at U1.11 (O6): now also J12.3 (Pin_3), R17.2
- net at U1.12 (O5): now also J12.2 (Pin_2), R18.2
- net at U1.13 (O4): now also J11.3 (Pin_3), R25.2
- net at U1.14 (O3): now also J11.2 (Pin_2), R26.2
- net at U1.7 (I7): now also D10.2 (A), JP6.2 (C), R24.1, TP1.1
- new net: J9.1 (Pin_1), JP9.2 (C)
- new net: J11.1 (Pin_1), JP8.2 (C), R25.1, R26.1
- new net: J11.4 (Pin_4), R22.2
- new net: J11.5 (Pin_5), R23.2
- new net: J11.6 (Pin_6), R24.2
- new net: C11.1, D9.2 (A), RV1.3, TP4.1, U4.9
- new net: JP6.1 (A), U4.11, U4.8
- new net: JP6.3 (B), U4.10
- new net: J12.1 (Pin_1), JP5.2 (C), R16.1, R17.1, R18.1
- new net: D9.1 (K), R20.2
- new net: D10.1 (K), R21.1
- new net: C10.1, R19.2
- new net: C10.2, D11.1 (K), RV2.1, TP3.1, U4.5
- new net: D6.2 (A), R8.2
- new net: JP7.1 (A), TP2.1, U4.2, U4.3
- new net: R20.1, U4.6
- new net: JP3.3 (B), U2.8
- new net: JP7.3 (B), U4.4
- new net: JP7.2 (C), R19.1
- new net: D5.2 (A), R5.2
- new net RELAY_IN_1: J3.1 (Pin_1), R27.1, R29.1
- new net RELAY_IN_2: J3.2 (Pin_2), R28.1, R30.1
Other:
- moved on the sheet: C2, C8, C9, D1, D2, D3, D4, D5, D6, J1, J10, J2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
