File: ESP/Energy Monitor - Transformer PCB R2/Energy Monitor - Transformer PCB R2.kicad_pcb (KiCad board)
At the start: 2 copper layers, 100 x 100 mm, 27 parts, among them J1 Conn_01x02, J10 Conn_02x05_Odd_Even, J11 Conn_02x05_Odd_Even, J2 Conn_01x02, J3 Conn_01x02, J4 Conn_02x05_Odd_Even, J5 Conn_02x05_Odd_Even, J6 Conn_02x05_Odd_Even, J7 Conn_02x05_Odd_Even, J8 Conn_02x05_Odd_Even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

Commit message: Ordered PCBs!
Other:
- net class Default removed
