File: ESP/Energy Monitor - ESP32 PCB/Power Supplies.kicad_sch (KiCad schematic)
At the start: 19 parts, among them J1 Conn_02x05_Odd_Even, U5 VXO7805-500-M, U6 VXO7803-500-M

Commit message: Moar.
Parts:
- added D1, D2: LED, custom:CHIPLED_0603, symbol Device:LED
- added R7, R8: 1K, Resistor_SMD:R_0603_1608Metric, symbol Device:R_Small
- C10, C11: footprint Capacitor_SMD:C_0603_1608Metric_Pad1.05x0.95mm_HandSolder -> Capacitor_SMD:C_0603_1608Metric
- C12, C13, C6, C7, C8, C9: footprint Capacitor_SMD:C_1206_3216Metric_Pad1.42x1.75mm_HandSolder -> Capacitor_SMD:C_1206_3216Metric
- C14, C5: footprint Capacitor_THT:CP_Radial_D12.5mm_P5.00mm -> Capacitor_THT:CP_Radial_D7.5mm_P2.50mm
- C15, C16: footprint Capacitor_THT:CP_Radial_D8.0mm_P3.50mm -> Capacitor_THT:CP_Radial_D7.5mm_P2.50mm
Connections:
- net +3.3V: now also R8.1
- net +5V: now also R7.1
- net GND: now also D1.1 (K), D2.1 (K)
- new net: D1.2 (A), R7.2
- new net: D2.2 (A), R8.2
