File: ESP/Energy Monitor - ESP32 PCB/ESP32 and Comms.kicad_sch (KiCad schematic)
At the start: 25 parts, among them J10 Conn_01x04, J11 Conn_01x05, J12 Conn_01x05, J2 Conn_02x07_Odd_Even, J3 Conn_02x07_Odd_Even, J4 Conn_02x07_Odd_Even, J5 Conn_02x07_Odd_Even, J6 Conn_02x07_Odd_Even, J7 Conn_02x07_Odd_Even, J8 Conn_01x04, J9 Conn_01x04, U1 4072, U2 ESP32-POE Module, U3 4072, U4 4072

Commit message: Moar.
Parts:
- removed J10: Conn_01x04, Connector_PinHeader_2.54mm:PinHeader_1x04_P2.54mm_Vertical, symbol Connector_Generic:Conn_01x04
- added C17, C18, C19, C20, C21, C22, C23, C24, C25, C26, C27, C28: 0.1 uF, Capacitor_SMD:C_0603_1608Metric, symbol Device:C_Small
- added D10, D3, D4, D5, D6, D7, D8, D9: LED, custom:CHIPLED_0603, symbol Device:LED
- added R13, R14, R15: 49.9K, Resistor_SMD:R_0603_1608Metric, symbol Device:R_Small
- added R16, R17, R18, R19, R20, R21, R22, R23, R24, R25, R30, R31: 100R, Resistor_SMD:R_0603_1608Metric, symbol Device:R_Small
- added R26, R27, R28, R29, R40, R41, R42, R43: 1K, Resistor_SMD:R_0603_1608Metric, symbol Device:R_Small
- added R34, R35, R44, R45, R46, R47, R48, R49, R50, R51, R52, R53: 22K, Resistor_SMD:R_0603_1608Metric, symbol Device:R_Small
- added U10, U12, U14, U16, U18, U8: 74AHC1G08, Package_TO_SOT_SMD:SOT-23-5, symbol 74xGxx:74AHC1G08
- added U11, U13, U15, U17, U7, U9: 74LS367, Package_SO:SOIC-16_3.9x9.9mm_P1.27mm, symbol 74xx:74LS367
- C1, C2, C3: footprint Capacitor_SMD:C_0603_1608Metric_Pad1.05x0.95mm_HandSolder -> Capacitor_SMD:C_0603_1608Metric
- J11, J12: footprint Connector_PinHeader_2.54mm:PinHeader_1x05_P2.54mm_Vertical -> Connector_JST:JST_XH_B5B-XH-A_1x05_P2.50mm_Vertical
- J8, J9: footprint Connector_PinHeader_2.54mm:PinHeader_1x04_P2.54mm_Vertical -> Connector_JST:JST_XH_B4B-XH-A_1x04_P2.50mm_Vertical
- LCD1: renamed from LCD?1; symbol custom:0.96_-SSD1306-DISP-I2C -> custom:0.96-SSD1306-DISP-I2C
- R1, R2, R3, R4, R5, R6: footprint Resistor_SMD:R_0603_1608Metric_Pad1.05x0.95mm_HandSolder -> Resistor_SMD:R_0603_1608Metric
- U4: value 4072 -> 74HC154
Connections:
- net +3.3V: now also C17.1, C18.1, C19.1, C20.1, C21.1, C22.1, C23.1, C24.1, C25.1, C26.1, C27.1, C28.1, D10.2 (A), D7.2 (A), D8.2 (A), D9.2 (A), U10.5 (V), U11.16 (VCC), U12.5 (V), U13.16 (VCC), U14.5 (V), U15.16 (VCC), U16.5 (V), U17.16 (VCC), U18.5 (V), U7.16 (VCC), U8.5 (V), U9.16 (VCC)
- net +5V: now also LCD1.1 (VCC)
- net GND: now also LCD1.2 (Gnd), C17.2, C18.2, C19.2, C20.2, C21.2, C22.2, C23.2, C24.2, C25.2, C26.2, C27.2, C28.2, D3.1 (K), D4.1 (K), D5.1 (K), D6.1 (K), R13.2, R14.2, R15.2, R34.2, R35.2, R44.2, R45.2, R46.2, R47.2, R48.2, R49.2, R50.2, R51.2, R52.2, R53.2, U10.3 (G), U11.10 (I4), U11.15 (OEb), U11.8 (GND), U12.3 (G), U13.10 (I4), U13.15 (OEb), U13.8 (GND), U14.3 (G), U15.10 (I4), U15.15 (OEb), U15.8 (GND), U16.3 (G), U17.10 (I4), U17.15 (OEb), U17.8 (GND), U18.3 (G), U7.10 (I4), U7.15 (OEb), U7.8 (GND), U8.3 (G), U9.10 (I4), U9.15 (OEb), U9.8 (GND)
- net IRQ_1: now also R48.1, U13.12 (I5); no longer U1.5
- net IRQ_10: now also R47.1, U9.14 (I6); no longer U3.5
- net IRQ_11: now also R34.1, U11.12 (I5); no longer U3.3
- net IRQ_12: now also R35.1, U11.14 (I6); no longer U3.2
- net IRQ_2: now also R49.1, U13.14 (I6); no longer U1.4
- net IRQ_3: now also R50.1, U15.12 (I5); no longer U1.11
- net IRQ_4: now also R51.1, U15.14 (I6); no longer U1.12
- net IRQ_5: now also R52.1, U17.12 (I5); no longer U1.9
- net IRQ_6: now also R53.1, U17.14 (I6); no longer U1.10
- net IRQ_7: now also R44.1, U7.12 (I5); no longer U3.11
- net IRQ_8: now also R45.1, U7.14 (I6); no longer U3.12
- net IRQ_9: now also R46.1, U9.12 (I5); no longer U3.4
- net MISO: now also R15.1, U11.5 (O2a), U13.5 (O2a), U15.5 (O2a), U17.5 (O2a), U7.5 (O2a), U9.5 (O2a); no longer J2.11 (Pin_11), J3.11 (Pin_11), J4.11 (Pin_11), J5.11 (Pin_11), J6.11 (Pin_11), J7.11 (Pin_11)
- net MOSI: now also R14.1, U11.6 (I3), U13.6 (I3), U15.6 (I3), U17.6 (I3), U7.6 (I3), U9.6 (I3); no longer J2.9 (Pin_9), J3.9 (Pin_9), J4.9 (Pin_9), J5.9 (Pin_9), J6.9 (Pin_9), J7.9 (Pin_9)
- net SCLK: now also R13.1, U11.2 (I1), U13.2 (I1), U15.2 (I1), U17.2 (I1), U7.2 (I1), U9.2 (I1); no longer J2.13 (Pin_13), J3.13 (Pin_13), J4.13 (Pin_13), J5.13 (Pin_13), J6.13 (Pin_13), J7.13 (Pin_13)
- net ~{CS_10}: now also R25.2; no longer U4.10 (S9)
- net ~{CS_11}: now also R30.2; no longer U4.11 (S10)
- net ~{CS_12}: now also R31.2; no longer U4.13 (S11)
- net ~{CS_1}: now also R16.2; no longer U4.1 (S0)
- net ~{CS_2}: now also R17.2; no longer U4.2 (S1)
- net ~{CS_3}: now also R18.2; no longer U4.3 (S2)
- net ~{CS_4}: now also R19.2; no longer U4.4 (S3)
- net ~{CS_5}: now also R20.2; no longer U4.5 (S4)
- net ~{CS_6}: now also R21.2; no longer U4.6 (S5)
- net ~{CS_7}: now also R22.2; no longer U4.7 (S6)
- net ~{CS_8}: now also R23.2; no longer U4.8 (S7)
- net ~{CS_9}: now also R24.2; no longer U4.9 (S8)
- net CS_A3: now reaches U2.10 (GPIO5/SPI_CS), U4.20 (A3)
- net CS_A3: now also R29.1
- net CS_A0: now reaches U2.16 (GPIO32), U4.23 (A0)
- net CS_A0: now also R26.1
- net CS_A1: now reaches U2.17 (GPIO16/I2C-SCL), U4.22 (A1)
- net CS_A1: now also R27.1
- net CS_A2: now reaches U2.20 (GPIO13/I2C-SDA), U4.21 (A2)
- net CS_A2: now also R28.1
- net at J11.4 (Pin_4), J12.4 (Pin_4), R4.2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: now also LCD1.4 (SDA)
- net at J11.3 (Pin_3), J12.3 (Pin_3), R5.2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: now also LCD1.3 (SCL)
- net CS_EN: now reaches R1.2, U2.9 (GPIO4/U1TXD), U4.18 (E0)
- net at U4.14 (S12): now also R40.2
- net at U4.15 (S13): now also R41.2
- net at U4.16 (S14): now also R42.2
- net at U4.17 (S15): now also R43.2
- new net: R16.1, U14.2, U4.1 (S0)
- new net: R25.1, U12.1, U4.10 (S9)
- new net: R30.1, U4.11 (S10), U8.2
- new net: R31.1, U4.13 (S11), U8.1
- new net: R17.1, U14.1, U4.2 (S1)
- new net: R18.1, U16.2, U4.3 (S2)
- new net: R19.1, U16.1, U4.4 (S3)
- new net: R20.1, U18.2, U4.5 (S4)
- new net: R21.1, U18.1, U4.6 (S5)
- new net: R22.1, U10.2, U4.7 (S6)
- new net: R23.1, U10.1, U4.8 (S7)
- new net: R24.1, U12.2, U4.9 (S8)
- new net: U11.13 (O6b), U3.2
- new net: U11.11 (O5b), U3.3
- new net: U3.4, U9.11 (O5b)
- new net: U3.5, U9.13 (O6b)
- new net: U1.10, U17.13 (O6b)
- new net: U1.11, U15.11 (O5b)
- new net: U1.12, U15.13 (O6b)
- new net: U1.9, U17.11 (O5b)
- new net: U1.4, U13.13 (O6b)
- new net: U1.5, U13.11 (O5b)
- new net: U3.11, U7.11 (O5b)
- new net: U3.12, U7.13 (O6b)
- new net: D8.1 (K), R41.1
- new net: D5.2 (A), R28.2
- new net: U12.4, U9.1 (OEa)
- new net: U13.1 (OEa), U14.4
- new net: D10.1 (K), R43.1
- new net: U11.1 (OEa), U8.4
- new net: D7.1 (K), R40.1
- new net: D6.2 (A), R29.2
- new net: D3.2 (A), R26.2
- new net: D4.2 (A), R27.2
- new net: U17.1 (OEa), U18.4
- new net: D9.1 (K), R42.1
- new net: U15.1 (OEa), U16.4
- new net: U10.4, U7.1 (OEa)
- new net MISO_1: J2.11 (Pin_11), U13.4 (I2)
- new net MISO_2: J3.11 (Pin_11), U15.4 (I2)
- new net MISO_3: J4.11 (Pin_11), U17.4 (I2)
- new net MISO_4: J5.11 (Pin_11), U7.4 (I2)
- new net MISO_5: J6.11 (Pin_11), U9.4 (I2)
- new net MISO_6: J7.11 (Pin_11), U11.4 (I2)
- new net MOSI_1: J2.9 (Pin_9), U13.7 (O3a)
- new net MOSI_2: J3.9 (Pin_9), U15.7 (O3a)
- new net MOSI_3: J4.9 (Pin_9), U17.7 (O3a)
- new net MOSI_4: J5.9 (Pin_9), U7.7 (O3a)
- new net MOSI_5: J6.9 (Pin_9), U9.7 (O3a)
- new net MOSI_6: J7.9 (Pin_9), U11.7 (O3a)
- new net SCLK_1: J2.13 (Pin_13), U13.3 (O1a)
- new net SCLK_2: J3.13 (Pin_13), U15.3 (O1a)
- new net SCLK_3: J4.13 (Pin_13), U17.3 (O1a)
- new net SCLK_4: J5.13 (Pin_13), U7.3 (O1a)
- new net SCLK_5: J6.13 (Pin_13), U9.3 (O1a)
- new net SCLK_6: J7.13 (Pin_13), U11.3 (O1a)
Other:
- moved on the sheet: C1, C2, C3, J11, J12, J2, J3, J4, J5, J6, J7, J8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

Commit message: Blerp.
Parts:
- added D11, D12, D13, D14, D15, D16, D17, D18, D19, D20, D21, D22: LED, custom:CHIPLED_0603, symbol Device:LED
- added R10, R11, R12, R32, R33, R36, R37, R38, R39, R54, R55, R9: 1K, Resistor_SMD:R_0603_1608Metric, symbol Device:R_Small
Connections:
- net +3.3V: now also D11.2 (A), D12.2 (A), D13.2 (A), D14.2 (A), D15.2 (A), D16.2 (A), D17.2 (A), D18.2 (A), D19.2 (A), D20.2 (A), D21.2 (A), D22.2 (A)
- net ~{CS_1}: now also R16.1, U14.2, U4.5 (S4), R32.2
- net ~{CS_2}: now also R17.1, U14.1, U4.6 (S5), R33.2
- net at R2.1: now also U2.15 (GPIO33); no longer U2.12 (GPIO36/U1RXD)
- net 1WIRE: now reaches J8.2 (Pin_2), J9.2 (Pin_2), R6.2
- net 1WIRE: now also U2.12 (GPIO36/U1RXD); no longer U2.15 (GPIO33)
- net I2C_SDA: now reaches J11.4 (Pin_4), J12.4 (Pin_4), LCD1.4 (SDA), R4.2, U2.5 (GPIO0)
- net I2C_SCL: now reaches J11.3 (Pin_3), J12.3 (Pin_3), LCD1.3 (SCL), R5.2, U2.7 (GPIO2/HS2_DATA0)
- net ~{CS_10_R}: now reaches R25.1, U12.1, U4.10 (S9)
- net ~{CS_10_R}: now also R39.2
- net ~{CS_11_R}: now reaches R30.1, U8.2
- net ~{CS_11_R}: now also U4.7 (S6), R36.2; no longer U4.11 (S10)
- net ~{CS_12_R}: now reaches R31.1, U8.1
- net ~{CS_12_R}: now also U4.8 (S7), R37.2; no longer U4.13 (S11)
- net C13: now reaches R40.2, U4.14 (S12)
- net C14: now reaches R41.2, U4.15 (S13)
- net C15: now reaches R42.2, U4.16 (S14)
- net C16: now reaches R43.2, U4.17 (S15)
- net ~{CS_3_R}: now reaches R18.1, U16.2, U4.3 (S2)
- net ~{CS_3_R}: now also R11.2
- net ~{CS_4_R}: now reaches R19.1, U16.1, U4.4 (S3)
- net ~{CS_4_R}: now also R12.2
- net ~{CS_5_R}: now reaches R20.1, U18.2
- net ~{CS_5_R}: now also U4.1 (S0), R9.2; no longer U4.5 (S4)
- net ~{CS_6_R}: now reaches R21.1, U18.1
- net ~{CS_6_R}: now also U4.2 (S1), R10.2; no longer U4.6 (S5)
- net ~{CS_7_R}: now reaches R22.1, U10.2
- net ~{CS_7_R}: now also U4.11 (S10), R54.2; no longer U4.7 (S6)
- net ~{CS_8_R}: now reaches R23.1, U10.1
- net ~{CS_8_R}: now also U4.13 (S11), R55.2; no longer U4.8 (S7)
- net ~{CS_9_R}: now reaches R24.1, U12.2, U4.9 (S8)
- net ~{CS_9_R}: now also R38.2
- new net: D20.1 (K), R39.1
- new net: D14.1 (K), R12.1
- new net: D12.1 (K), R10.1
- new net: D18.1 (K), R37.1
- new net: D22.1 (K), R55.1
- new net: D13.1 (K), R11.1
- new net: D16.1 (K), R33.1
- new net: D17.1 (K), R36.1
- new net: D11.1 (K), R9.1
- new net: D19.1 (K), R38.1
- new net: D15.1 (K), R32.1
- new net: D21.1 (K), R54.1
Other:
- moved on the sheet: D10, D7, D8, D9, R40, R41, R42, R43
