File: ESP/Energy Monitor - ESP32 PCB/EnergyMonitor - ESP PCB.kicad_pcb (KiCad board)
At the start: 4 copper layers, 9 parts, among them J10 Conn_01x04, J11 Conn_01x05, J12 Conn_01x05, J8 Conn_01x04, J9 Conn_01x04

Commit message: Projects Projects Projects Projects.
Parts:
- added C1: 0.1 uF, Capacitor_SMD:C_0603_1608Metric_Pad1.05x0.95mm_HandSolder, F.Cu at (100.5, 86.5)
- added C10: 0.1 uF, Capacitor_SMD:C_0603_1608Metric_Pad1.05x0.95mm_HandSolder, F.Cu at (95.1, 108.0)
- added C11: 0.1 uF, Capacitor_SMD:C_0603_1608Metric_Pad1.05x0.95mm_HandSolder, F.Cu at (114.1, 108.0)
- added C12: 22 uF, Capacitor_SMD:C_1206_3216Metric_Pad1.42x1.75mm_HandSolder, F.Cu at (95.5, 98.5)
- added C13: 22 uF, Capacitor_SMD:C_1206_3216Metric_Pad1.42x1.75mm_HandSolder, F.Cu at (114.5, 98.5)
- added C14: CP1, Capacitor_THT:CP_Radial_D12.5mm_P5.00mm, F.Cu at (85.0, 129.0)
- added C15: CP1, Capacitor_THT:CP_Radial_D8.0mm_P3.50mm, F.Cu at (90.0, 101.0)
- added C16: CP1, Capacitor_THT:CP_Radial_D8.0mm_P3.50mm, F.Cu at (109.5, 101.0)
- added C2: 0.1 uF, Capacitor_SMD:C_0603_1608Metric_Pad1.05x0.95mm_HandSolder, F.Cu at (71.0, 94.0)
- added C3: 0.1 uF, Capacitor_SMD:C_0603_1608Metric_Pad1.05x0.95mm_HandSolder, F.Cu at (43.5, 85.5)
- added C4: CP1, Capacitor_THT:CP_Radial_D12.5mm_P5.00mm, F.Cu at (126.0, 129.0)
- added C5: CP1, Capacitor_THT:CP_Radial_D12.5mm_P5.00mm, F.Cu at (100.0, 129.0)
- added C6: 10 uF, 35V, Capacitor_SMD:C_1206_3216Metric_Pad1.42x1.75mm_HandSolder, F.Cu at (81.0, 120.5)
- added C7: 10 uF, 35V, Capacitor_SMD:C_1206_3216Metric_Pad1.42x1.75mm_HandSolder, F.Cu at (100.0, 120.5)
- added C8: 22 uF, Capacitor_SMD:C_1206_3216Metric_Pad1.42x1.75mm_HandSolder, F.Cu at (100.0, 112.5)
- added C9: 22 uF, Capacitor_SMD:C_1206_3216Metric_Pad1.42x1.75mm_HandSolder, F.Cu at (119.0, 112.5)
- added H1: MountingHole, MountingHole:MountingHole_3.2mm_M3_Pad_Via, F.Cu at (44.0, 44.0)
- added H2: MountingHole, MountingHole:MountingHole_3.2mm_M3_Pad_Via, F.Cu at (44.0, 136.0)
- added H3: MountingHole, MountingHole:MountingHole_3.2mm_M3_Pad_Via, F.Cu at (136.0, 44.0)
- added H4: MountingHole, MountingHole:MountingHole_3.2mm_M3_Pad_Via, F.Cu at (136.0, 136.0)
- added J1: Conn_02x05_Odd_Even, Connector_IDC:IDC-Header_2x05_P2.54mm_Vertical, F.Cu at (133.0, 106.0)
- added J2: Conn_02x07_Odd_Even, Connector_IDC:IDC-Header_2x07_P2.54mm_Vertical, F.Cu at (97.0, 45.0)
- added J3: Conn_02x07_Odd_Even, Connector_IDC:IDC-Header_2x07_P2.54mm_Vertical, F.Cu at (97.0, 56.0)
- added J4: Conn_02x07_Odd_Even, Connector_IDC:IDC-Header_2x07_P2.54mm_Vertical, F.Cu at (97.0, 67.0)
- added J5: Conn_02x07_Odd_Even, Connector_IDC:IDC-Header_2x07_P2.54mm_Vertical, F.Cu at (70.0, 45.0)
- added J6: Conn_02x07_Odd_Even, Connector_IDC:IDC-Header_2x07_P2.54mm_Vertical, F.Cu at (70.0, 56.0)
- added J7: Conn_02x07_Odd_Even, Connector_IDC:IDC-Header_2x07_P2.54mm_Vertical, F.Cu at (70.0, 67.0)
- added L1: 47 uH, Inductor_SMD:L_Bourns-SRU8028_8.0x8.0mm, F.Cu at (113.0, 129.0)
- added L2: 47 uH, Inductor_SMD:L_Bourns-SRU8028_8.0x8.0mm, F.Cu at (100.0, 104.0)
- added L3: 47 uH, Inductor_SMD:L_Bourns-SRU8028_8.0x8.0mm, F.Cu at (119.0, 104.0)
- added R1: 10K, Resistor_SMD:R_0603_1608Metric_Pad1.05x0.95mm_HandSolder, F.Cu at (79.5, 89.2)
- added R2: 330R, Resistor_SMD:R_0603_1608Metric_Pad1.05x0.95mm_HandSolder, F.Cu at (62.5, 113.5)
- added R3: 330R, Resistor_SMD:R_0603_1608Metric_Pad1.05x0.95mm_HandSolder, F.Cu at (45.5, 96.0)
- added U1: 4072, Package_SO:SOIC-14_3.9x8.7mm_P1.27mm, F.Cu at (103.0, 80.0)
- added U2: ESP32-POE Module, Energy Monitor - ESP32 PCB:ESP32-POE, F.Cu at (63.0, 140.0)
- added U3: 4072, Package_SO:SOIC-14_3.9x8.7mm_P1.27mm, F.Cu at (46.0, 79.0)
- added U4: 4072, Package_SO:SOIC-24W_7.5x15.4mm_P1.27mm, F.Cu at (64.0, 86.0)
- added U5: VXO7805-500-M, custom:VXO78x-500-M, F.Cu at (90.5, 116.5)
- added U6: VXO7803-500-M, custom:VXO78x-500-M, F.Cu at (109.5, 116.5)
- LCD1: value 0.96 -> 0.96"-SSD1306-DISP-I2C
Routing:
- net +5V: track 0.00 -> 285.5 mm
- net /ESP1/MISO: track 0.00 -> 127.1 mm
- net /ESP1/MOSI: track 0.00 -> 115.5 mm, vias 0 -> 1
- net GND: track 0.00 -> 104.8 mm, vias 0 -> 22
- net Net-(J10-Pad2): track 0.00 -> 103.8 mm
- net /ESP1/SCLK: track 0.00 -> 103.4 mm
- net Net-(J11-Pad4): track 0.00 -> 99.0 mm
- net Net-(J11-Pad3): track 0.00 -> 94.7 mm
- net /ESP1/~{CS_2}: track 0.00 -> 67.1 mm
- net /ESP1/~{CS_1}: track 0.00 -> 64.8 mm
- net Net-(R2-Pad2): track 0.00 -> 62.4 mm, vias 0 -> 2
- net /ESP1/~{CS_4}: track 0.00 -> 55.7 mm
- net /ESP1/IRQ_7: track 0.00 -> 55.7 mm
- net /ESP1/IRQ_2: track 0.00 -> 55.2 mm
- net /ESP1/~{CS_3}: track 0.00 -> 53.8 mm
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- added copper zone on In2.Cu, net +3V3
- added copper zone on In1.Cu, net GND
Other:
- board outline added: 100 x 100 mm
- net class Default removed

Commit message: Moar.
Parts:
- removed J10: Conn_01x04, Connector_PinHeader_2.54mm:PinHeader_1x04_P2.54mm_Vertical
- added C17: 0.1 uF, Capacitor_SMD:C_0603_1608Metric, F.Cu at (83.8, 52.8)
- added C18: 0.1 uF, Capacitor_SMD:C_0603_1608Metric, F.Cu at (74.3, 53.3)
- added C19: 0.1 uF, Capacitor_SMD:C_0603_1608Metric, F.Cu at (74.3, 67.3)
- added C20: 0.1 uF, Capacitor_SMD:C_0603_1608Metric, F.Cu at (74.3, 81.3)
- added C21: 0.1 uF, Capacitor_SMD:C_0603_1608Metric, F.Cu at (114.3, 53.3)
- added C22: 0.1 uF, Capacitor_SMD:C_0603_1608Metric, F.Cu at (114.3, 67.3)
- added C23: 0.1 uF, Capacitor_SMD:C_0603_1608Metric, F.Cu at (114.3, 81.3)
- added C24: 0.1 uF, Capacitor_SMD:C_0603_1608Metric, F.Cu at (123.8, 52.8)
- added C25: 0.1 uF, Capacitor_SMD:C_0603_1608Metric, F.Cu at (123.8, 66.8)
- added C26: 0.1 uF, Capacitor_SMD:C_0603_1608Metric, F.Cu at (123.8, 80.8)
- added C27: 0.1 uF, Capacitor_SMD:C_0603_1608Metric, F.Cu at (83.8, 66.8)
- added C28: 0.1 uF, Capacitor_SMD:C_0603_1608Metric, F.Cu at (83.8, 80.8)
- added D1: LED, custom:CHIPLED_0603, F.Cu at (42.7, 109.8)
- added D10: LED, custom:CHIPLED_0603, F.Cu at (42.1, 119.8)
- added D2: LED, custom:CHIPLED_0603, F.Cu at (42.7, 107.9)
- added D3: LED, custom:CHIPLED_0603, F.Cu at (42.7, 106.0)
- added D4: LED, custom:CHIPLED_0603, F.Cu at (42.7, 104.1)
- added D5: LED, custom:CHIPLED_0603, F.Cu at (42.7, 102.2)
- added D6: LED, custom:CHIPLED_0603, F.Cu at (42.7, 100.3)
- added D7: LED, custom:CHIPLED_0603, F.Cu at (42.1, 112.5)
- added D8: LED, custom:CHIPLED_0603, F.Cu at (42.1, 115.0)
- added D9: LED, custom:CHIPLED_0603, F.Cu at (42.1, 117.4)
- added R13: 49.9K, Resistor_SMD:R_0603_1608Metric, F.Cu at (29.6, 93.1)
- added R14: 49.9K, Resistor_SMD:R_0603_1608Metric, F.Cu at (30.3, 89.9)
- added R15: 49.9K, Resistor_SMD:R_0603_1608Metric, F.Cu at (29.6, 95.6)
- added R16: 100R, Resistor_SMD:R_0603_1608Metric, F.Cu at (106.7, 53.3)
- added R17: 100R, Resistor_SMD:R_0603_1608Metric, F.Cu at (104.8, 53.3)
- added R18: 100R, Resistor_SMD:R_0603_1608Metric, F.Cu at (106.7, 67.3)
- added R19: 100R, Resistor_SMD:R_0603_1608Metric, F.Cu at (104.8, 67.3)
- added R20: 100R, Resistor_SMD:R_0603_1608Metric, F.Cu at (106.7, 81.3)
- added R21: 100R, Resistor_SMD:R_0603_1608Metric, F.Cu at (104.8, 81.3)
- added R22: 100R, Resistor_SMD:R_0603_1608Metric, F.Cu at (66.7, 53.3)
- added R23: 100R, Resistor_SMD:R_0603_1608Metric, F.Cu at (64.8, 53.3)
- added R24: 100R, Resistor_SMD:R_0603_1608Metric, F.Cu at (66.7, 67.3)
- added R25: 100R, Resistor_SMD:R_0603_1608Metric, F.Cu at (64.8, 67.3)
- added R26: 1K, Resistor_SMD:R_0603_1608Metric, F.Cu at (46.5, 106.0)
- added R27: 1K, Resistor_SMD:R_0603_1608Metric, F.Cu at (46.5, 104.1)
- added R28: 1K, Resistor_SMD:R_0603_1608Metric, F.Cu at (46.5, 102.2)
- added R29: 1K, Resistor_SMD:R_0603_1608Metric, F.Cu at (46.5, 100.3)
- added R30: 100R, Resistor_SMD:R_0603_1608Metric, F.Cu at (66.7, 81.3)
- added R31: 100R, Resistor_SMD:R_0603_1608Metric, F.Cu at (64.8, 81.3)
- added R34: 22K, Resistor_SMD:R_0603_1608Metric, F.Cu at (62.9, 81.3)
- added R35: 22K, Resistor_SMD:R_0603_1608Metric, F.Cu at (60.3, 81.3)
- added R40: 1K, Resistor_SMD:R_0603_1608Metric, F.Cu at (46.5, 112.4)
- added R41: 1K, Resistor_SMD:R_0603_1608Metric, F.Cu at (46.5, 114.9)
- added R42: 1K, Resistor_SMD:R_0603_1608Metric, F.Cu at (46.5, 117.5)
- added R43: 1K, Resistor_SMD:R_0603_1608Metric, F.Cu at (46.5, 120.0)
- added R44: 22K, Resistor_SMD:R_0603_1608Metric, F.Cu at (62.9, 53.3)
- added R45: 22K, Resistor_SMD:R_0603_1608Metric, F.Cu at (60.3, 53.3)
- added R46: 22K, Resistor_SMD:R_0603_1608Metric, F.Cu at (62.9, 67.3)
- added R47: 22K, Resistor_SMD:R_0603_1608Metric, F.Cu at (60.3, 67.3)
- added R48: 22K, Resistor_SMD:R_0603_1608Metric, F.Cu at (102.9, 53.3)
- added R49: 22K, Resistor_SMD:R_0603_1608Metric, F.Cu at (100.3, 53.3)
- added R50: 22K, Resistor_SMD:R_0603_1608Metric, F.Cu at (102.9, 67.3)
- added R51: 22K, Resistor_SMD:R_0603_1608Metric, F.Cu at (100.3, 67.3)
- added R52: 22K, Resistor_SMD:R_0603_1608Metric, F.Cu at (102.9, 81.3)
- added R53: 22K, Resistor_SMD:R_0603_1608Metric, F.Cu at (100.3, 81.3)
- added R7: 1K, Resistor_SMD:R_0603_1608Metric, F.Cu at (46.5, 109.8)
- added R8: 1K, Resistor_SMD:R_0603_1608Metric, F.Cu at (46.5, 107.9)
- added U10: 74AHC1G08, Package_TO_SOT_SMD:SOT-23-5, F.Cu at (70.5, 54.0)
- added U11: 74LS367, Package_SO:SOIC-16_3.9x9.9mm_P1.27mm, F.Cu at (80.0, 76.3)
- added U12: 74AHC1G08, Package_TO_SOT_SMD:SOT-23-5, F.Cu at (70.5, 67.9)
- added U13: 74LS367, Package_SO:SOIC-16_3.9x9.9mm_P1.27mm, F.Cu at (120.0, 48.3)
- added U14: 74AHC1G08, Package_TO_SOT_SMD:SOT-23-5, F.Cu at (110.5, 54.0)
- added U15: 74LS367, Package_SO:SOIC-16_3.9x9.9mm_P1.27mm, F.Cu at (120.0, 62.3)
- added U16: 74AHC1G08, Package_TO_SOT_SMD:SOT-23-5, F.Cu at (110.5, 67.9)
- added U17: 74LS367, Package_SO:SOIC-16_3.9x9.9mm_P1.27mm, F.Cu at (120.0, 76.3)
- added U18: 74AHC1G08, Package_TO_SOT_SMD:SOT-23-5, F.Cu at (110.5, 81.9)
- added U7: 74LS367, Package_SO:SOIC-16_3.9x9.9mm_P1.27mm, F.Cu at (80.0, 48.3)
- added U8: 74AHC1G08, Package_TO_SOT_SMD:SOT-23-5, F.Cu at (70.5, 81.9)
- added U9: 74LS367, Package_SO:SOIC-16_3.9x9.9mm_P1.27mm, F.Cu at (80.0, 62.3)
- C1, C10, C11, C2, C3: footprint Capacitor_SMD:C_0603_1608Metric_Pad1.05x0.95mm_HandSolder -> Capacitor_SMD:C_0603_1608Metric
- C12, C13, C6, C7, C8, C9: footprint Capacitor_SMD:C_1206_3216Metric_Pad1.42x1.75mm_HandSolder -> Capacitor_SMD:C_1206_3216Metric
- C14, C5: footprint Capacitor_THT:CP_Radial_D12.5mm_P5.00mm -> Capacitor_THT:CP_Radial_D7.5mm_P2.50mm
- C15, C16: footprint Capacitor_THT:CP_Radial_D8.0mm_P3.50mm -> Capacitor_THT:CP_Radial_D7.5mm_P2.50mm
- J11, J12: footprint Connector_PinHeader_2.54mm:PinHeader_1x05_P2.54mm_Vertical -> Connector_JST:JST_XH_B5B-XH-A_1x05_P2.50mm_Vertical
- J8, J9: footprint Connector_PinHeader_2.54mm:PinHeader_1x04_P2.54mm_Vertical -> Connector_JST:JST_XH_B4B-XH-A_1x04_P2.50mm_Vertical
- R1, R2, R3, R4, R5, R6: footprint Resistor_SMD:R_0603_1608Metric_Pad1.05x0.95mm_HandSolder -> Resistor_SMD:R_0603_1608Metric
- U4: value 4072 -> 74HC154
- moved R6 78.1 mm to (68.6, 153.0), turned to 180 degrees
- moved R2 63.6 mm to (123.8, 96.5), turned to 90 degrees
- moved R5 62.9 mm to (66.0, 157.5), turned to 180 degrees
- moved LCD1 62.7 mm to (80.2, 98.4), turned to 90 degrees
- moved R4 58.9 mm to (61.4, 156.2), turned to 0 degrees
- moved U2 57.4 mm to (63.5, 82.6), turned to 180 degrees
- moved J11 51.1 mm to (129.5, 92.7)
- moved R1 50.2 mm to (54.0, 132.5), turned to -90 degrees
- moved J12 48.3 mm to (136.0, 92.6)
- moved U3 47.4 mm to (92.8, 86.9)
- moved R3 33.7 mm to (76.2, 109.8)
- moved C2 27.7 mm to (71.1, 121.7)
- moved U4 27.7 mm to (64.1, 113.7)
- moved J9 24.3 mm to (136.0, 63.4), turned to 90 degrees
- moved C1 20.6 mm to (118.7, 96.3)
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Connections:
- net +3V3 renamed +3.3V
- net Net-(R1-Pad2) renamed /ESP1/CS_EN
- net Net-(U2-Pad10) renamed /ESP1/CS_A3
- net Net-(U2-Pad16) renamed /ESP1/CS_A0
- net Net-(U2-Pad17) renamed /ESP1/CS_A1
- net Net-(U2-Pad20) renamed /ESP1/CS_A2
- J1 pad 2: Net-(J1-Pad2) -> unconnected-(J1-Pin_2-Pad2)
- J1 pad 9: Net-(J1-Pad9) -> unconnected-(J1-Pin_9-Pad9)
- J2 pad 11: /ESP1/MISO -> /ESP1/MISO_1
- J2 pad 13: /ESP1/SCLK -> /ESP1/SCLK_1
- J2 pad 9: /ESP1/MOSI -> /ESP1/MOSI_1
- J3 pad 11: /ESP1/MISO -> /ESP1/MISO_2
- J3 pad 13: /ESP1/SCLK -> /ESP1/SCLK_2
- J3 pad 9: /ESP1/MOSI -> /ESP1/MOSI_2
- J4 pad 11: /ESP1/MISO -> /ESP1/MISO_3
- J4 pad 13: /ESP1/SCLK -> /ESP1/SCLK_3
- J4 pad 9: /ESP1/MOSI -> /ESP1/MOSI_3
- J5 pad 11: /ESP1/MISO -> /ESP1/MISO_4
- J5 pad 13: /ESP1/SCLK -> /ESP1/SCLK_4
- J5 pad 9: /ESP1/MOSI -> /ESP1/MOSI_4
- J6 pad 11: /ESP1/MISO -> /ESP1/MISO_5
- J6 pad 13: /ESP1/SCLK -> /ESP1/SCLK_5
- J6 pad 9: /ESP1/MOSI -> /ESP1/MOSI_5
- J7 pad 11: /ESP1/MISO -> /ESP1/MISO_6
- J7 pad 13: /ESP1/SCLK -> /ESP1/SCLK_6
- J7 pad 9: /ESP1/MOSI -> /ESP1/MOSI_6
- U1 pad 10: /ESP1/IRQ_6 -> Net-(U17-O6b)
- U1 pad 11: /ESP1/IRQ_3 -> Net-(U15-O5b)
- U1 pad 12: /ESP1/IRQ_4 -> Net-(U15-O6b)
- U1 pad 4: /ESP1/IRQ_2 -> Net-(U13-O6b)
- U1 pad 5: /ESP1/IRQ_1 -> Net-(U13-O5b)
- U1 pad 9: /ESP1/IRQ_5 -> Net-(U17-O5b)
- U2 pad 14: Net-(U2-Pad14) -> unconnected-(U2-GPIO34/BUT1-Pad14)
- U2 pad 2: Net-(U2-Pad2) -> unconnected-(U2-3.3V-Pad2)
- U2 pad 4: Net-(U2-Pad4) -> unconnected-(U2-ESP_EN-Pad4)
- U2 pad 6: Net-(U2-Pad6) -> unconnected-(U2-GPIO1/U0TXD-Pad6)
- U2 pad 8: Net-(U2-Pad8) -> unconnected-(U2-GPIO3/U0RXD-Pad8)
- U3 pad 11: /ESP1/IRQ_7 -> Net-(U7-O5b)
- U3 pad 12: /ESP1/IRQ_8 -> Net-(U7-O6b)
- U3 pad 2: /ESP1/IRQ_12 -> Net-(U11-O6b)
- U3 pad 3: /ESP1/IRQ_11 -> Net-(U11-O5b)
- U3 pad 4: /ESP1/IRQ_9 -> Net-(U9-O5b)
- U3 pad 5: /ESP1/IRQ_10 -> Net-(U9-O6b)
- U4 pad 1: /ESP1/~{CS_1} -> Net-(U4-S0)
- U4 pad 10: /ESP1/~{CS_10} -> Net-(U4-S9)
- U4 pad 11: /ESP1/~{CS_11} -> Net-(U4-S10)
- U4 pad 13: /ESP1/~{CS_12} -> Net-(U4-S11)
- U4 pad 2: /ESP1/~{CS_2} -> Net-(U4-S1)
- U4 pad 3: /ESP1/~{CS_3} -> Net-(U4-S2)
- U4 pad 4: /ESP1/~{CS_4} -> Net-(U4-S3)
- U4 pad 5: /ESP1/~{CS_5} -> Net-(U4-S4)
- U4 pad 6: /ESP1/~{CS_6} -> Net-(U4-S5)
- U4 pad 7: /ESP1/~{CS_7} -> Net-(U4-S6)
- U4 pad 8: /ESP1/~{CS_8} -> Net-(U4-S7)
- U4 pad 9: /ESP1/~{CS_9} -> Net-(U4-S8)
- U5 pad 4: Net-(U5-Pad4) -> unconnected-(U5-On/~{Off}-Pad4)
- U6 pad 4: Net-(U6-Pad4) -> unconnected-(U6-On/~{Off}-Pad4)
Routing:
- net +5V: track 285.5 -> 32.1 mm
- net /ESP1/MOSI: track 115.5 -> 226.6 mm, vias 1 -> 6
- net /ESP1/SCLK: track 103.4 -> 207.3 mm, vias 0 -> 7
- net Net-(J8-Pin_2): track 103.8 -> 0.00 mm
- net Net-(J11-Pin_4): track 99.0 -> 0.00 mm
- net Net-(J11-Pin_3): track 94.7 -> 0.00 mm
- net /ESP1/MISO: track 127.1 -> 212.0 mm, vias 0 -> 8
- net /ESP1/~{CS_2}: track 67.1 -> 4.52 mm
- net /ESP1/~{CS_1}: track 64.8 -> 4.25 mm
- net Net-(R2-Pad2): track 62.4 -> 2.18 mm, vias 2 -> 0
- net /ESP1/~{CS_4}: track 55.7 -> 4.52 mm
- net /ESP1/~{CS_3}: track 53.8 -> 4.26 mm
- net Net-(U13-O6b): track 0.00 -> 49.1 mm
- net Net-(U13-O5b): track 0.00 -> 47.8 mm
- net /ESP1/~{CS_8}: track 49.5 -> 4.52 mm
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Other:
- board text added: "J2"
- board text added: "U14"

Commit message: Blerp.
Parts:
- added D11: LED, custom:CHIPLED_0603, F.Cu at (42.7, 97.5)
- added D12: LED, custom:CHIPLED_0603, F.Cu at (42.7, 99.4)
- added D13: LED, custom:CHIPLED_0603, F.Cu at (42.7, 101.3)
- added D14: LED, custom:CHIPLED_0603, F.Cu at (42.7, 103.2)
- added D15: LED, custom:CHIPLED_0603, F.Cu at (42.7, 105.1)
- added D16: LED, custom:CHIPLED_0603, F.Cu at (42.7, 107.0)
- added D17: LED, custom:CHIPLED_0603, F.Cu at (42.7, 86.0)
- added D18: LED, custom:CHIPLED_0603, F.Cu at (42.7, 87.9)
- added D19: LED, custom:CHIPLED_0603, F.Cu at (42.7, 89.8)
- added D20: LED, custom:CHIPLED_0603, F.Cu at (42.7, 91.7)
- added D21: LED, custom:CHIPLED_0603, F.Cu at (42.7, 93.6)
- added D22: LED, custom:CHIPLED_0603, F.Cu at (42.7, 95.5)
- added R10: 1K, Resistor_SMD:R_0603_1608Metric, F.Cu at (52.1, 99.4)
- added R11: 1K, Resistor_SMD:R_0603_1608Metric, F.Cu at (52.1, 101.3)
- added R12: 1K, Resistor_SMD:R_0603_1608Metric, F.Cu at (52.1, 103.2)
- added R32: 1K, Resistor_SMD:R_0603_1608Metric, F.Cu at (52.1, 105.1)
- added R33: 1K, Resistor_SMD:R_0603_1608Metric, F.Cu at (52.1, 107.0)
- added R36: 1K, Resistor_SMD:R_0603_1608Metric, F.Cu at (52.1, 86.0)
- added R37: 1K, Resistor_SMD:R_0603_1608Metric, F.Cu at (52.1, 87.9)
- added R38: 1K, Resistor_SMD:R_0603_1608Metric, F.Cu at (52.1, 89.8)
- added R39: 1K, Resistor_SMD:R_0603_1608Metric, F.Cu at (52.1, 91.7)
- added R54: 1K, Resistor_SMD:R_0603_1608Metric, F.Cu at (52.1, 93.6)
- added R55: 1K, Resistor_SMD:R_0603_1608Metric, F.Cu at (52.1, 95.5)
- added R9: 1K, Resistor_SMD:R_0603_1608Metric, F.Cu at (52.1, 97.5)
- moved R13 58.7 mm to (72.4, 133.3), turned to 180 degrees
- moved R14 58.7 mm to (72.4, 130.8), turned to 180 degrees
- moved R15 54.3 mm to (78.7, 118.9), turned to -90 degrees
- moved C3 50.5 mm to (90.8, 81.0), turned to 90 degrees
- moved R6 39.4 mm to (78.7, 114.9), turned to -90 degrees
- moved R29 37.2 mm to (54.0, 136.8), turned to -90 degrees
- moved R4 33.7 mm to (54.3, 123.3), turned to 180 degrees
- moved R5 31.4 mm to (54.3, 128.3)
- moved R26 26.3 mm to (59.0, 129.2)
- moved R27 26.1 mm to (59.0, 127.0)
- moved R28 26.1 mm to (59.0, 125.1)
- moved D3 22.9 mm to (42.7, 128.9)
- moved D4 22.9 mm to (42.7, 127.0)
- moved D5 22.9 mm to (42.7, 125.1)
- moved D6 22.9 mm to (42.7, 123.2)
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Connections:
- net Net-(J11-Pin_3) renamed /ESP1/I2C_SCL
- net Net-(J11-Pin_4) renamed /ESP1/I2C_SDA
- net Net-(U4-S12) renamed /ESP1/C13
- net Net-(U4-S13) renamed /ESP1/C14
- net Net-(U4-S14) renamed /ESP1/C15
- net Net-(U4-S15) renamed /ESP1/C16
- net Net-(U4-S2) renamed /ESP1/~{CS_3_R}
- net Net-(U4-S3) renamed /ESP1/~{CS_4_R}
- net Net-(U4-S8) renamed /ESP1/~{CS_9_R}
- net Net-(U4-S9) renamed /ESP1/~{CS_10_R}
- J8 pad 2: Net-(J8-Pin_2) -> /ESP1/1WIRE
- J9 pad 2: Net-(J8-Pin_2) -> /ESP1/1WIRE
- R16 pad 1: Net-(U4-S0) -> /ESP1/~{CS_1}
- R17 pad 1: Net-(U4-S1) -> /ESP1/~{CS_2}
- R2 pad 1: Net-(U2-GPIO36/U1RXD) -> Net-(U2-GPIO33)
- R20 pad 1: Net-(U4-S4) -> /ESP1/~{CS_5_R}
- R21 pad 1: Net-(U4-S5) -> /ESP1/~{CS_6_R}
- R22 pad 1: Net-(U4-S6) -> /ESP1/~{CS_7_R}
- R23 pad 1: Net-(U4-S7) -> /ESP1/~{CS_8_R}
- R30 pad 1: Net-(U4-S10) -> /ESP1/~{CS_11_R}
- R31 pad 1: Net-(U4-S11) -> /ESP1/~{CS_12_R}
- R6 pad 2: Net-(J8-Pin_2) -> /ESP1/1WIRE
- U10 pad 1: Net-(U4-S7) -> /ESP1/~{CS_8_R}
- U10 pad 2: Net-(U4-S6) -> /ESP1/~{CS_7_R}
- U14 pad 1: Net-(U4-S1) -> /ESP1/~{CS_2}
- U14 pad 2: Net-(U4-S0) -> /ESP1/~{CS_1}
- U18 pad 1: Net-(U4-S5) -> /ESP1/~{CS_6_R}
- U18 pad 2: Net-(U4-S4) -> /ESP1/~{CS_5_R}
- U2 pad 12: Net-(U2-GPIO36/U1RXD) -> /ESP1/1WIRE
- U2 pad 15: Net-(J8-Pin_2) -> Net-(U2-GPIO33)
- U4 pad 1: Net-(U4-S0) -> /ESP1/~{CS_5_R}
- U4 pad 11: Net-(U4-S10) -> /ESP1/~{CS_7_R}
- U4 pad 13: Net-(U4-S11) -> /ESP1/~{CS_8_R}
- U4 pad 2: Net-(U4-S1) -> /ESP1/~{CS_6_R}
- U4 pad 5: Net-(U4-S4) -> /ESP1/~{CS_1}
- U4 pad 6: Net-(U4-S5) -> /ESP1/~{CS_2}
- U4 pad 7: Net-(U4-S6) -> /ESP1/~{CS_11_R}
- U4 pad 8: Net-(U4-S7) -> /ESP1/~{CS_12_R}
- U8 pad 1: Net-(U4-S11) -> /ESP1/~{CS_12_R}
- U8 pad 2: Net-(U4-S10) -> /ESP1/~{CS_11_R}
Routing:
- net +5V: track 32.1 -> 330.0 mm, vias 0 -> 2
- net /ESP1/~{CS_1}: track 4.25 -> 115.0 mm, vias 0 -> 3
- net /ESP1/I2C_SCL: track 0.00 -> 109.4 mm, vias 0 -> 1
- net /ESP1/1WIRE: track 0.00 -> 108.3 mm, vias 0 -> 1
- net /ESP1/~{CS_2}: track 4.52 -> 111.9 mm, vias 0 -> 3
- net /ESP1/I2C_SDA: track 0.00 -> 107.2 mm, vias 0 -> 1
- net /ESP1/~{CS_3_R}: track 6.91 -> 100.2 mm, vias 1 -> 3
- net /ESP1/~{CS_4_R}: track 6.13 -> 96.3 mm, vias 1 -> 3
- net /ESP1/~{CS_8_R}: track 0.00 -> 89.4 mm, vias 0 -> 1
- net /ESP1/~{CS_7_R}: track 0.00 -> 84.1 mm, vias 0 -> 3
- net /ESP1/~{CS_5_R}: track 0.00 -> 81.2 mm, vias 0 -> 3
- net /ESP1/~{CS_6_R}: track 0.00 -> 77.3 mm, vias 0 -> 3
- net GND: track 94.9 -> 168.2 mm, vias 34 -> 56
- net /ESP1/~{CS_9_R}: track 6.91 -> 72.2 mm, vias 1 -> 3
- net /ESP1/~{CS_10_R}: track 6.13 -> 69.2 mm, vias 1 -> 3
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Other:
- outline, holes or cut-outs redrawn
- board text added: "3V3 3V3 IRQ_1 IRQ_2 MOSI MISO SCLK"
- board text added: "3V3 3V3 IRQ_11 IRQ_12 MOSI MISO SCLK"
- board text added: "3V3 3V3 IRQ_3 IRQ_4 MOSI MISO SCLK"
- board text added: "3V3 3V3 IRQ_5 IRQ_6 MOSI MISO SCLK"
- board text added: "3V3 3V3 IRQ_7 IRQ_8 MOSI MISO SCLK"
- board text added: "3V3 3V3 IRQ_9 IRQ_10 MOSI MISO SCLK"
- board text added: "3V3 5V"
- board text added: "5V 3V3 SIG GND"
- board text added: "5V CS1 CS2 GND GND GND GND"
- board text added: "5V CS11 CS12 GND GND GND GND"
- board text added: "5V CS3 CS4 GND GND GND GND"
- board text added: "5V CS5 CS6 GND GND GND GND"
- board text added: "5V CS7 CS8 GND GND GND GND"
- board text added: "5V CS9 CS10 GND GND GND GND"
- board text added: "A3 A2 A1 A0"
- board text added: "C13 C14 C15 C16"
- board text added: "CS11 CS12 CS9 CS10 CS7 CS8 CS5 CS6 CS3 CS4 CS1 CS2"
- board text added: "Energy Monitor CPU PCB"
- board text added: "GND SDA SCL 3V3 5V"
- board text added: "NC 9V GND 9V GND 9V GND 9V NC 9V"
- board text added: "R1, C. Wolf"
- board text added: "SDA SCL GND 5V"
- board text removed: "J2"
