File: ESP/Multi-PZEM/PZEM-Single R1/PZEM-Single R1.kicad_pcb (KiCad board)
At the start: 2 copper layers, 60 x 97 mm, 18 parts, among them J1 Conn_01x04, J3 Conn_01x02, J4 Conn_01x04, U2 AMS1117-3.3, U4 ESP32-WROOM-32

Commit message: Boards!
Parts:
- added C3: C_Small, Capacitor_SMD:C_1206_3216Metric_Pad1.33x1.80mm_HandSolder, F.Cu at (11.5, -56.0)
- added C4: C_Small, Capacitor_SMD:C_1206_3216Metric_Pad1.33x1.80mm_HandSolder, F.Cu at (4.00, -50.5)
- added R3: R_Small, Resistor_SMD:R_1206_3216Metric_Pad1.30x1.75mm_HandSolder, F.Cu at (13.0, -62.5)
- C1: footprint Capacitor_THT:CP_Radial_D8.0mm_P2.50mm -> Capacitor_Tantalum_SMD:CP_EIA-7343-40_Kemet-Y
- R1, R2, R5: footprint Resistor_THT:R_Axial_DIN0207_L6.3mm_D2.5mm_P10.16mm_Horizontal -> Resistor_SMD:R_1206_3216Metric_Pad1.30x1.75mm_HandSolder
- moved J4 15.0 mm to (27.0, -93.0)
- moved R1 11.5 mm to (14.6, -88.0)
- moved U2 6.09 mm to (5.35, -55.7)
- moved C1 4.95 mm to (5.50, -62.5), turned to 180 degrees
- moved R2 3.65 mm to (21.0, -88.0), turned to 0 degrees
- moved C2 2.68 mm to (17.1, -51.2), turned to -90 degrees
- moved R5 2.00 mm to (37.0, -91.0), turned to -90 degrees
- moved U4 1.13 mm to (9.67, -75.8)
- moved D2 1.06 mm to (19.5, -91.2), turned to 90 degrees
- moved D1 0.58 mm to (13.0, -91.2), turned to 90 degrees
Connections:
- U3 pad 3: GND -> +5V
- U3 pad 4: +5V -> GND
- U4 pad 10: Net-(J4-Pin_1) -> unconnected-(U4-IO25-Pad10)
- U4 pad 12: unconnected-(U4-IO27-Pad12) -> Net-(U1-RX)
- U4 pad 14: unconnected-(U4-IO12-Pad14) -> Net-(U1-TX)
- U4 pad 16: unconnected-(U4-IO13-Pad16) -> Net-(U1-CF)
- U4 pad 27: Net-(U1-CF) -> Net-(J4-Pin_1)
- U4 pad 28: Net-(U1-TX) -> unconnected-(U4-IO17-Pad28)
- U4 pad 3: unconnected-(U4-EN-Pad3) -> Net-(U4-EN)
- U4 pad 30: Net-(U1-RX) -> unconnected-(U4-IO18-Pad30)
- U4 pad 36: unconnected-(U4-IO22-Pad36) -> Net-(D2-A)
- U4 pad 8: Net-(D2-A) -> unconnected-(U4-IO32-Pad8)
Routing:
- net GND: track 12.1 -> 138.3 mm, vias 2 -> 4
- net +3V3: track 14.8 -> 120.0 mm, vias 2 -> 1
- net Net-(U1-RX): track 0.00 -> 40.0 mm
- net +5V: track 4.06 -> 43.1 mm
- net Net-(U1-TX): track 0.00 -> 32.5 mm
- net Net-(U1-CF): track 0.00 -> 27.0 mm
- net Net-(U4-EN): track 0.00 -> 14.3 mm
- net Net-(D2-A): track 10.7 -> 23.2 mm
- net Net-(D1-K): track 12.2 -> 3.22 mm
- net Net-(J4-Pin_1): track 34.9 -> 31.1 mm
- net unconnected-(U4-IO32-Pad8): track 0.00 -> 2.46 mm, vias 0 -> 1
- net unconnected-(U4-IO25-Pad10): track 0.00 -> 2.46 mm, vias 0 -> 1
- net Net-(D2-K): track 3.84 -> 3.25 mm
- removed copper zone on B.Cu, net GND
Other:
- outline, holes or cut-outs redrawn
