File: ESP/Water Meter Analog - R1/Water Meter Analog - R1.kicad_sch (KiCad schematic)
At the start: 33 parts, among them J1 Conn_01x04, J2 Conn_01x04, J3 Conn_01x02, J4 Conn_01x04, U1 LF33_TO220, U2 LM393, U4 ESP32-WROOM-32, U5 LF33_TO220

Commit message: Boards!
Parts:
- added U3: DS18B20, Package_TO_SOT_THT:TO-92_Inline_Wide, symbol Sensor_Temperature:DS18B20
- R4: footprint Resistor_THT:R_Axial_DIN0207_L6.3mm_D2.5mm_P10.16mm_Horizontal -> Resistor_THT:R_Axial_DIN0207_L6.3mm_D2.5mm_P7.62mm_Horizontal
Connections:
- net +3V3: now also U3.3 (V_{DD})
- net GND: now also U3.1 (GND)
- net at J4.1 (Pin_1), R5.2, U4.10 (IO25): now also U3.2 (DQ)
Changed lines of the file:
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@@
   (junction (at 45.72 36.83) (diameter 0) (color 0 0 0 0)
   )
+  (junction (at 96.52 158.75) (diameter 0) (color 0 0 0 0)
+  )
   (junction (at 76.2 36.83) (diameter 0) (color 0 0 0 0)
   )
@@
   (junction (at 80.01 36.83) (diameter 0) (color 0 0 0 0)
   )
+  (junction (at 74.93 147.32) (diameter 0) (color 0 0 0 0)
+  )
   (junction (at 218.44 135.89) (diameter 0) (color 0 0 0 0)
   )
@@
     (stroke (width 0) (type default))
   )
+  (wire (pts (xy 110.49 147.32) (xy 110.49 151.13))
+    (stroke (width 0) (type default))
+  )
   (wire (pts (xy 116.84 120.65) (xy 116.84 121.92))
     (stroke (width 0) (type default))
@@
     (stroke (width 0) (type default))
   )
+  (wire (pts (xy 81.28 147.32) (xy 81.28 149.86))
+    (stroke (width 0) (type default))
+  )
   (wire (pts (xy 119.38 83.82) (xy 116.84 83.82))
     (stroke (width 0) (type default))
@@
     (stroke (width 0) (type default))
   )
-  (wire (pts (xy 81.28 147.32) (xy 81.28 149.86))
+  (wire (pts (xy 81.28 147.32) (xy 110.49 147.32))
     (stroke (width 0) (type default))
   )
@@
   )
   (wire (pts (xy 262.89 147.32) (xy 262.89 146.05))
+    (stroke (width 0) (type default))
+  )
+  (wire (pts (xy 96.52 158.75) (xy 102.87 158.75))
     (stroke (width 0) (type default))
   )
@@
       (effects (font (size 1.27 1.27)) (justify left) hide)
     )
-    (property "Footprint" "Resistor_THT:R_Axial_DIN0207_L6.3mm_D2.5mm_P10.16mm_Horizontal" (at 220.98 92.71 0)
+    (property "Footprint" "Resistor_THT:R_Axial_DIN0207_L6.3mm_D2.5mm_P7.62mm_Horizontal" (at 220.98 92.71 0)
       (effects (font (size 1.27 1.27)) hide)
     )
@@
     )
   )
+  (symbol (lib_id "power:GND") (at 110.49 166.37 0) (unit 1)
+    (in_bom yes) (on_board yes) (dnp no)
+    (property "Reference" "#PWR031" (at 110.49 172.72 0)
+      (effects (font (size 1.27 1.27)) hide)
+    )
+    (property "Value" "GND" (at 110.617 170.7642 0)
+      (effects (font (size 1.27 1.27)))
+    )
+    (property "Footprint" "" (at 110.49 166.37 0)
+      (effects (font (size 1.27 1.27)) hide)
+    )
+    (property "Datasheet" "" (at 110.49 166.37 0)
+      (effects (font (size 1.27 1.27)) hide)
+    )
+    (pin "1")
+    (instances
+      (project "Water Meter Analog - R1"
+        (path "/16cc9b8c-fde0-4c98-881a-85837ff5aa29"
+          (reference "#PWR031") (unit 1)
+        )
+      )
+    )
+  )
   (symbol (lib_id "power:GND") (at 262.89 147.32 0) (unit 1)
     (in_bom yes) (on_board yes) (dnp no)
@@
     )
   )
-  (symbol (lib_id "power:+3V3") (at 81.28 147.32 0) (unit 1)
-    (in_bom yes) (on_board yes) (dnp no)
-    (property "Reference" "#PWR08" (at 81.28 151.13 0)
-      (effects (font (size 1.27 1.27)) hide)
-    )
-    (property "Value" "+3V3" (at 81.661 142.9258 0)
-      (effects (font (size 1.27 1.27)))
-    )
-    (property "Footprint" "" (at 81.28 147.32 0)
-      (effects (font (size 1.27 1.27)) hide)
-    )
-    (property "Datasheet" "" (at 81.28 147.32 0)
+  (symbol (lib_id "power:+3V3") (at 74.93 147.32 0) (unit 1)
+    (in_bom yes) (on_board yes) (dnp no)
+    (property "Reference" "#PWR08" (at 74.93 151.13 0)
+      (effects (font (size 1.27 1.27)) hide)
+    )
+    (property "Value" "+3V3" (at 75.311 142.9258 0)
+      (effects (font (size 1.27 1.27)))
+    )
+    (property "Footprint" "" (at 74.93 147.32 0)
+      (effects (font (size 1.27 1.27)) hide)
+    )
+    (property "Datasheet" "" (at 74.93 147.32 0)
       (effects (font (size 1.27 1.27)) hide)
     )
@@
         )
       )
+    )
+  )
+  (symbol (lib_id "Sensor_Temperature:DS18B20") (at 110.49 158.75 0) (mirror y) (unit 1)
+    (in_bom yes) (on_board yes) (dnp no)
+    (property "Reference" "U3" (at 116.3319 157.5379 0)
+      (effects (font (size 1.27 1.27)) (justify right))
+    )
+    (property "Value" "DS18B20" (at 116.3319 159.9621 0)
+      (effects (font (size 1.27 1.27)) (justify right))
+    )
+    (property "Footprint" "Package_TO_SOT_THT:TO-92_Inline_Wide" (at 135.89 165.1 0)
+      (effects (font (size 1.27 1.27)) hide)
+    )
+    (property "Datasheet" "http://datasheets.maximintegrated.com/en/ds/DS18B20.pdf" (at 114.3 152.4 0)
+      (effects (font (size 1.27 1.27)) hide)
+    )
+    (pin "1")
+    (pin "2")
+    (pin "3")
+    (instances
+      (project "Water Meter Analog - R1"
+        (path "/16cc9b8c-fde0-4c98-881a-85837ff5aa29"
+          (reference "U3") (unit 1)
+        )
+      )
