File: ESP/Water Meter Analog - R2/Water Meter Analog - R2.kicad_pcb (KiCad board)
At the start: 2 copper layers, 60 x 63.2 mm, 34 parts, among them J1 Conn_01x04, J2 Conn_01x04, J3 Conn_01x02, J4 Conn_01x04, U1 LF33_TO220, U2 LM393, U3 DS18B20, U4 ESP32-WROOM-32, U5 LF33_TO220

Commit message: Boards!
Parts:
- removed C3, C6, C7: C_Small, Capacitor_SMD:C_1206_3216Metric_Pad1.33x1.80mm_HandSolder
- removed D3: LED, LED_THT:LED_D5.0mm
- removed J2: Conn_01x04, Connector_JST:JST_XH_B3B-XH-A_1x03_P2.50mm_Vertical
- removed R8: R_Small, Resistor_THT:R_Axial_DIN0207_L6.3mm_D2.5mm_P10.16mm_Horizontal
- removed R9: R_Small, Resistor_THT:R_Axial_DIN0309_L9.0mm_D3.2mm_P2.54mm_Vertical
- removed RV1, RV2: R_Potentiometer, Potentiometer_THT:Potentiometer_Bourns_3299Y_Vertical
- removed U2: LM393, Package_SO:SO-8_5.3x6.2mm_P1.27mm
- J1: footprint Connector_JST:JST_XH_B6B-XH-A_1x06_P2.50mm_Vertical -> Connector_JST:JST_XH_B8B-XH-A_1x08_P2.50mm_Vertical
- R4: footprint Resistor_THT:R_Axial_DIN0207_L6.3mm_D2.5mm_P7.62mm_Horizontal -> Resistor_THT:R_Axial_DIN0207_L6.3mm_D2.5mm_P10.16mm_Horizontal
- moved R4 25.4 mm to (31.0, -58.8), turned to 90 degrees
- moved R6 20.7 mm to (34.5, -58.9), turned to 90 degrees
- moved J1 16.6 mm to (42.0, -55.5)
- moved R7 15.3 mm to (37.5, -59.0), turned to 90 degrees
- moved J4 13.5 mm to (42.0, -79.5), turned to 90 degrees
- moved H3 13.0 mm to (43.0, -38.0)
- moved H4 13.0 mm to (43.0, -93.0)
- moved U3 12.5 mm to (34.0, -81.0), turned to 90 degrees
- moved C4 3.62 mm to (31.5, -51.0), turned to 90 degrees
- moved C2 2.24 mm to (13.5, -43.5)
Connections:
- J1 pad 1: +3V3 -> GND
- J1 pad 2: Net-(J1-Pin_2) -> +5V
- J1 pad 3: Net-(J1-Pin_3) -> +3V3
- J1 pad 6: GND -> Net-(J1-Pin_6)
- R4 pad 1: Net-(R4-Pad1) -> +3V3
- R4 pad 2: Net-(J2-Pin_2) -> Net-(J1-Pin_4)
- R6 pad 1: Net-(D3-K) -> +3V3
- R6 pad 2: Net-(U4-IO15) -> Net-(J1-Pin_5)
- R7 pad 1: Net-(U4-IO15) -> +3V3
- R7 pad 2: Net-(U2A-+) -> Net-(J1-Pin_6)
- U4 pad 23: Net-(U4-IO15) -> unconnected-(U4-IO15-Pad23)
- U4 pad 27: Net-(J1-Pin_5) -> Net-(J1-Pin_7)
- U4 pad 28: Net-(J1-Pin_4) -> Net-(J1-Pin_6)
- U4 pad 30: Net-(J1-Pin_3) -> Net-(J1-Pin_5)
- U4 pad 31: Net-(J1-Pin_2) -> Net-(J1-Pin_4)
- U4 pad 4: Net-(U4-SENSOR_VP) -> unconnected-(U4-SENSOR_VP-Pad4)
Routing:
- net Net-(J1-Pin_2): track 53.0 -> 0.00 mm
- net Net-(J1-Pin_3): track 50.5 -> 0.00 mm
- net +3V3: track 162.4 -> 124.9 mm, vias 4 -> 2
- net Net-(U4-SENSOR_VP): track 36.5 -> 0.00 mm
- net Net-(J1-Pin_6): track 0.00 -> 34.7 mm
- net Net-(U4-IO15): track 34.5 -> 0.00 mm
- net Net-(J1-Pin_7): track 0.00 -> 32.9 mm
- net Net-(J2-Pin_2): track 32.3 -> 0.00 mm
- net +5V: track 97.7 -> 71.4 mm
- net Net-(C7-Pad2): track 13.6 -> 0.00 mm
- net GND: track 155.1 -> 141.9 mm, vias 14 -> 6
- net Net-(J4-Pin_1): track 45.4 -> 35.2 mm
- net Net-(J1-Pin_4): track 48.4 -> 38.4 mm
- net Net-(J1-Pin_5): track 47.7 -> 37.9 mm
- net Net-(U2A-+): track 9.37 -> 0.00 mm
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Other:
- board size 60 x 63.2 mm -> 47 x 63.2 mm
