File: ESP/Water Meter Analog - R2/Water Meter Analog - R2.kicad_sch (KiCad schematic)
At the start: 21 parts, among them J1 Conn_01x04, J3 Conn_01x02, J4 Conn_01x04, U2 AMS1117-3.3, U4 ESP32-WROOM-32

Commit message: Boards!
Parts:
- removed C2: CP, Capacitor_THT:CP_Radial_D10.0mm_P2.50mm_P5.00mm, symbol Device:C_Polarized
- removed C3, C4: C_Small, Capacitor_SMD:C_1206_3216Metric_Pad1.33x1.80mm_HandSolder, symbol Device:C_Small
- removed J1: Conn_01x04, Connector_JST:JST_XH_B2B-XH-A_1x02_P2.50mm_Vertical, symbol Connector_Generic:Conn_01x02
- removed U1: ~, custom:PZEM-004T-100A-D-P, symbol custom:PZEM-004T-100A-D-P
- removed U2: AMS1117-3.3, Package_TO_SOT_SMD:SOT-223-3_TabPin2, symbol Regulator_Linear:AMS1117-3.3
- removed U3: ~, custom:HLK-PM01, symbol custom:HLK-PM01
- added C2, C5: CP, Capacitor_THT:CP_Radial_D8.0mm_P2.50mm, symbol Device:CP
- added C4: CP, Capacitor_THT:CP_Radial_D10.0mm_P2.50mm_P5.00mm, symbol Device:C_Polarized
- added J1: Conn_01x04, Connector_JST:JST_XH_B8B-XH-A_1x08_P2.50mm_Vertical, symbol Connector_Generic:Conn_01x08
- added R4, R6, R7: R_Small, Resistor_THT:R_Axial_DIN0207_L6.3mm_D2.5mm_P10.16mm_Horizontal, symbol Device:R_Small
- added U1, U5: LF33_TO220, Package_TO_SOT_THT:TO-220-3_Vertical, symbol Regulator_Linear:LF33_TO220
- added U3: DS18B20, Package_TO_SOT_THT:TO-92_Inline_Wide, symbol Sensor_Temperature:DS18B20
- C1: footprint Capacitor_Tantalum_SMD:CP_EIA-7343-40_Kemet-Y -> Capacitor_THT:CP_Radial_D8.0mm_P2.50mm
- R1, R2, R5: footprint Resistor_SMD:R_1206_3216Metric_Pad1.30x1.75mm_HandSolder -> Resistor_THT:R_Axial_DIN0207_L6.3mm_D2.5mm_P10.16mm_Horizontal
- R3: footprint Resistor_SMD:R_1206_3216Metric_Pad1.30x1.75mm_HandSolder -> Resistor_THT:R_Axial_DIN0309_L9.0mm_D3.2mm_P2.54mm_Vertical
Connections:
- net +3V3: now also J4.2 (Pin_2), R3.2, J1.3 (Pin_3), R4.1, R6.1, R7.1, U3.3 (V_{DD}), U5.3 (VO); no longer J4.3 (Pin_3), R3.1
- net +5V: now also C2.1, C5.1, J1.2 (Pin_2), U1.3 (VO), U5.1 (VI)
- net GND: now also J3.2 (Pin_2), J4.3 (Pin_3), C2.2, C4.2, C5.2, J1.1 (Pin_1), J1.8 (Pin_8), U1.2 (GND), U3.1 (GND), U5.2 (GND); no longer J4.2 (Pin_2)
- net at U4.3 (EN): now also R3.1; no longer R3.2
- net at J3.1 (Pin_1): now also C4.1, U1.1 (VI)
- net at J4.1 (Pin_1), R5.2: now also U4.10 (IO25), U3.2 (DQ); no longer U4.27 (IO16)
- net at U4.28 (IO17): now also J1.6 (Pin_6), R7.2
- net at U4.30 (IO18): now also J1.5 (Pin_5), R6.2
- net at U4.31 (IO19): now also J1.4 (Pin_4), R4.2
- net at U4.36 (IO22): no longer D2.2 (A)
- net at U4.8 (IO32): now also D2.2 (A)
- new net: J1.7 (Pin_7), U4.27 (IO16)
Other:
- moved on the sheet: C1, J3
