File: misc/PWMMapper/R4-Kicad/PWMMapper R4.kicad_sch (KiCad schematic)
At the start: 46 parts, among them J1 Conn_01x04, J2 Conn_01x04, J3 Conn_01x04, J4 Conn_01x04, J5 Conn_01x04, J6 Conn_01x04, P1 Header 3, P6 Header 3, U1 ATTiny1616-MFR, U2 TPS70950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

Commit message: So many bits and bobs.
Parts:
- added H1, H2: MountingHole, MountingHole:MountingHole_3.2mm_M3_Pad_Via, symbol Mechanical:MountingHole
Changed lines of the file:
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@@
+    )
+  )
+  (symbol (lib_id "Mechanical:MountingHole") (at 229.87 17.78 0) (unit 1)
+    (in_bom yes) (on_board yes) (dnp no) (fields_autoplaced)
+    (property "Reference" "H2" (at 232.41 16.5679 0)
+      (effects (font (size 1.27 1.27)) (justify left))
+    )
+    (property "Value" "MountingHole" (at 232.41 18.9921 0)
+      (effects (font (size 1.27 1.27)) (justify left))
+    )
+    (property "Footprint" "MountingHole:MountingHole_3.2mm_M3_Pad_Via" (at 229.87 17.78 0)
+      (effects (font (size 1.27 1.27)) hide)
+    )
+    (property "Datasheet" "~" (at 229.87 17.78 0)
+      (effects (font (size 1.27 1.27)) hide)
+    )
+    (instances
+      (project "PWMMapper R4"
+        (path "/10232e0b-ad50-41f9-9b8d-558c674a4395"
+          (reference "H2") (unit 1)
+        )
+      )
     )
   )
@@
         )
       )
+    )
+  )
+  (symbol (lib_id "Mechanical:MountingHole") (at 229.87 11.43 0) (unit 1)
+    (in_bom yes) (on_board yes) (dnp no) (fields_autoplaced)
+    (property "Reference" "H1" (at 232.41 10.2179 0)
+      (effects (font (size 1.27 1.27)) (justify left))
+    )
+    (property "Value" "MountingHole" (at 232.41 12.6421 0)
+      (effects (font (size 1.27 1.27)) (justify left))
+    )
+    (property "Footprint" "MountingHole:MountingHole_3.2mm_M3_Pad_Via" (at 229.87 11.43 0)
+      (effects (font (size 1.27 1.27)) hide)
+    )
+    (property "Datasheet" "~" (at 229.87 11.43 0)
+      (effects (font (size 1.27 1.27)) hide)
+    )
+    (instances
+      (project "PWMMapper R4"
+        (path "/10232e0b-ad50-41f9-9b8d-558c674a4395"
+          (reference "H1") (unit 1)
+        )
+      )
