File: ESP/Multi-PZEM/PZEM-Single Ultra-Compact LPKF - R1/PZEM-Single LPKF - R2.kicad_pcb (KiCad board)
At the start: 2 copper layers, 30 x 95 mm, 10 parts, among them J1 Conn_01x02, U4 SEEEDUINO-XIAO-ESP32C3

Commit message: Ordered stuff!
Parts:
- added J2: Conn_01x04_Pin, Connector_JST:JST_XH_B4B-XH-A_1x04_P2.50mm_Vertical, F.Cu at (46.5, -90.5)
- H1, H2, H3, H4: footprint MountingHole:MountingHole_3.2mm_M3_Pad_Via -> MountingHole:MountingHole_3.2mm_M3_Pad
- moved C2 0.55 mm to (33.2, -50.5), turned to -90 degrees
Connections:
- U3 pad 3: GND -> +5V
- U3 pad 4: +5V -> GND
- U4 pad 1: unconnected-(U4-PA02_A0_D0-Pad1) -> Net-(U1-RX)
- U4 pad 2: unconnected-(U4-PA4_A1_D1-Pad2) -> Net-(U1-TX)
- U4 pad 7: Net-(U1-RX) -> unconnected-(U4-PB08_A6_D6_TX-Pad7)
- U4 pad 8: Net-(U1-TX) -> Net-(J2-Pin_2)
- U4 pad 9: unconnected-(U4-PA7_A8_D8_SCK-Pad9) -> Net-(J2-Pin_3)
Routing:
- net GND: track 50.4 -> 102.3 mm
- net Net-(J2-Pin_3): track 0.00 -> 39.5 mm
- net Net-(J2-Pin_2): track 0.00 -> 38.1 mm
- net Net-(U1-TX): track 40.5 -> 17.6 mm
- net Net-(U1-RX): track 4.91 -> 23.4 mm
- net +5V: track 47.3 -> 65.8 mm
- net +3V3: track 33.5 -> 28.1 mm
- net unconnected-(U4-PA4_A1_D1-Pad2): track 0.52 -> 0.00 mm
Other:
- outline, holes or cut-outs redrawn
