File: ESP/Multi-PZEM/PZEM-Single Ultra-Compact LPKF - R1/PZEM-Single LPKF - R2.kicad_sch (KiCad schematic)
At the start: 10 parts, among them J1 Conn_01x02, U4 SEEEDUINO-XIAO-ESP32C3

Commit message: Ordered stuff!
Parts:
- added J2: Conn_01x04_Pin, Connector_JST:JST_XH_B4B-XH-A_1x04_P2.50mm_Vertical, symbol Connector:Conn_01x04_Pin
- H1, H2, H3, H4: footprint MountingHole:MountingHole_3.2mm_M3_Pad_Via -> MountingHole:MountingHole_3.2mm_M3_Pad
Connections:
- net +5V: now also U3.3 (+Vo), J2.1 (Pin_1); no longer U3.4 (+Vo)
- net GND: now also U3.4 (-Vo), J2.4 (Pin_4); no longer U3.3 (-Vo)
- net at U4.1 (PA02_A0_D0): now also U1.6 (RX)
- net at U4.2 (PA4_A1_D1): now also U1.7 (TX)
- net at U4.7 (PB08_A6_D6_TX): no longer U1.6 (RX)
- net at U4.8 (PB09_A7_D7_RX): now also J2.2 (Pin_2); no longer U1.7 (TX)
- net at U4.9 (PA7_A8_D8_SCK): now also J2.3 (Pin_3)
