File: misc/EZ Stepper Line Driver - R2/EZ Stepper Line Driver - R2.kicad_pcb (KiCad board)
At the start: 2 copper layers, 18.5 x 22.9 mm, 17 parts, among them J1 Conn_02x04_Odd_Even, U1 EZ Driver Interface, U2 74LVC2G17, U3 74LVC2G17

Commit message: Ordered stuff!
Routing:
- net GND: track 27.8 -> 27.2 mm
